File: PCB/Bus/Bus.kicad_pcb (KiCad board)
At the start: 2 copper layers, 102 x 102 mm, 74 parts, among them J15 Conn_01x24, J16 Conn_01x24, J17 Conn_01x24, J18 Conn_01x24, J19 Conn_01x24, J20 Conn_01x24, J21 Conn_01x03, J22 Conn_01x03, J23 Conn_01x03, J24 Conn_01x03, J25 Conn_01x03, J26 Conn_01x03, J27 Conn_01x03, J28 Conn_01x03, J29 Conn_01x03, J30 Conn_01x03, J31 Conn_01x03, J32 Conn_01x03, J33 Conn_01x03, J34 Conn_01x03, J35 Conn_01x03, J36 Conn_01x03

Commit message: WIP
Parts:
- removed the J15 at (73.5, 119.8)
- removed the J15 at (139.5, 119.8)
- removed the J15 at (106.5, 119.8)
- removed the J16 at (126.5, 119.8)
- removed the J16 at (60.5, 119.8)
- removed the J16 at (93.5, 119.8)
- removed the J17 at (106.5, 85.4)
- removed the J17 at (139.5, 85.4)
- removed the J17 at (73.5, 85.4)
- removed J18 (x3), J19 (x3), J20 (x3): Conn_01x24, matseng:PinHeader_1x24_P1.27mm_NoTop
- removed J21 (x3), J22 (x3), J23 (x3), J24 (x3), J25 (x3), J26 (x3), J27 (x3), J28 (x3), J29 (x3), J30 (x3), J31 (x3), J32 (x3), J33 (x3), J34 (x3), J35 (x3), J36 (x3): Conn_01x03, matseng:PinHeader_1x03_P2.54mm_Vertical_SMD_Pin1Left_FAT
- removed TP1, TP2, TP3, TP4: TestPoint, TestPoint:TestPoint_THTPad_1.5x1.5mm_Drill0.7mm
- added H10: MountingHole, matseng:MountingHole_M2, F.Cu at (177.2, 340.4)
- added H11: MountingHole, matseng:MountingHole_M2, F.Cu at (153.0, 167.6)
- added H12: MountingHole, matseng:MountingHole_M2, F.Cu at (153.0, 238.8)
- added H13: MountingHole, matseng:MountingHole_M2, F.Cu at (177.2, 167.6)
- added H14: MountingHole, matseng:MountingHole_M2, F.Cu at (177.2, 238.8)
- added H15: MountingHole, matseng:MountingHole_M2, F.Cu at (177.2, 250.2)
- added H16: MountingHole, matseng:MountingHole_M2, F.Cu at (153.0, 250.2)
- added H5: MountingHole, matseng:MountingHole_M2, F.Cu at (177.2, 321.3)
- added H6: MountingHole, matseng:MountingHole_M2, F.Cu at (177.2, 66.0)
- added H7: MountingHole, matseng:MountingHole_M2, F.Cu at (153.0, 85.1)
- added H8: MountingHole, matseng:MountingHole_M2, F.Cu at (177.2, 85.1)
- added H9: MountingHole, matseng:MountingHole_M2, F.Cu at (153.0, 340.4)
- added J1: Conn_01x25_Pin, Connector_PinSocket_2.54mm:PinSocket_1x25_P2.54mm_Vertical, F.Cu at (176.5, 255.3)
- added J10: Conn_01x12_Socket, Connector_PinSocket_2.54mm:PinSocket_1x12_P2.54mm_Vertical, F.Cu at (151.1, 334.0)
- added J11: Conn_01x25_Pin, Connector_PinSocket_2.54mm:PinSocket_1x25_P2.54mm_Vertical, F.Cu at (176.5, 90.2)
- added J12: Conn_01x25_Pin, Connector_PinSocket_2.54mm:PinSocket_1x25_P2.54mm_Vertical, F.Cu at (179.1, 172.7)
- added J13: Conn_01x25_Pin, Connector_PinSocket_2.54mm:PinSocket_1x25_P2.54mm_Vertical, F.Cu at (176.5, 172.7)
- added J14: Conn_01x25_Pin, Connector_PinSocket_2.54mm:PinSocket_1x25_P2.54mm_Vertical, F.Cu at (151.1, 90.2)
- added J15: Conn_01x25_Pin, Connector_PinSocket_2.54mm:PinSocket_1x25_P2.54mm_Vertical, F.Cu at (153.7, 90.2)
- added J16: Conn_01x25_Pin, Connector_PinSocket_2.54mm:PinSocket_1x25_P2.54mm_Vertical, F.Cu at (179.1, 90.2)
- added J17: Conn_01x12_Socket, Connector_PinSocket_2.54mm:PinSocket_1x12_P2.54mm_Vertical, F.Cu at (151.1, 69.8)
- added J2: Conn_01x25_Pin, Connector_PinSocket_2.54mm:PinSocket_1x25_P2.54mm_Vertical, F.Cu at (179.1, 255.3)
- added J3: Conn_01x25_Pin, Connector_PinSocket_2.54mm:PinSocket_1x25_P2.54mm_Vertical, F.Cu at (153.7, 172.7)
- added J4: Conn_01x25_Pin, Connector_PinSocket_2.54mm:PinSocket_1x25_P2.54mm_Vertical, F.Cu at (151.1, 172.7)
- added J5: Conn_01x25_Pin, Connector_PinSocket_2.54mm:PinSocket_1x25_P2.54mm_Vertical, F.Cu at (153.7, 255.3)
- added J6: Conn_01x25_Pin, Connector_PinSocket_2.54mm:PinSocket_1x25_P2.54mm_Vertical, F.Cu at (151.1, 255.3)
- added J8: Conn_01x12_Socket, Connector_PinSocket_2.54mm:PinSocket_1x12_P2.54mm_Vertical, F.Cu at (151.2, 72.4)
- added J9: Conn_01x12_Socket, Connector_PinSocket_2.54mm:PinSocket_1x12_P2.54mm_Vertical, F.Cu at (151.1, 336.6)
- added kibuzzard-656A4AAD: G***, kibuzzard-656A4AAD, F.Cu at (165.2, 80.3)
- added kibuzzard-656A4AB4: G***, kibuzzard-656A4AB4, F.Cu at (165.2, 203.1)
- added kibuzzard-656A4ABF: G***, kibuzzard-656A4ABF, F.Cu at (165.1, 326.3)
- H1, H2, H3, H4: footprint MountingHole:MountingHole_2.2mm_M2_DIN965_Pad_TopBottom -> matseng:MountingHole_M2
- moved H4 249.9 mm to (153.0, 321.3)
- moved H3 91.1 mm to (177.2, 156.2)
- moved H2 85.4 mm to (153.0, 156.2), turned to 90 degrees
- moved H1 59.2 mm to (153.0, 66.0)
Routing:
- net /ABUS18: track 751.0 -> 0.00 mm, vias 9 -> 0
- net /ABUS15: track 595.8 -> 0.00 mm, vias 9 -> 0
- net /ABUS12: track 504.8 -> 0.00 mm, vias 6 -> 0
- net /ABUS23: track 503.8 -> 0.00 mm, vias 6 -> 0
- net /ABUS24: track 502.9 -> 0.00 mm, vias 9 -> 0
- net /ABUS9: track 492.4 -> 0.00 mm, vias 6 -> 0
- net /ABUS21: track 488.0 -> 0.00 mm, vias 6 -> 0
- net /ABUS22: track 486.6 -> 0.00 mm, vias 6 -> 0
- net /ABUS20: track 470.1 -> 0.00 mm, vias 6 -> 0
- net /ABUS19: track 467.0 -> 0.00 mm, vias 6 -> 0
- net /ABUS11: track 463.2 -> 0.00 mm, vias 6 -> 0
- net /ABUS10: track 459.7 -> 0.00 mm, vias 3 -> 0
- net /ABUS8: track 459.4 -> 0.00 mm, vias 6 -> 0
- net /ABUS7: track 455.9 -> 0.00 mm, vias 6 -> 0
- net /ABUS6: track 455.6 -> 0.00 mm, vias 6 -> 0
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- added copper zone on B.Cu, net GNDD
- added copper zone on F.Cu, net GNDD
- added copper zone on B.Cu, net VCC
- added copper zone on F.Cu, net VCC
- removed copper zone on B.Cu, net /ABUS18
- removed copper zone on B.Cu, net Net-(TP3-Pad1)
Other:
- board size 102 x 102 mm -> 33 x 279.4 mm
- board text added: "CONTROL PANEL"
- board text added: "GPIO"
- board text added: "LATCHED SUBTRACTOR"
- board text added: "MAR NEG-DETECT"
- board text added: "MEMORY"
- board text added: "MICRO-OPS"
- board text added: "PROGRAM COUNTER"
- board text added: "SPARE"
- board text added: "UART & LOADER"
- board text removed: "ADDRESS BUS"
- board text removed: "DATA BUS"
- board text removed: "DISCRETE 24 BIT SUBLEQ TRIPLE BUS GITHUB.COM/MENGSTR/SUBLEQ24 18 OCTOBER 2003"
- board text removed: "GND"
- board text removed: "MISC BUS"
- board text removed: "VCC"
- board text removed: "locked"
