File: PCB/Bus/Bus.kicad_sch (KiCad schematic)
At the start: 30 parts, among them J1 Conn_01x24, J2 Conn_01x24, J21 Conn_01x03, J22 Conn_01x03, J23 Conn_01x03, J24 Conn_01x03, J25 Conn_01x03, J26 Conn_01x03, J27 Conn_01x03, J28 Conn_01x03, J29 Conn_01x03, J3 Conn_01x24, J30 Conn_01x03, J31 Conn_01x03, J32 Conn_01x03, J33 Conn_01x03, J34 Conn_01x03, J35 Conn_01x03, J36 Conn_01x03

Commit message: WIP
Parts:
- removed J1 (x2), J2 (x2), J3 (x2): Conn_01x24, matseng:PinHeader_1x24_P1.27mm_NoTop, symbol Connector_Generic:Conn_01x24
- removed J21, J22, J23, J24, J25, J26, J27, J28, J29, J30, J31, J32, J33, J34, J35, J36: Conn_01x03, matseng:PinHeader_1x03_P2.54mm_Vertical_SMD_Pin1Left_FAT, symbol Connector_Generic:Conn_01x03
- removed TP1, TP2, TP3, TP4: TestPoint, TestPoint:TestPoint_THTPad_1.5x1.5mm_Drill0.7mm, symbol Connector:TestPoint
- added H10, H11, H12, H13, H14, H15, H16, H5, H6, H7, H8, H9: MountingHole, matseng:MountingHole_M2, symbol Mechanical:MountingHole
- added J1, J11, J12, J13, J14, J15, J16, J2, J3, J4, J5, J6: Conn_01x25_Pin, Connector_PinSocket_2.54mm:PinSocket_1x25_P2.54mm_Vertical, symbol Connector:Conn_01x25_Pin
- added J10, J17, J18, J7, J8, J9: Conn_01x12_Socket, Connector_PinSocket_2.54mm:PinSocket_1x12_P2.54mm_Vertical, symbol Connector:Conn_01x12_Socket
- H1, H2, H3, H4: footprint MountingHole:MountingHole_2.2mm_M2_DIN965_Pad_TopBottom -> matseng:MountingHole_M2
Connections:
- new net A0: J1.1 (Pin_1), J11.1 (Pin_1), J13.1 (Pin_1), J15.1 (Pin_1), J3.1 (Pin_1), J5.1 (Pin_1)
- new net A1: J12.1 (Pin_1), J14.1 (Pin_1), J16.1 (Pin_1), J2.1 (Pin_1), J4.1 (Pin_1), J6.1 (Pin_1)
- new net A10: J1.6 (Pin_6), J11.6 (Pin_6), J13.6 (Pin_6), J15.6 (Pin_6), J3.6 (Pin_6), J5.6 (Pin_6)
- new net A11: J12.6 (Pin_6), J14.6 (Pin_6), J16.6 (Pin_6), J2.6 (Pin_6), J4.6 (Pin_6), J6.6 (Pin_6)
- new net A12: J1.7 (Pin_7), J11.7 (Pin_7), J13.7 (Pin_7), J15.7 (Pin_7), J3.7 (Pin_7), J5.7 (Pin_7)
- new net A13: J12.7 (Pin_7), J14.7 (Pin_7), J16.7 (Pin_7), J2.7 (Pin_7), J4.7 (Pin_7), J6.7 (Pin_7)
- new net A14: J1.8 (Pin_8), J11.8 (Pin_8), J13.8 (Pin_8), J15.8 (Pin_8), J3.8 (Pin_8), J5.8 (Pin_8)
- new net A15: J12.8 (Pin_8), J14.8 (Pin_8), J16.8 (Pin_8), J2.8 (Pin_8), J4.8 (Pin_8), J6.8 (Pin_8)
- new net A16: J1.9 (Pin_9), J11.9 (Pin_9), J13.9 (Pin_9), J15.9 (Pin_9), J3.9 (Pin_9), J5.9 (Pin_9)
- new net A17: J12.9 (Pin_9), J14.9 (Pin_9), J16.9 (Pin_9), J2.9 (Pin_9), J4.9 (Pin_9), J6.9 (Pin_9)
- new net A18: J1.10 (Pin_10), J11.10 (Pin_10), J13.10 (Pin_10), J15.10 (Pin_10), J3.10 (Pin_10), J5.10 (Pin_10)
- new net A19: J12.10 (Pin_10), J14.10 (Pin_10), J16.10 (Pin_10), J2.10 (Pin_10), J4.10 (Pin_10), J6.10 (Pin_10)
- new net A2: J1.2 (Pin_2), J11.2 (Pin_2), J13.2 (Pin_2), J15.2 (Pin_2), J3.2 (Pin_2), J5.2 (Pin_2)
- new net A20: J1.11 (Pin_11), J11.11 (Pin_11), J13.11 (Pin_11), J15.11 (Pin_11), J3.11 (Pin_11), J5.11 (Pin_11)
- new net A21: J12.11 (Pin_11), J14.11 (Pin_11), J16.11 (Pin_11), J2.11 (Pin_11), J4.11 (Pin_11), J6.11 (Pin_11)
- new net A22: J1.12 (Pin_12), J11.12 (Pin_12), J13.12 (Pin_12), J15.12 (Pin_12), J3.12 (Pin_12), J5.12 (Pin_12)
- new net A23: J12.12 (Pin_12), J14.12 (Pin_12), J16.12 (Pin_12), J2.12 (Pin_12), J4.12 (Pin_12), J6.12 (Pin_12)
- new net A3: J12.2 (Pin_2), J14.2 (Pin_2), J16.2 (Pin_2), J2.2 (Pin_2), J4.2 (Pin_2), J6.2 (Pin_2)
- new net A4: J1.3 (Pin_3), J11.3 (Pin_3), J13.3 (Pin_3), J15.3 (Pin_3), J3.3 (Pin_3), J5.3 (Pin_3)
- new net A5: J12.3 (Pin_3), J14.3 (Pin_3), J16.3 (Pin_3), J2.3 (Pin_3), J4.3 (Pin_3), J6.3 (Pin_3)
- new net A6: J1.4 (Pin_4), J11.4 (Pin_4), J13.4 (Pin_4), J15.4 (Pin_4), J3.4 (Pin_4), J5.4 (Pin_4)
- new net A7: J12.4 (Pin_4), J14.4 (Pin_4), J16.4 (Pin_4), J2.4 (Pin_4), J4.4 (Pin_4), J6.4 (Pin_4)
- new net A8: J1.5 (Pin_5), J11.5 (Pin_5), J13.5 (Pin_5), J15.5 (Pin_5), J3.5 (Pin_5), J5.5 (Pin_5)
- new net A9: J12.5 (Pin_5), J14.5 (Pin_5), J16.5 (Pin_5), J2.5 (Pin_5), J4.5 (Pin_5), J6.5 (Pin_5)
- new net D0: J1.13 (Pin_13), J11.13 (Pin_13), J13.13 (Pin_13), J15.13 (Pin_13), J3.13 (Pin_13), J5.13 (Pin_13)
- new net D1: J12.13 (Pin_13), J14.13 (Pin_13), J16.13 (Pin_13), J2.13 (Pin_13), J4.13 (Pin_13), J6.13 (Pin_13)
- new net D10: J1.18 (Pin_18), J11.18 (Pin_18), J13.18 (Pin_18), J15.18 (Pin_18), J3.18 (Pin_18), J5.18 (Pin_18)
- new net D11: J12.18 (Pin_18), J14.18 (Pin_18), J16.18 (Pin_18), J2.18 (Pin_18), J4.18 (Pin_18), J6.18 (Pin_18)
- new net D12: J1.19 (Pin_19), J11.19 (Pin_19), J13.19 (Pin_19), J15.19 (Pin_19), J3.19 (Pin_19), J5.19 (Pin_19)
- new net D13: J12.19 (Pin_19), J14.19 (Pin_19), J16.19 (Pin_19), J2.19 (Pin_19), J4.19 (Pin_19), J6.19 (Pin_19)
- new net D14: J1.20 (Pin_20), J11.20 (Pin_20), J13.20 (Pin_20), J15.20 (Pin_20), J3.20 (Pin_20), J5.20 (Pin_20)
- new net D15: J12.20 (Pin_20), J14.20 (Pin_20), J16.20 (Pin_20), J2.20 (Pin_20), J4.20 (Pin_20), J6.20 (Pin_20)
- new net D16: J1.21 (Pin_21), J11.21 (Pin_21), J13.21 (Pin_21), J15.21 (Pin_21), J3.21 (Pin_21), J5.21 (Pin_21)
- new net D17: J12.21 (Pin_21), J14.21 (Pin_21), J16.21 (Pin_21), J2.21 (Pin_21), J4.21 (Pin_21), J6.21 (Pin_21)
- new net D18: J1.22 (Pin_22), J11.22 (Pin_22), J13.22 (Pin_22), J15.22 (Pin_22), J3.22 (Pin_22), J5.22 (Pin_22)
- new net D19: J12.22 (Pin_22), J14.22 (Pin_22), J16.22 (Pin_22), J2.22 (Pin_22), J4.22 (Pin_22), J6.22 (Pin_22)
- new net D2: J1.14 (Pin_14), J11.14 (Pin_14), J13.14 (Pin_14), J15.14 (Pin_14), J3.14 (Pin_14), J5.14 (Pin_14)
- new net D20: J1.23 (Pin_23), J11.23 (Pin_23), J13.23 (Pin_23), J15.23 (Pin_23), J3.23 (Pin_23), J5.23 (Pin_23)
- new net D21: J12.23 (Pin_23), J14.23 (Pin_23), J16.23 (Pin_23), J2.23 (Pin_23), J4.23 (Pin_23), J6.23 (Pin_23)
- new net D22: J1.24 (Pin_24), J11.24 (Pin_24), J13.24 (Pin_24), J15.24 (Pin_24), J3.24 (Pin_24), J5.24 (Pin_24)
- new net D23: J12.24 (Pin_24), J14.24 (Pin_24), J16.24 (Pin_24), J2.24 (Pin_24), J4.24 (Pin_24), J6.24 (Pin_24)
- new net D3: J12.14 (Pin_14), J14.14 (Pin_14), J16.14 (Pin_14), J2.14 (Pin_14), J4.14 (Pin_14), J6.14 (Pin_14)
- new net D4: J1.15 (Pin_15), J11.15 (Pin_15), J13.15 (Pin_15), J15.15 (Pin_15), J3.15 (Pin_15), J5.15 (Pin_15)
- new net D5: J12.15 (Pin_15), J14.15 (Pin_15), J16.15 (Pin_15), J2.15 (Pin_15), J4.15 (Pin_15), J6.15 (Pin_15)
- new net D6: J1.16 (Pin_16), J11.16 (Pin_16), J13.16 (Pin_16), J15.16 (Pin_16), J3.16 (Pin_16), J5.16 (Pin_16)
- new net D7: J12.16 (Pin_16), J14.16 (Pin_16), J16.16 (Pin_16), J2.16 (Pin_16), J4.16 (Pin_16), J6.16 (Pin_16)
- new net D8: J1.17 (Pin_17), J11.17 (Pin_17), J13.17 (Pin_17), J15.17 (Pin_17), J3.17 (Pin_17), J5.17 (Pin_17)
- new net D9: J12.17 (Pin_17), J14.17 (Pin_17), J16.17 (Pin_17), J2.17 (Pin_17), J4.17 (Pin_17), J6.17 (Pin_17)
- new net GNDD: J12.25 (Pin_25), J14.25 (Pin_25), J16.25 (Pin_25), J2.25 (Pin_25), J4.25 (Pin_25), J6.25 (Pin_25)
- new net VCC: J1.25 (Pin_25), J11.25 (Pin_25), J13.25 (Pin_25), J15.25 (Pin_25), J3.25 (Pin_25), J5.25 (Pin_25)
