File: PCB/OLD/OLD1/Subtractor/Subtractor.kicad_pcb (KiCad board)
At the start: 2 copper layers, 102 x 102 mm, 82 parts, among them U1 74LS540, U10 74LS283, U12 74LS283, U13 74HC245, U15 74LS283, U16 74LS30, U17 74LS27, U18 74LS27, U19 74LS27, U2 74LS283, U20 74LS00, U21 74LS540, U3 74HC245, U4 74LS540, U5 74LS283, U7 74LS283, U8 74HC245

Commit message: WIP
Parts:
- turned D27 to 180 degrees
Connections:
- D27 pad 1: Net-(D27-K) -> GNDD
- D27 pad 2: GNDD -> Net-(D27-A)
- R2 pad 1: Net-(D27-K) -> Net-(D27-A)
Routing:
- net Net-(D27-K): track 2.55 -> 0.00 mm
- net Net-(D27-A): track 0.00 -> 2.55 mm
Changed lines of the file:
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@@
   (net 171 "Net-(D26-K)")
   (net 172 "Net-(D26-A)")
-  (net 173 "Net-(D27-K)")
+  (net 173 "Net-(D27-A)")
   (footprint "LED_SMD:LED_0805_2012Metric_Pad1.15x1.40mm_HandSolder" (layer "F.Cu")
     (at 67.437 77.089)
@@
       (stroke (width 0.1) (type solid)) (layer "F.Fab"))
     (pad "1" smd roundrect (at -1 0) (size 1.2 1.4) (layers "F.Cu" "F.Paste" "F.Mask") (roundrect_rratio 0.2083333333)
-      (net 173 "Net-(D27-K)") (pintype "passive"))
+      (net 173 "Net-(D27-A)") (pintype "passive"))
     (pad "2" smd roundrect (at 1 0) (size 1.2 1.4) (layers "F.Cu" "F.Paste" "F.Mask") (roundrect_rratio 0.2083333333)
       (net 46 "VCC") (pintype "passive"))
@@
   )
   (footprint "LED_SMD:LED_0805_2012Metric_Pad1.15x1.40mm_HandSolder" (layer "F.Cu")
-    (at 137.16 144.78)
+    (at 137.16 144.78 180)
     (descr "LED SMD 0805 (2012 Metric), square (rectangular) end terminal, IPC_7351 nominal, (Body size source: https://docs.google.com/spreadsheets/d/1BsfQQcO9C6DZCsRaXUlFlo91Tg2WpOkGARC1WS5S8t0/edit?usp=sharing), generated with kicad-footprint-generator")
     (tags "LED handsolder")
@@
     (fp_line (start 1 0.6) (end 1 -0.6)
       (stroke (width 0.1) (type solid)) (layer "F.Fab"))
-    (pad "1" smd roundrect (at -1.025 0) (size 1.15 1.4) (layers "F.Cu" "F.Paste" "F.Mask") (roundrect_rratio 0.2173913043)
-      (net 173 "Net-(D27-K)") (pinfunction "K") (pintype "passive"))
-    (pad "2" smd roundrect (at 1.025 0) (size 1.15 1.4) (layers "F.Cu" "F.Paste" "F.Mask") (roundrect_rratio 0.2173913043)
-      (net 45 "GNDD") (pinfunction "A") (pintype "passive"))
+    (pad "1" smd roundrect (at -1.025 0 180) (size 1.15 1.4) (layers "F.Cu" "F.Paste" "F.Mask") (roundrect_rratio 0.2173913043)
+      (net 45 "GNDD") (pinfunction "K") (pintype "passive"))
+    (pad "2" smd roundrect (at 1.025 0 180) (size 1.15 1.4) (layers "F.Cu" "F.Paste" "F.Mask") (roundrect_rratio 0.2173913043)
+      (net 173 "Net-(D27-A)") (pinfunction "A") (pintype "passive"))
     (model "${KICAD6_3DMODEL_DIR}/LED_SMD.3dshapes/LED_0805_2012Metric.wrl"
       (offset (xyz 0 0 0))
