File: PCB/OLD/OLD1/Subtractor/Subtractor.kicad_sch (KiCad schematic)
At the start: 82 parts, among them J1 Conn_01x24, J2 Conn_01x24, J3 Conn_01x24, U1 74LS540, U10 74LS283, U12 74LS283, U13 74HC245, U15 74LS283, U16 74LS30, U17 74LS27, U18 74LS27, U19 74LS27, U2 74LS283, U20 74LS00, U21 74LS540, U3 74HC245, U4 74LS540, U5 74LS283, U7 74LS283, U8 74HC245

Commit message: WIP
Connections:
- net GNDD: now also D27.1 (K); no longer D27.2 (A)
- net at R2.1: now also D27.2 (A); no longer D27.1 (K)
Other:
- moved on the sheet: D27, H1, H2, H3, H4, J1, J2, J3, TP1, TP4
