File: PCB/Backplane/Backplane.kicad_pcb (KiCad board)
At the start: 2 copper layers, 33 x 279.4 mm, 35 parts, among them J1 Conn_01x25_Pin, J10 Conn_01x12_Socket, J11 Conn_01x25_Pin, J12 Conn_01x25_Pin, J13 Conn_01x25_Pin, J14 Conn_01x25_Pin, J15 Conn_01x25_Pin, J16 Conn_01x25_Pin, J17 Conn_01x12_Socket, J2 Conn_01x25_Pin, J3 Conn_01x25_Pin, J4 Conn_01x25_Pin, J5 Conn_01x25_Pin, J6 Conn_01x25_Pin, J8 Conn_01x12_Socket, J9 Conn_01x12_Socket

Commit message: Update readme
Parts:
- moved kibuzzard-656A4AAD 1.00 mm to (165.2, 79.3)
- moved kibuzzard-656A4ABF 1.00 mm to (165.1, 327.3)
Connections:
- J10 pad 1: unconnected-(J10-Pin_1-Pad1) -> /A3
- J10 pad 10: unconnected-(J10-Pin_10-Pad10) -> /D15
- J10 pad 11: unconnected-(J10-Pin_11-Pad11) -> /D19
- J10 pad 12: unconnected-(J10-Pin_12-Pad12) -> /D23
- J10 pad 2: unconnected-(J10-Pin_2-Pad2) -> /A7
- J10 pad 3: unconnected-(J10-Pin_3-Pad3) -> /A11
- J10 pad 4: unconnected-(J10-Pin_4-Pad4) -> /A15
- J10 pad 5: unconnected-(J10-Pin_5-Pad5) -> /A19
- J10 pad 6: unconnected-(J10-Pin_6-Pad6) -> /A23
- J10 pad 7: unconnected-(J10-Pin_7-Pad7) -> /D3
- J10 pad 8: unconnected-(J10-Pin_8-Pad8) -> /D7
- J10 pad 9: unconnected-(J10-Pin_9-Pad9) -> /D11
- J17 pad 1: unconnected-(J17-Pin_1-Pad1) -> /A0
- J17 pad 10: unconnected-(J17-Pin_10-Pad10) -> /D12
- J17 pad 11: unconnected-(J17-Pin_11-Pad11) -> /D16
- J17 pad 12: unconnected-(J17-Pin_12-Pad12) -> /D20
- J17 pad 2: unconnected-(J17-Pin_2-Pad2) -> /A4
- J17 pad 3: unconnected-(J17-Pin_3-Pad3) -> /A8
- J17 pad 4: unconnected-(J17-Pin_4-Pad4) -> /A12
- J17 pad 5: unconnected-(J17-Pin_5-Pad5) -> /A16
- J17 pad 6: unconnected-(J17-Pin_6-Pad6) -> /A20
- J17 pad 7: unconnected-(J17-Pin_7-Pad7) -> /D0
- J17 pad 8: unconnected-(J17-Pin_8-Pad8) -> /D4
- J17 pad 9: unconnected-(J17-Pin_9-Pad9) -> /D8
- J8 pad 1: unconnected-(J8-Pin_1-Pad1) -> /A1
- J8 pad 10: unconnected-(J8-Pin_10-Pad10) -> /D13
- J8 pad 11: unconnected-(J8-Pin_11-Pad11) -> /D17
- J8 pad 12: unconnected-(J8-Pin_12-Pad12) -> /D21
- J8 pad 2: unconnected-(J8-Pin_2-Pad2) -> /A5
- J8 pad 3: unconnected-(J8-Pin_3-Pad3) -> /A9
- J8 pad 4: unconnected-(J8-Pin_4-Pad4) -> /A13
- J8 pad 5: unconnected-(J8-Pin_5-Pad5) -> /A17
- J8 pad 6: unconnected-(J8-Pin_6-Pad6) -> /A21
- J8 pad 7: unconnected-(J8-Pin_7-Pad7) -> /D1
- J8 pad 8: unconnected-(J8-Pin_8-Pad8) -> /D5
- J8 pad 9: unconnected-(J8-Pin_9-Pad9) -> /D9
- J9 pad 1: unconnected-(J9-Pin_1-Pad1) -> /A2
- J9 pad 10: unconnected-(J9-Pin_10-Pad10) -> /D14
- J9 pad 11: unconnected-(J9-Pin_11-Pad11) -> /D18
- J9 pad 12: unconnected-(J9-Pin_12-Pad12) -> /D22
- J9 pad 2: unconnected-(J9-Pin_2-Pad2) -> /A6
- J9 pad 3: unconnected-(J9-Pin_3-Pad3) -> /A10
- J9 pad 4: unconnected-(J9-Pin_4-Pad4) -> /A14
- J9 pad 5: unconnected-(J9-Pin_5-Pad5) -> /A18
- J9 pad 6: unconnected-(J9-Pin_6-Pad6) -> /A22
- J9 pad 7: unconnected-(J9-Pin_7-Pad7) -> /D2
- J9 pad 8: unconnected-(J9-Pin_8-Pad8) -> /D6
- J9 pad 9: unconnected-(J9-Pin_9-Pad9) -> /D10
Routing:
- net /A1: track 327.4 -> 271.3 mm, vias 5 -> 3
- net /A0: track 309.9 -> 257.2 mm, vias 5 -> 3
- net /A5: track 327.7 -> 276.2 mm, vias 5 -> 3
- net /D23: track 327.7 -> 276.6 mm, vias 5 -> 3
- net /D22: track 309.7 -> 261.2 mm, vias 5 -> 3
- net /A4: track 310.0 -> 261.9 mm, vias 5 -> 3
- net /A9: track 327.6 -> 280.9 mm, vias 5 -> 3
- net /D19: track 327.6 -> 281.2 mm, vias 5 -> 3
- net /D18: track 309.6 -> 266.1 mm, vias 5 -> 3
- net /A8: track 309.9 -> 266.5 mm, vias 5 -> 3
- net /A13: track 327.7 -> 285.5 mm, vias 5 -> 3
- net /D15: track 327.7 -> 285.9 mm, vias 5 -> 3
- net /D14: track 309.7 -> 270.8 mm, vias 5 -> 3
- net /A12: track 310.0 -> 271.2 mm, vias 5 -> 3
- net /A17: track 327.6 -> 290.2 mm, vias 5 -> 3
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Other:
- board text added: "3V3"
- board text added: "Backplane"
- board text added: "GND"
- board text added: "github.com/mengstr/SUBLEQ24"
- board text added: "rev1"
