File: PCB/Backplane/Backplane.kicad_sch (KiCad schematic)
At the start: 34 parts, among them J1 Conn_01x25_Pin, J10 Conn_01x12_Socket, J11 Conn_01x25_Pin, J12 Conn_01x25_Pin, J13 Conn_01x25_Pin, J14 Conn_01x25_Pin, J15 Conn_01x25_Pin, J16 Conn_01x25_Pin, J17 Conn_01x12_Socket, J18 Conn_01x12_Socket, J2 Conn_01x25_Pin, J3 Conn_01x25_Pin, J4 Conn_01x25_Pin, J5 Conn_01x25_Pin, J6 Conn_01x25_Pin, J7 Conn_01x12_Socket, J8 Conn_01x12_Socket, J9 Conn_01x12_Socket

Commit message: Update readme
Parts:
- removed J18, J7: Conn_01x12_Socket, Connector_PinSocket_2.54mm:PinSocket_1x12_P2.54mm_Vertical, symbol Connector:Conn_01x12_Socket
Connections:
- net A0: now also J17.1 (Pin_1)
- net A1: now also J8.1 (Pin_1)
- net A10: now also J9.3 (Pin_3)
- net A11: now also J10.3 (Pin_3)
- net A12: now also J17.4 (Pin_4)
- net A13: now also J8.4 (Pin_4)
- net A14: now also J9.4 (Pin_4)
- net A15: now also J10.4 (Pin_4)
- net A16: now also J17.5 (Pin_5)
- net A17: now also J8.5 (Pin_5)
- net A18: now also J9.5 (Pin_5)
- net A19: now also J10.5 (Pin_5)
- net A2: now also J9.1 (Pin_1)
- net A20: now also J17.6 (Pin_6)
- net A21: now also J8.6 (Pin_6)
- net A22: now also J9.6 (Pin_6)
- net A23: now also J10.6 (Pin_6)
- net A3: now also J10.1 (Pin_1)
- net A4: now also J17.2 (Pin_2)
- net A5: now also J8.2 (Pin_2)
- net A6: now also J9.2 (Pin_2)
- net A7: now also J10.2 (Pin_2)
- net A8: now also J17.3 (Pin_3)
- net A9: now also J8.3 (Pin_3)
- net D0: now also J17.7 (Pin_7)
- net D1: now also J8.7 (Pin_7)
- net D10: now also J9.9 (Pin_9)
- net D11: now also J10.9 (Pin_9)
- net D12: now also J17.10 (Pin_10)
- net D13: now also J8.10 (Pin_10)
- net D14: now also J9.10 (Pin_10)
- net D15: now also J10.10 (Pin_10)
- net D16: now also J17.11 (Pin_11)
- net D17: now also J8.11 (Pin_11)
- net D18: now also J9.11 (Pin_11)
- net D19: now also J10.11 (Pin_11)
- net D2: now also J9.7 (Pin_7)
- net D20: now also J17.12 (Pin_12)
- net D21: now also J8.12 (Pin_12)
- net D22: now also J9.12 (Pin_12)
- net D23: now also J10.12 (Pin_12)
- net D3: now also J10.7 (Pin_7)
- net D4: now also J17.8 (Pin_8)
- net D5: now also J8.8 (Pin_8)
- net D6: now also J9.8 (Pin_8)
- net D7: now also J10.8 (Pin_8)
- net D8: now also J17.9 (Pin_9)
- net D9: now also J8.9 (Pin_9)
Other:
- moved on the sheet: J10, J17, J8, J9
