File: PCB/BusConnector/BusConnector.kicad_pcb (KiCad board)
At the start: 2 copper layers, 264.2 x 10.2 mm, 3 parts, among them J1 Conn_02x12_Counter_Clockwise, J3 Conn_02x12_Counter_Clockwise

Commit message: Update readme
Other:
- board text added: "•BusConnector • github.com/mengstr/SUBLEQ24 • rev 1 •"
- board text removed: "• SUBLEQ24 • BusConnector • December 2023 • github.com/mengstr •"
