File: PCB/Disp24-7/5xDisp24-7.kicad_pcb (KiCad board)
At the start: 2 copper layers, 86.7 x 95 mm, 140 parts, among them J1 Conn_01x24_Pin, J2 Conn_01x02_Pin, J3 Conn_01x02_Pin, J4 Conn_PIC_ICSP_ICD, Q1 DTA123J, Q2 DTA123J, Q3 DTA123J, Q4 DTA123J, Q5 DTA123J, Q6 DTA123J, U1 PIC16LF15385-xPT

Commit message: Update readme with images
Other:
- board text added: "UP"

Commit message: Update readme
Other:
- board text added: "rev1"
Changed lines of the file:
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@@
       (plot_on_all_layers_selection 0x0000000_00000000)
       (disableapertmacros false)
-      (usegerberextensions false)
-      (usegerberattributes true)
-      (usegerberadvancedattributes true)
-      (creategerberjobfile true)
+      (usegerberextensions true)
+      (usegerberattributes false)
+      (usegerberadvancedattributes false)
+      (creategerberjobfile false)
       (dashed_line_dash_ratio 12.000000)
       (dashed_line_gap_ratio 3.000000)
@@
       (psa4output false)
       (plotreference true)
-      (plotvalue true)
+      (plotvalue false)
       (plotinvisibletext false)
       (sketchpadsonfab false)
-      (subtractmaskfromsilk false)
+      (subtractmaskfromsilk true)
       (outputformat 1)
       (mirror false)
-      (drillshape 1)
+      (drillshape 0)
       (scaleselection 1)
       (outputdirectory "")
@@
     )
   )
+  (gr_text "rev1" (at 94.107 112.83) (layer "F.Mask")
+    (effects (font (size 1.2 1.2) (thickness 0.15)) (justify left bottom))
+  )
+  (gr_text "rev1" (at 94.107 55.83) (layer "F.Mask")
+    (effects (font (size 1.2 1.2) (thickness 0.15)) (justify left bottom))
+  )
+  (gr_text "rev1" (at 94.107 93.83) (layer "F.Mask")
+    (effects (font (size 1.2 1.2) (thickness 0.15)) (justify left bottom))
+  )
+  (gr_text "rev1" (at 94.107 74.83) (layer "F.Mask")
+    (effects (font (size 1.2 1.2) (thickness 0.15)) (justify left bottom))
+  )
+  (gr_text "rev1" (at 94.107 36.83) (layer "F.Mask")
+    (effects (font (size 1.2 1.2) (thickness 0.15)) (justify left bottom))
+  )
   (segment (start 91.366 78.2795) (end 91.366 77.306) (width 0.127) (layer "F.Cu") (net 1))
