File: PCB/Signalling/Signalling.kicad_pcb (KiCad board)
At the start: 2 copper layers, 17.8 x 236.2 mm, 438 parts

Commit message: Update readme
Other:
- board text added: "Signalling"
- board text added: "github.com/ /mengstr/SUBLEQ24"
- board text added: "rev1"
