File: PCB/Programcounter/Programcounter.kicad_sch (KiCad schematic)
At the start: 87 parts, among them J1 Conn_01x24, J2 Conn_01x24, U10 74LS157, U11 74LS157, U12 74LS157, U13 74LS157, U14 74LS157, U15 74LS157, U4 74LS163, U5 74LS163, U6 74LS163, U6 74LS541, U7 74LS163, U8 74LS163, U9 74LS163

Commit message: WIP
Parts:
- removed C1: C, Capacitor_SMD:C_Elec_6.3x5.8, symbol Device:C
- removed C10, C11, C12, C13, C14, C15, C16, C17, C18, C7, C9: C, Capacitor_SMD:C_0805_2012Metric_Pad1.18x1.45mm_HandSolder, symbol Device:C
- removed D1, D10, D11, D12, D13, D14, D15, D16, D17, D18, D19, D2, D20, D21, D22, D23, D24, D25, D26, D27, D28, D29, D3, D30, D4, D5, D6, D7, D8, D9: LED, LED_SMD:LED_0805_2012Metric_Pad1.15x1.40mm_HandSolder, symbol Device:LED
- removed H3, H4: MountingHole, matseng:MountingHole_M2, symbol Mechanical:MountingHole
- removed J1, J2: Conn_01x24, matseng:PinHeader_1x24_P1.27mm_NoSilk, symbol Connector_Generic:Conn_01x24
- removed R1, R2, R3, R4, R5, R6: R, Resistor_SMD:R_0805_2012Metric_Pad1.20x1.40mm_HandSolder, symbol Device:R
- removed RN1, RN2, RN3, RN4, RN5, RN6: R_Pack04, Resistor_SMD:R_Array_Concave_4x0603, symbol Device:R_Pack04
- removed TP1 (x6): TestPoint, TestPoint:TestPoint_THTPad_2.0x2.0mm_Drill1.0mm, symbol Connector:TestPoint
- removed TP2, TP3: TestPoint, TestPoint:TestPoint_THTPad_1.5x1.5mm_Drill0.7mm, symbol Connector:TestPoint
- removed U6 (x3): 74LS541, Package_SO:SOIC-20W_7.5x15.4mm_P1.27mm, symbol 74xx:74LS541
- added BUS1: Conn_02x25_Odd_Even, Connector_PinHeader_2.54mm:PinHeader_2x25_P2.54mm_Vertical, symbol Connector_Generic:Conn_02x25_Odd_Even
- added C1 (x2), C10 (x2), C2, C7 (x2), C8 (x2), C9 (x2), C98, C99: C, Capacitor_SMD:C_0805_2012Metric_Pad1.18x1.45mm_HandSolder, symbol Device:C
- added D99: LED, LED_SMD:LED_0805_2012Metric_Pad1.15x1.40mm_HandSolder, symbol Device:LED
- added J1a1, J1b1, J1c1: Conn_02x04_Odd_Even, Connector_PinHeader_2.54mm:PinHeader_2x04_P2.54mm_Vertical, symbol Connector_Generic:Conn_02x04_Odd_Even
- added J3: Conn_01x08_Pin, Connector_PinHeader_2.54mm:PinHeader_1x08_P2.54mm_Vertical, symbol Connector:Conn_01x08_Pin
- added R99: R, Resistor_SMD:R_0805_2012Metric_Pad1.20x1.40mm_HandSolder, symbol Device:R
- added U6 (x3): 74LS541, Package_SO:SOIC-20W_7.5x12.8mm_P1.27mm, symbol 74xx:74LS541
- H1, H2: now in the parts list
Connections:
- net CP: now also J3.3 (Pin_3)
- net GNDD: now also U15.10 (I1c), BUS1.50 (Pin_50), C1.2, C1.2, C10.2, C10.2, C2.2, C7.2, C7.2, C8.2, C8.2, C9.2, C9.2, C98.2, C99.2, D99.1 (K), U6.10 (GND), U6.10 (GND), U6.10 (GND); no longer U15.13 (I1d)
- net PC0: now also J1a1.1 (Pin_1), U6.2 (A0)
- net PC1: now also J1a1.2 (Pin_2), U6.3 (A1)
- net PC10: now also J1b1.3 (Pin_3), U6.4 (A2)
- net PC11: now also J1b1.4 (Pin_4), U6.5 (A3)
- net PC12: now also J1b1.5 (Pin_5), U6.6 (A4)
- net PC13: now also J1b1.6 (Pin_6), U6.7 (A5)
- net PC14: now also J1b1.7 (Pin_7), U6.8 (A6)
- net PC15: now also J1b1.8 (Pin_8), U6.9 (A7)
- net PC16: now also J1c1.1 (Pin_1), U6.2 (A0)
- net PC17: now also J1c1.2 (Pin_2), U6.3 (A1)
- net PC18: now also J1c1.3 (Pin_3), U6.4 (A2)
- net PC19: now also J1c1.4 (Pin_4), U6.5 (A3)
- net PC2: now also J1a1.3 (Pin_3), U6.4 (A2)
- net PC20: now also J1c1.5 (Pin_5), U6.6 (A4)
- net PC21: now also J1c1.6 (Pin_6), U6.7 (A5)
- net PC22: now also J1c1.7 (Pin_7), U6.8 (A6)
- net PC23: now also J1c1.8 (Pin_8), U6.9 (A7)
- net PC3: now also J1a1.4 (Pin_4), U6.5 (A3)
- net PC4: now also J1a1.5 (Pin_5), U6.6 (A4)
- net PC5: now also J1a1.6 (Pin_6), U6.7 (A5)
- net PC6: now also J1a1.7 (Pin_7), U6.8 (A6)
- net PC7: now also J1a1.8 (Pin_8), U6.9 (A7)
- net PC8: now also J1b1.1 (Pin_1), U6.2 (A0)
- net PC9: now also J1b1.2 (Pin_2), U6.3 (A1)
- net SEL: now also J3.5 (Pin_5)
- net VCC: now also BUS1.49 (Pin_49), C1.1, C1.1, C10.1, C10.1, C2.1, C7.1, C7.1, C8.1, C8.1, C9.1, C9.1, C98.1, C99.1, R99.1, U6.20 (VCC), U6.20 (VCC), U6.20 (VCC)
- net ~{OE}: now also J3.1 (Pin_1), U6.1 (G1), U6.1 (G1), U6.1 (G1), U6.19 (G2), U6.19 (G2), U6.19 (G2)
- net ~{PE}: now also J3.2 (Pin_2)
- net BOOTADDR renamed BootAddr
- net BootAddr: now also U15.13 (I1d), J3.4 (Pin_4); no longer U15.10 (I1c)
- net IN0 renamed D0
- net D0: now also BUS1.25 (Pin_25)
- net IN1 renamed D2
- net D2: now also BUS1.27 (Pin_27)
- net IN10 renamed D11
- net D11: now also BUS1.36 (Pin_36)
- net IN11 renamed D9
- net D9: now also BUS1.34 (Pin_34)
- net IN12 renamed D12
- net D12: now also BUS1.37 (Pin_37)
- net IN13 renamed D14
- net D14: now also BUS1.39 (Pin_39)
- net IN14 renamed D15
- net D15: now also BUS1.40 (Pin_40)
- net IN15 renamed D13
- net D13: now also BUS1.38 (Pin_38)
- net IN16 renamed D16
- net D16: now also BUS1.41 (Pin_41)
- net IN17 renamed D18
- net D18: now also BUS1.43 (Pin_43)
- net IN18 renamed D19
- net D19: now also BUS1.44 (Pin_44)
- net IN19 renamed D17
- net D17: now also BUS1.42 (Pin_42)
- net IN2 renamed D3
- net D3: now also BUS1.28 (Pin_28)
- net IN20 renamed D20
- net D20: now also BUS1.45 (Pin_45)
- net IN21 renamed D22
- net D22: now also BUS1.47 (Pin_47)
- net IN22 renamed D23
- net D23: now also BUS1.48 (Pin_48)
- net IN23 renamed D21
- net D21: now also BUS1.46 (Pin_46)
- net IN3 renamed D1
- net D1: now also BUS1.26 (Pin_26)
- net IN4 renamed D4
- net D4: now also BUS1.29 (Pin_29)
- net IN5 renamed D6
- net D6: now also BUS1.31 (Pin_31)
- net IN6 renamed D7
- net D7: now also BUS1.32 (Pin_32)
- net IN7 renamed D5
- net D5: now also BUS1.30 (Pin_30)
- net IN8 renamed D8
- net D8: now also BUS1.33 (Pin_33)
- net IN9 renamed D10
- net D10: now also BUS1.35 (Pin_35)
- net NEWCNT0 renamed New0
- net NEWCNT1 renamed New1
- net New1: now also U10.12 (Zd); no longer U10.7 (Zb)
- net NEWCNT10 renamed New10
- net New10: now also U12.7 (Zb); no longer U12.9 (Zc)
- net NEWCNT11 renamed New11
- net New11: now also U12.9 (Zc); no longer U12.12 (Zd)
- net NEWCNT12 renamed New12
- net NEWCNT13 renamed New13
- net New13: now also U13.12 (Zd); no longer U13.7 (Zb)
- net NEWCNT14 renamed New14
- net New14: now also U13.7 (Zb); no longer U13.9 (Zc)
- net NEWCNT15 renamed New15
- net New15: now also U13.9 (Zc); no longer U13.12 (Zd)
- net NEWCNT16 renamed New16
- net NEWCNT17 renamed New17
- net New17: now also U14.12 (Zd); no longer U14.7 (Zb)
- net NEWCNT18 renamed New18
- net New18: now also U14.7 (Zb); no longer U14.9 (Zc)
- net NEWCNT19 renamed New19
- net New19: now also U14.9 (Zc); no longer U14.12 (Zd)
- net NEWCNT2 renamed New2
- net New2: now also U10.7 (Zb); no longer U10.9 (Zc)
- net NEWCNT20 renamed New20
- net NEWCNT21 renamed New21
- net New21: now also U15.12 (Zd); no longer U15.7 (Zb)
- net NEWCNT22 renamed New22
- net New22: now also U15.7 (Zb); no longer U15.9 (Zc)
- net NEWCNT23 renamed New23
- net New23: now also U15.9 (Zc); no longer U15.12 (Zd)
- net NEWCNT3 renamed New3
- net New3: now also U10.9 (Zc); no longer U10.12 (Zd)
- net NEWCNT4 renamed New4
- net NEWCNT5 renamed New5
- net New5: now also U11.12 (Zd); no longer U11.7 (Zb)
- net NEWCNT6 renamed New6
- net New6: now also U11.7 (Zb); no longer U11.9 (Zc)
- net NEWCNT7 renamed New7
- net New7: now also U11.9 (Zc); no longer U11.12 (Zd)
- net NEWCNT8 renamed New8
- net NEWCNT9 renamed New9
- net New9: now also U12.12 (Zd); no longer U12.7 (Zb)
- new net: D99.2 (A), R99.2
- new net A0: BUS1.1 (Pin_1), U6.18 (Y0)
- new net A1: BUS1.2 (Pin_2), U6.17 (Y1)
- new net A10: BUS1.11 (Pin_11), U6.16 (Y2)
- new net A11: BUS1.12 (Pin_12), U6.15 (Y3)
- new net A12: BUS1.13 (Pin_13), U6.14 (Y4)
- new net A13: BUS1.14 (Pin_14), U6.13 (Y5)
- new net A14: BUS1.15 (Pin_15), U6.12 (Y6)
- new net A15: BUS1.16 (Pin_16), U6.11 (Y7)
- new net A16: BUS1.17 (Pin_17), U6.18 (Y0)
- new net A17: BUS1.18 (Pin_18), U6.17 (Y1)
- new net A18: BUS1.19 (Pin_19), U6.16 (Y2)
- new net A19: BUS1.20 (Pin_20), U6.15 (Y3)
- new net A2: BUS1.3 (Pin_3), U6.16 (Y2)
- new net A20: BUS1.21 (Pin_21), U6.14 (Y4)
- new net A21: BUS1.22 (Pin_22), U6.13 (Y5)
- new net A22: BUS1.23 (Pin_23), U6.12 (Y6)
- new net A23: BUS1.24 (Pin_24), U6.11 (Y7)
- new net A3: BUS1.4 (Pin_4), U6.15 (Y3)
- new net A4: BUS1.5 (Pin_5), U6.14 (Y4)
- new net A5: BUS1.6 (Pin_6), U6.13 (Y5)
- new net A6: BUS1.7 (Pin_7), U6.12 (Y6)
- new net A7: BUS1.8 (Pin_8), U6.11 (Y7)
- new net A8: BUS1.9 (Pin_9), U6.18 (Y0)
- new net A9: BUS1.10 (Pin_10), U6.17 (Y1)
Other:
- note added: "RAM BANK 0 - A0..A20, A21=0, A22=0, A23=0 RAM BANK 1 - A0..A20, A21=1, A22=0, A23=0 RAM BANK 2 - A0..A20, A21=1, A22=0, A23=0 FLASH BANK 0 - A0..A18, A19=0, A20=0, A21=1, A22=1, A23=0 FLASH BANK 1 - A0..A18, A19=1, A20=0, A21=1, A22=1, A23=0 FLASH BANK 2 - A0..A18, A19=0, A20=1, A21=1, A22=1, A23=0 FLASH BANK 3 - A0..A18, A19=1, A20=1, A21=1, A22=1, A23=0"

Commit message: Update readme
Parts:
- added D1, D2, D3, D4, D5: LED, LED_SMD:LED_0805_2012Metric_Pad1.15x1.40mm_HandSolder, symbol Device:LED
- added R1, R2, R3, R4, R5: R, Resistor_SMD:R_0805_2012Metric_Pad1.20x1.40mm_HandSolder, symbol Device:R
- C99: footprint Capacitor_SMD:C_0805_2012Metric_Pad1.18x1.45mm_HandSolder -> Capacitor_SMD:C_1206_3216Metric_Pad1.33x1.80mm_HandSolder
- renumbered U10 to U1, U7 to U10, U8 to U11, U9 to U12, U11 to U2, U12 to U3, U13 to U4, U14 to U5, U15 to U6, U4 to U7, U5 to U8, U6 to U9
Connections:
- net BootAddr: now also R2.1
- net CP: now also R3.1
- net GNDD: now also D1.1 (K), D2.1 (K), D3.1 (K)
- net SEL: now also R1.1
- net VCC: now also D4.2 (A), D5.2 (A)
- net ~{OE}: now also R5.1
- net ~{PE}: now also R4.1
- new net: D5.1 (K), R5.2
- new net: D1.2 (A), R1.2
- new net: D4.1 (K), R4.2
- new net: D3.2 (A), R3.2
- new net: D2.2 (A), R2.2
