File: PCB/GPIO/GPIO.kicad_pcb (KiCad board)
At the start: 2 copper layers, 101.6 x 76.2 mm, 78 parts, among them J1 Conn_01x09_Pin, J10 Conn_01x08_Pin, J11 Conn_01x08_Pin, J12 Conn_01x16_Pin, J2 Conn_01x09_Pin, J3 Conn_01x09_Pin, J5 Conn_01x09_Pin, J6 Conn_01x09_Pin, J7 Conn_01x09_Pin, J8 Conn_01x09_Pin, J9 Conn_01x09_Pin, U1 74HC138, U10 74LS540, U11 74LS540, U12 74LS574, U13 74LS540, U14 74LS574, U15 74HC04, U16 ICL7660, U2 74HC138, U3 74LS175, U4 74LS574, U5 74LS574, U6 74LS574, U7 74LS540, U8 74LS540, U9 74LS540

Commit message: Updates ;-)
Parts:
- removed C13, C16, C18, C19, C20, C21: C, Capacitor_SMD:C_0805_2012Metric_Pad1.18x1.45mm_HandSolder
- removed D10, D11, D12, D13, D14, D15, D16, D6, D7, D8, D9: LED, LED_SMD:LED_0805_2012Metric_Pad1.15x1.40mm_HandSolder
- removed D2, D3, D4, D5: D, Diode_SMD:D_SOD-123
- removed J11: Conn_01x08_Pin, matseng:SUBLEQ_B2B
- removed J12: Conn_01x16_Pin, Connector_PinHeader_2.54mm:PinHeader_1x16_P2.54mm_Vertical
- removed JP4: SolderJumper_3_Open, Jumper:SolderJumper-3_P1.3mm_Open_Pad1.0x1.5mm
- removed R3, R4, R8: R, Resistor_SMD:R_0805_2012Metric_Pad1.20x1.40mm_HandSolder
- removed U16: ICL7660, matseng:SOIC-8_3.9x4.9mm_P1.27mm
- added J4: Conn_01x12, Connector_PinHeader_2.54mm:PinHeader_1x12_P2.54mm_Vertical, F.Cu at (41.1, 26.4)
- added R2: R, Resistor_SMD:R_0805_2012Metric_Pad1.20x1.40mm_HandSolder, F.Cu at (61.5, 43.8)
- added U17: 74LS175, Package_SO:SOIC-16_4.55x10.3mm_P1.27mm, F.Cu at (44.5, 69.8)
- J10: value Conn_01x08_Pin -> Conn_01x08; footprint matseng:SUBLEQ_B2B -> Connector_PinHeader_2.54mm:PinHeader_1x08_P2.54mm_Vertical; moved to B.Cu
- U1: value 74HC138 -> 74HC238; footprint Package_SO:SOIC-16W_5.3x10.2mm_P1.27mm -> Package_SO:SOIC-16_4.55x10.3mm_P1.27mm
- U10, U11, U13, U7, U8, U9: value 74LS540 -> 74HCT541
- U12, U4, U5, U6: value 74LS574 -> 74LS564
- U15: value 74HC04 -> TPS60403DBV; footprint Package_SO:SO-14_3.9x8.65mm_P1.27mm -> Package_TO_SOT_SMD:SOT-23-5
- U2, U3: footprint Package_SO:SOIC-16W_5.3x10.2mm_P1.27mm -> Package_SO:SOIC-16_4.55x10.3mm_P1.27mm
- moved C2 90.9 mm to (108.5, 26.2), turned to 180 degrees
- moved C3 77.7 mm to (95.1, 26.2), turned to 180 degrees
- moved C11 73.7 mm to (54.5, 46.5), turned to 180 degrees
- moved C7 68.3 mm to (95.2, 95.2)
- moved J10 65.6 mm to (128.8, 51.8), turned to 180 degrees
- moved C17 62.5 mm to (49.5, 40.6)
- moved C10 55.9 mm to (45.7, 78.9)
- moved C8 47.5 mm to (69.0, 33.8)
- moved C4 44.9 mm to (95.1, 58.4)
- moved C9 39.1 mm to (54.7, 78.9), turned to 180 degrees
- moved C6 38.6 mm to (108.5, 95.2), turned to 180 degrees
- moved J1 38.5 mm to (118.6, 27.7)
- moved J7 38.3 mm to (118.6, 65.8)
- moved U1 38.1 mm to (54.6, 53.3)
- moved C5 36.4 mm to (108.6, 58.4), turned to 180 degrees
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Connections:
- C14 pad 1: Net-(U16-VOUT) -> Net-(U15-OUT)
- C15 pad 1: Net-(U16-CAP+) -> Net-(U15-C_{FLY-})
- C15 pad 2: Net-(U16-CAP-) -> Net-(U15-C_{FLY+})
- J10 pad 1: VCC -> Ack
- J10 pad 2: unconnected-(J10-Pin_2-Pad2) -> Bck
- J10 pad 3: ~{RES} -> ~{E}
- J10 pad 4: TS1 -> ~{IOwP}
- J10 pad 5: OUT1 -> ~{IOrdP}
- J10 pad 6: OUT2 -> ~{Wr-1}
- J10 pad 7: ~{E} -> ~{Rd-2}
- J10 pad 8: GNDD -> ~{Rd-1}
- JP2 pad 3: /A3 -> Net-(JP2-B)
- JP3 pad 1: Net-(D5-K) -> VCC
- JP3 pad 2: /LCD_VCC -> Net-(JP3-C)
- JP3 pad 3: VCC -> GNDD
- R1 pad 1: GNDD -> VCC
- RV1 pad 1: VCC -> Net-(JP3-C)
- RV1 pad 3: Net-(U16-VOUT) -> Net-(U15-OUT)
- U1 pad 10: /IOR-3 -> /~{Wr-3}
- U1 pad 11: /IOR-4 -> /~{Wr-4}
- U1 pad 12: /IOR-5 -> /~{Wr-5}
- U1 pad 13: unconnected-(U1-~{Y2}-Pad13) -> /~{Wr-6}
- U1 pad 14: unconnected-(U1-~{Y1}-Pad14) -> /~{Wr-7}
- U1 pad 15: unconnected-(U1-~{Y0}-Pad15) -> /~{Wr-8}
- U1 pad 4: Net-(JP1-C) -> ~{E}
- U1 pad 5: ~{E} -> ~{IOwP}
- U1 pad 6: GPIOrd -> Net-(JP1-C)
- U1 pad 7: /IOR-1 -> ~{Wr-1}
- U1 pad 9: /IOR-2 -> /~{Wr-2}
- U10 pad 1: /IOR-2 -> /~{Rd-6}
- U10 pad 11: Net-(J7-Pin_1) -> Net-(J5-Pin_8)
- U10 pad 12: Net-(J7-Pin_2) -> Net-(J5-Pin_7)
- U10 pad 13: Net-(J7-Pin_3) -> Net-(J5-Pin_6)
- U10 pad 14: Net-(J7-Pin_4) -> Net-(J5-Pin_5)
- U10 pad 15: Net-(J7-Pin_5) -> Net-(J5-Pin_4)
- U10 pad 16: Net-(J7-Pin_6) -> Net-(J5-Pin_3)
- U10 pad 17: Net-(J7-Pin_7) -> Net-(J5-Pin_2)
- U10 pad 18: Net-(J7-Pin_8) -> Net-(J5-Pin_1)
- U10 pad 19: /IOR-2 -> /~{Rd-6}
- U10 pad 2: /D7 -> /D0
- U10 pad 3: /D6 -> /D1
- U10 pad 4: /D5 -> /D2
- U10 pad 5: /D4 -> /D3
- U10 pad 6: /D3 -> /D4
- U10 pad 7: /D2 -> /D5
- U10 pad 8: /D1 -> /D6
- U10 pad 9: /D0 -> /D7
- U11 pad 1: /IOR-3 -> /~{Rd-5}
- U11 pad 11: Net-(J5-Pin_8) -> Net-(J7-Pin_8)
- U11 pad 12: Net-(J5-Pin_7) -> Net-(J7-Pin_7)
- U11 pad 13: Net-(J5-Pin_6) -> Net-(J7-Pin_6)
- U11 pad 14: Net-(J5-Pin_5) -> Net-(J7-Pin_5)
- U11 pad 15: Net-(J5-Pin_4) -> Net-(J7-Pin_4)
- U11 pad 16: Net-(J5-Pin_3) -> Net-(J7-Pin_3)
- U11 pad 17: Net-(J5-Pin_2) -> Net-(J7-Pin_2)
- U11 pad 18: Net-(J5-Pin_1) -> Net-(J7-Pin_1)
- U11 pad 19: /IOR-3 -> /~{Rd-5}
- U12 pad 11: /IOW-3 -> /~{Wr-4}
- U13 pad 1: /IOR-5 -> /~{Rd-3}
- U13 pad 11: Net-(J9-Pin_8) -> Net-(J6-Pin_8)
- U13 pad 12: Net-(J9-Pin_7) -> Net-(J6-Pin_7)
- U13 pad 13: Net-(J9-Pin_6) -> Net-(J6-Pin_6)
- U13 pad 14: Net-(J9-Pin_5) -> Net-(J6-Pin_5)
- U13 pad 15: Net-(J9-Pin_4) -> Net-(J6-Pin_4)
- U13 pad 16: Net-(J9-Pin_3) -> Net-(J6-Pin_3)
- U13 pad 17: Net-(J9-Pin_2) -> Net-(J6-Pin_2)
- U13 pad 18: Net-(J9-Pin_1) -> Net-(J6-Pin_1)
- U13 pad 19: /IOR-5 -> /~{Rd-3}
- U14 pad 11: /IOW-6 -> /~{Wr-7}
- U15 pad 1: VCC -> Net-(U15-OUT)
- U15 pad 2: unconnected-(U15-Pad2) -> VCC
- U15 pad 3: VCC -> Net-(U15-C_{FLY-})
- U15 pad 4: unconnected-(U15-Pad4) -> GNDD
- U15 pad 5: /IOR-1 -> Net-(U15-C_{FLY+})
- U2 pad 1: /A0 -> Net-(U17-Q0)
- U2 pad 10: /IOW-3 -> /~{Rd-3}
- U2 pad 11: /IOW-4 -> /~{Rd-4}
- U2 pad 12: /IOW-5 -> /~{Rd-5}
- U2 pad 13: /IOW-6 -> /~{Rd-6}
- U2 pad 14: unconnected-(U2-~{Y1}-Pad14) -> /~{Rd-7}
- U2 pad 15: unconnected-(U2-~{Y0}-Pad15) -> /~{Rd-8}
- U2 pad 2: /A1 -> Net-(U17-Q1)
- U2 pad 3: /A2 -> Net-(U17-Q2)
- U2 pad 4: Net-(JP2-C) -> ~{E}
- U2 pad 5: ~{E} -> ~{IOrdP}
- U2 pad 6: GPIOwr -> Net-(JP2-C)
- U2 pad 7: /IOW-1 -> ~{Rd-1}
- U2 pad 9: /IOW-2 -> ~{Rd-2}
- U3 pad 1: ~{RES} -> VCC
- U3 pad 12: /A2 -> /D2
- U3 pad 13: /A3 -> /D3
- U3 pad 4: /A0 -> /D0
- U3 pad 5: /A1 -> /D1
- U3 pad 9: Net-(U3-Cp) -> Bck
- U4 pad 11: /IOW-2 -> /~{Wr-5}
- U4 pad 12: Net-(J1-Pin_1) -> Net-(J1-Pin_8)
- U4 pad 13: Net-(J1-Pin_2) -> Net-(J1-Pin_7)
- U4 pad 14: Net-(J1-Pin_3) -> Net-(J1-Pin_6)
- U4 pad 15: Net-(J1-Pin_4) -> Net-(J1-Pin_5)
- U4 pad 16: Net-(J1-Pin_5) -> Net-(J1-Pin_4)
- U4 pad 17: Net-(J1-Pin_6) -> Net-(J1-Pin_3)
- U4 pad 18: Net-(J1-Pin_7) -> Net-(J1-Pin_2)
- U4 pad 19: Net-(J1-Pin_8) -> Net-(J1-Pin_1)
- U4 pad 2: /D7 -> /D0
- U4 pad 3: /D6 -> /D1
- U4 pad 4: /D5 -> /D2
- U4 pad 5: /D4 -> /D3
- U4 pad 6: /D3 -> /D4
- U4 pad 7: /D2 -> /D5
- U4 pad 8: /D1 -> /D6
- U4 pad 9: /D0 -> /D7
- U5 pad 11: /IOW-5 -> /~{Wr-6}
- U6 pad 11: /IOW-4 -> /~{Wr-3}
- U6 pad 12: Net-(J3-Pin_1) -> Net-(J3-Pin_8)
- U6 pad 13: Net-(J3-Pin_2) -> Net-(J3-Pin_7)
- U6 pad 14: Net-(J3-Pin_3) -> Net-(J3-Pin_6)
- U6 pad 15: Net-(J3-Pin_4) -> Net-(J3-Pin_5)
- U6 pad 16: Net-(J3-Pin_5) -> Net-(J3-Pin_4)
- U6 pad 17: Net-(J3-Pin_6) -> Net-(J3-Pin_3)
- U6 pad 18: Net-(J3-Pin_7) -> Net-(J3-Pin_2)
- U6 pad 19: Net-(J3-Pin_8) -> Net-(J3-Pin_1)
- U6 pad 2: /D7 -> /D0
- U6 pad 3: /D6 -> /D1
- U6 pad 4: /D5 -> /D2
- U6 pad 5: /D4 -> /D3
- U6 pad 6: /D3 -> /D4
- U6 pad 7: /D2 -> /D5
- U6 pad 8: /D1 -> /D6
- U6 pad 9: /D0 -> /D7
- U7 pad 1: ~{DBUSFORCE} -> ~{IOrdP}
- U7 pad 11: /D8 -> /D14
- U7 pad 12: /D10 -> /D15
- U7 pad 14: /D14 -> /D13
- U7 pad 15: /D16 -> /D10
- U7 pad 16: /D18 -> /D11
- U7 pad 17: /D20 -> /D8
- U7 pad 18: /D22 -> /D9
- U7 pad 19: ~{DBUSFORCE} -> ~{IOrdP}
- U7 pad 2: Net-(JP4-C) -> GNDD
- U7 pad 3: Net-(JP4-C) -> GNDD
- U7 pad 4: Net-(JP4-C) -> GNDD
- U7 pad 5: Net-(JP4-C) -> GNDD
- U7 pad 6: Net-(JP4-C) -> GNDD
- U7 pad 7: Net-(JP4-C) -> GNDD
- U7 pad 8: Net-(JP4-C) -> GNDD
- U7 pad 9: Net-(JP4-C) -> GNDD
- U8 pad 1: ~{DBUSFORCE} -> ~{IOrdP}
- U8 pad 11: /D9 -> /D22
- U8 pad 12: /D11 -> /D23
- U8 pad 13: /D13 -> /D20
- U8 pad 14: /D15 -> /D21
- U8 pad 15: /D17 -> /D18
- U8 pad 17: /D21 -> /D16
- U8 pad 18: /D23 -> /D17
- U8 pad 19: ~{DBUSFORCE} -> ~{IOrdP}
- U8 pad 2: Net-(JP4-C) -> GNDD
- U8 pad 3: Net-(JP4-C) -> GNDD
- U8 pad 4: Net-(JP4-C) -> GNDD
- U8 pad 5: Net-(JP4-C) -> GNDD
- U8 pad 6: Net-(JP4-C) -> GNDD
- U8 pad 7: Net-(JP4-C) -> GNDD
- U8 pad 8: Net-(JP4-C) -> GNDD
- U8 pad 9: ~{D23FORCE} -> GNDD
- U9 pad 1: /IOR-4 -> /~{Rd-4}
- U9 pad 11: Net-(J6-Pin_1) -> Net-(J9-Pin_8)
- U9 pad 12: Net-(J6-Pin_2) -> Net-(J9-Pin_7)
- U9 pad 13: Net-(J6-Pin_3) -> Net-(J9-Pin_6)
- U9 pad 14: Net-(J6-Pin_4) -> Net-(J9-Pin_5)
- U9 pad 15: Net-(J6-Pin_5) -> Net-(J9-Pin_4)
- U9 pad 16: Net-(J6-Pin_6) -> Net-(J9-Pin_3)
- U9 pad 17: Net-(J6-Pin_7) -> Net-(J9-Pin_2)
- U9 pad 18: Net-(J6-Pin_8) -> Net-(J9-Pin_1)
- U9 pad 19: /IOR-4 -> /~{Rd-4}
- U9 pad 2: /D7 -> /D0
- U9 pad 3: /D6 -> /D1
- U9 pad 4: /D5 -> /D2
- U9 pad 5: /D4 -> /D3
- U9 pad 6: /D3 -> /D4
- U9 pad 7: /D2 -> /D5
- U9 pad 8: /D1 -> /D6
- U9 pad 9: /D0 -> /D7
Routing:
- net Ack: track 0.00 -> 171.4 mm, vias 0 -> 6
- net Bck: track 0.00 -> 155.4 mm, vias 0 -> 4
- net ~{Wr-1}: track 0.00 -> 146.1 mm, vias 0 -> 2
- net ~{IOrdP}: track 0.00 -> 127.7 mm, vias 0 -> 4
- net ~{Rd-1}: track 0.00 -> 125.7 mm
- net /IOW-5: track 120.7 -> 0.00 mm, vias 8 -> 0
- net ~{Rd-2}: track 0.00 -> 119.9 mm
- net /IOR-4: track 117.0 -> 0.00 mm, vias 2 -> 0
- net /~{Rd-6}: track 0.00 -> 95.0 mm, vias 0 -> 4
- net ~{IOwP}: track 0.00 -> 91.1 mm, vias 0 -> 2
- net /~{Wr-6}: track 0.00 -> 89.1 mm, vias 0 -> 2
- net /IOW-2: track 86.1 -> 0.00 mm, vias 6 -> 0
- net /IOW-6: track 83.3 -> 0.00 mm, vias 6 -> 0
- net /IOW-4: track 82.4 -> 0.00 mm, vias 4 -> 0
- net ~{E}: track 75.0 -> 151.2 mm, vias 5 -> 6
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Other:
- board text added: "+"
- board text added: "-"
- board text added: "-3"
- board text added: "-4"
- board text added: "-5"
- board text added: "-6"
- board text added: "138"
- board text added: "175"
- board text added: "238"
- board text added: "541"
- board text added: "564"
- board text added: "Out1"
- board text added: "Out2"
- board text added: "aCk"
- board text added: "bCk"
- board text added: "locked"
- board text added: "~{E}"
- board text added: "~{Rd1}"
- board text added: "~{Rd2}"
- board text added: "~{Wr1}"
- board text added: "~{rP}"
- board text added: "~{wP}"
- board text removed: "Rd 1 2 3 4 5"
- board text removed: "Wr 1 2 3 4 5 6"
- board text removed: "• SUBLEQ24 • GPIO • December 2023 • github.com/mengstr •"
