File: PCB/GPIO/GPIO.kicad_sch (KiCad schematic)
At the start: 78 parts, among them J1 Conn_01x09_Pin, J12 Conn_01x16_Pin, J2 Conn_01x09_Pin, J3 Conn_01x09_Pin, J4 Conn_01x08_Pin, J5 Conn_01x09_Pin, J6 Conn_01x09_Pin, J7 Conn_01x09_Pin, J8 Conn_01x09_Pin, J9 Conn_01x09_Pin, U1 74HC138, U10 74LS540, U11 74LS540, U12 74LS574, U13 74LS540, U14 74LS574, U15 74HC04, U16 ICL7660, U2 74HC138, U3 74LS175, U4 74LS574, U5 74LS574, U6 74LS574, U7 74LS540, U8 74LS540, U9 74LS540

Commit message: Updates ;-)
Parts:
- removed C1 (x2), C8 (x4): C, Capacitor_SMD:C_0805_2012Metric_Pad1.18x1.45mm_HandSolder, symbol Device:C
- removed D2, D3, D4, D5: D, Diode_SMD:D_SOD-123, symbol Device:D
- removed D25 (x11): LED, LED_SMD:LED_0805_2012Metric_Pad1.15x1.40mm_HandSolder, symbol Device:LED
- removed J12: Conn_01x16_Pin, Connector_PinHeader_2.54mm:PinHeader_1x16_P2.54mm_Vertical, symbol Connector:Conn_01x16_Pin
- removed J4 (x2): Conn_01x08_Pin, matseng:SUBLEQ_B2B, symbol Connector:Conn_01x08_Pin
- removed JP4: SolderJumper_3_Open, Jumper:SolderJumper-3_P1.3mm_Open_Pad1.0x1.5mm, symbol Jumper:SolderJumper_3_Open
- removed R1 (x3): R, Resistor_SMD:R_0805_2012Metric_Pad1.20x1.40mm_HandSolder, symbol Device:R
- removed U1: 74HC138, Package_SO:SOIC-16W_5.3x10.2mm_P1.27mm, symbol 74xx:74HC138
- removed U10, U11, U13, U7, U8, U9: 74LS540, Package_SO:SOIC-20W_7.5x12.8mm_P1.27mm, symbol 74xx:74LS540
- removed U15: 74HC04, Package_SO:SO-14_3.9x8.65mm_P1.27mm, symbol 74xx:74HC04
- removed U16: ICL7660, matseng:SOIC-8_3.9x4.9mm_P1.27mm, symbol Regulator_SwitchedCapacitor:ICL7660
- added J10: Conn_01x08, Connector_PinHeader_2.54mm:PinHeader_1x08_P2.54mm_Vertical, symbol Connector_Generic:Conn_01x08
- added J4: Conn_01x12, Connector_PinHeader_2.54mm:PinHeader_1x12_P2.54mm_Vertical, symbol Connector_Generic:Conn_01x12
- added R2: R, Resistor_SMD:R_0805_2012Metric_Pad1.20x1.40mm_HandSolder, symbol Device:R
- added U1: 74HC238, Package_SO:SOIC-16_4.55x10.3mm_P1.27mm, symbol 74xx:74HC238
- added U10, U11, U13, U7, U8, U9: 74HCT541, Package_SO:SOIC-20W_7.5x12.8mm_P1.27mm, symbol 74xx:74HCT541
- added U15: TPS60403DBV, Package_TO_SOT_SMD:SOT-23-5, symbol Regulator_SwitchedCapacitor:TPS60403DBV
- added U17: 74LS175, Package_SO:SOIC-16_4.55x10.3mm_P1.27mm, symbol 74xx:74LS175
- C96: footprint Capacitor_SMD:C_0805_2012Metric_Pad1.18x1.45mm_HandSolder -> Capacitor_SMD:C_1206_3216Metric_Pad1.33x1.80mm_HandSolder
- U12, U4, U5, U6: value 74LS574 -> 74LS564
- U2, U3: footprint Package_SO:SOIC-16W_5.3x10.2mm_P1.27mm -> Package_SO:SOIC-16_4.55x10.3mm_P1.27mm
Connections:
- net GPIOwr is gone; now on an unnamed net: U2.6 (E2)
- net ~{RES} is gone; now on net VCC: U3.1 (~{Mr})
- net A0: no longer U2.1 (A0), U3.4 (D0)
- net A1: no longer U2.2 (A1), U3.5 (D1)
- net A2: no longer U2.3 (A2), U3.12 (D2)
- net A3: no longer JP2.3 (B), U3.13 (D3)
- net D0: now also U3.4 (D0), U4.2 (D0), U6.2 (D0), U10.2 (A0), U11.2 (A0), U13.2 (A0), U17.4 (D0), U9.2 (A0); no longer U4.9 (D7), U6.9 (D7)
- net D1: now also U3.5 (D1), U4.3 (D1), U6.3 (D1), U10.3 (A1), U11.3 (A1), U13.3 (A1), U17.5 (D1), U9.3 (A1); no longer U4.8 (D6), U6.8 (D6)
- net D10: now also U7.15 (Y3)
- net D11: now also U7.16 (Y2)
- net D12: now also U7.13 (Y5)
- net D13: now also U7.14 (Y4)
- net D14: now also U7.11 (Y7)
- net D15: now also U7.12 (Y6)
- net D16: now also U8.17 (Y1)
- net D17: now also U8.18 (Y0)
- net D18: now also U8.15 (Y3)
- net D19: now also U8.16 (Y2)
- net D2: now also U3.12 (D2), U4.4 (D2), U6.4 (D2), U10.4 (A2), U11.4 (A2), U13.4 (A2), U17.12 (D2), U9.4 (A2); no longer U4.7 (D5), U6.7 (D5)
- net D20: now also U8.13 (Y5)
- net D21: now also U8.14 (Y4)
- net D22: now also U8.11 (Y7)
- net D23: now also U8.12 (Y6)
- net D3: now also U3.13 (D3), U4.5 (D3), U6.5 (D3), U10.5 (A3), U11.5 (A3), U13.5 (A3), U17.13 (D3), U9.5 (A3); no longer U4.6 (D4), U6.6 (D4)
- net D4: now also U4.6 (D4), U6.6 (D4), U10.6 (A4), U11.6 (A4), U13.6 (A4), U9.6 (A4); no longer U4.5 (D3), U6.5 (D3)
- net D5: now also U4.7 (D5), U6.7 (D5), U10.7 (A5), U11.7 (A5), U13.7 (A5), U9.7 (A5); no longer U4.4 (D2), U6.4 (D2)
- net D6: now also U4.8 (D6), U6.8 (D6), U10.8 (A6), U11.8 (A6), U13.8 (A6), U9.8 (A6); no longer U4.3 (D1), U6.3 (D1)
- net D7: now also U4.9 (D7), U6.9 (D7), U10.9 (A7), U11.9 (A7), U13.9 (A7), U9.9 (A7); no longer U4.2 (D0), U6.2 (D0)
- net D8: now also U7.17 (Y1)
- net D9: now also U7.18 (Y0)
- net GNDD: now also JP3.3 (B), J4.1 (Pin_1), J4.12 (Pin_12), J4.5 (Pin_5), R2.1, U1.8 (GND), U10.10 (GND), U11.10 (GND), U13.10 (GND), U15.4 (GND), U17.8 (GND), U7.10 (GND), U7.2 (A0), U7.3 (A1), U7.4 (A2), U7.5 (A3), U7.6 (A4), U7.7 (A5), U7.8 (A6), U7.9 (A7), U8.10 (GND), U8.2 (A0), U8.3 (A1), U8.4 (A2), U8.5 (A3), U8.6 (A4), U8.7 (A5), U8.8 (A6), U8.9 (A7), U9.10 (GND); no longer R1.1
- net VCC: now also JP3.1 (A), R1.1, J4.2 (Pin_2), U1.16 (VCC), U10.20 (VCC), U11.20 (VCC), U13.20 (VCC), U15.2 (IN), U17.1 (~{Mr}), U17.16 (VCC), U7.20 (VCC), U8.20 (VCC), U9.20 (VCC); no longer JP3.3 (B), RV1.1
- net VEE: now also J4.3 (Pin_3)
- net ~{E}: now also U2.4 (~{E0}), J10.3 (Pin_3), R2.2, U1.4 (~{E1}); no longer U2.5 (~{E1})
- net at C1.1, RV1.3: now also U15.1 (OUT)
- net at J9.8 (Pin_8): now also U9.11 (Y7)
- net at J9.7 (Pin_7): now also U9.12 (Y6)
- net at J9.6 (Pin_6): now also U9.13 (Y5)
- net at J9.5 (Pin_5): now also U9.14 (Y4)
- net at J9.4 (Pin_4): now also U9.15 (Y3)
- net at J9.3 (Pin_3): now also U9.16 (Y2)
- net at J9.2 (Pin_2): now also U9.17 (Y1)
- net at J9.1 (Pin_1): now also U9.18 (Y0)
- net at J5.1 (Pin_1): now also U10.18 (Y0)
- net at J5.2 (Pin_2): now also U10.17 (Y1)
- net at J5.3 (Pin_3): now also U10.16 (Y2)
- net at J5.4 (Pin_4): now also U10.15 (Y3)
- net at J5.5 (Pin_5): now also U10.14 (Y4)
- net at J5.6 (Pin_6): now also U10.13 (Y5)
- net at J5.7 (Pin_7): now also U10.12 (Y6)
- net at J5.8 (Pin_8): now also U10.11 (Y7)
- net at JP2.1 (A): now also U17.14 (~{Q3})
- net at U14.19 (Q0): now also J4.7 (Pin_7)
- net at U14.18 (Q1): now also J4.8 (Pin_8)
- net at U14.17 (Q2): now also J4.9 (Pin_9)
- net at U14.16 (Q3): now also J4.10 (Pin_10)
- net at R1.2: now also J4.11 (Pin_11)
- net at U14.14 (Q5): now also J4.4 (Pin_4)
- net at U14.15 (Q4): now also J4.6 (Pin_6)
- net at J1.1 (Pin_1): now also U4.19 (Q0); no longer U4.12 (Q7)
- net at J1.2 (Pin_2): now also U4.18 (Q1); no longer U4.13 (Q6)
- net at J1.3 (Pin_3): now also U4.17 (Q2); no longer U4.14 (Q5)
- net at J1.4 (Pin_4): now also U4.16 (Q3); no longer U4.15 (Q4)
- net at J1.5 (Pin_5): now also U4.15 (Q4); no longer U4.16 (Q3)
- net at J1.6 (Pin_6): now also U4.14 (Q5); no longer U4.17 (Q2)
- net at J1.7 (Pin_7): now also U4.13 (Q6); no longer U4.18 (Q1)
- net at J1.8 (Pin_8): now also U4.12 (Q7); no longer U4.19 (Q0)
- net Bck: now reaches U3.9 (Cp)
- net Bck: now also J10.2 (Pin_2)
- net at J6.1 (Pin_1): now also U13.18 (Y0)
- net at J6.2 (Pin_2): now also U13.17 (Y1)
- net at J6.3 (Pin_3): now also U13.16 (Y2)
- net at J6.4 (Pin_4): now also U13.15 (Y3)
- net at J6.5 (Pin_5): now also U13.14 (Y4)
- net at J6.6 (Pin_6): now also U13.13 (Y5)
- net at J6.7 (Pin_7): now also U13.12 (Y6)
- net at J6.8 (Pin_8): now also U13.11 (Y7)
- net at JP1.2 (C): now also U1.6 (E3)
- net at U3.10 (Q2): now also U1.3 (A2)
- net at U3.2 (Q0): now also U1.1 (A0)
- net at U3.7 (Q1): now also U1.2 (A1)
- net at J3.1 (Pin_1): now also U6.19 (Q0); no longer U6.12 (Q7)
- net at J3.2 (Pin_2): now also U6.18 (Q1); no longer U6.13 (Q6)
- net at J3.3 (Pin_3): now also U6.17 (Q2); no longer U6.14 (Q5)
- net at J3.4 (Pin_4): now also U6.16 (Q3); no longer U6.15 (Q4)
- net at J3.5 (Pin_5): now also U6.15 (Q4); no longer U6.16 (Q3)
- net at J3.6 (Pin_6): now also U6.14 (Q5); no longer U6.17 (Q2)
- net at J3.7 (Pin_7): now also U6.13 (Q6); no longer U6.18 (Q1)
- net at J3.8 (Pin_8): now also U6.12 (Q7); no longer U6.19 (Q0)
- net at C1.1: now also U15.3 (C_{FLY-})
- net at C1.2: now also U15.5 (C_{FLY+})
- net at J7.1 (Pin_1): now also U11.18 (Y0)
- net at J7.2 (Pin_2): now also U11.17 (Y1)
- net at J7.3 (Pin_3): now also U11.16 (Y2)
- net at J7.4 (Pin_4): now also U11.15 (Y3)
- net at J7.5 (Pin_5): now also U11.14 (Y4)
- net at J7.6 (Pin_6): now also U11.13 (Y5)
- net at J7.7 (Pin_7): now also U11.12 (Y6)
- net at J7.8 (Pin_8): now also U11.11 (Y7)
- net at JP2.2 (C): no longer U2.4 (~{E0})
- net ~{Rd-7}: now reaches U2.14 (~{Y1})
- net ~{Rd-8}: now reaches U2.15 (~{Y0})
- net IOW-1 renamed ~{Rd-1}
- net ~{Rd-1}: now also J10.8 (Pin_8)
- net IOW-2 renamed ~{Rd-2}
- net ~{Rd-2}: now also J10.7 (Pin_7); no longer U4.11 (Cp)
- net IOW-3 renamed ~{Rd-3}
- net ~{Rd-3}: now also U13.1 (G1), U13.19 (G2); no longer U12.11 (Cp)
- net IOW-4 renamed ~{Rd-4}
- net ~{Rd-4}: now also U9.1 (G1), U9.19 (G2); no longer U6.11 (Cp)
- net IOW-5 renamed ~{Rd-5}
- net ~{Rd-5}: now also U11.1 (G1), U11.19 (G2); no longer U5.11 (Cp)
- net IOW-6 renamed ~{Rd-6}
- net ~{Rd-6}: now also U10.1 (G1), U10.19 (G2); no longer U14.11 (Cp)
- net LCD_VCC: no longer names the net of JP3.2 (C)
- net LCD_VCC: now also RV1.1
- new net: U17.10 (Q2), U2.3 (A2)
- new net: JP2.3 (B), U17.15 (Q3)
- new net: U17.2 (Q0), U2.1 (A0)
- new net: U17.7 (Q1), U2.2 (A1)
- new net Ack: J10.1 (Pin_1), U17.9 (Cp)
- new net ~{IOrdP}: J10.5 (Pin_5), U2.5 (~{E1}), U7.1 (G1), U7.19 (G2), U8.1 (G1), U8.19 (G2)
- new net ~{IOwP}: J10.4 (Pin_4), U1.5 (~{E2})
- new net ~{Wr-1}: J10.6 (Pin_6), U1.7 (Y7)
- new net ~{Wr-2}: U1.9 (Y6)
- new net ~{Wr-3}: U1.10 (Y5), U6.11 (Cp)
- new net ~{Wr-4}: U1.11 (Y4), U12.11 (Cp)
- new net ~{Wr-5}: U1.12 (Y3), U4.11 (Cp)
- new net ~{Wr-6}: U1.13 (Y2), U5.11 (Cp)
- new net ~{Wr-7}: U1.14 (Y1), U14.11 (Cp)
- new net ~{Wr-8}: U1.15 (Y0)
- no-connect marks 15 -> 0
Other:
- moved on the sheet: C1, C96, C97, D97, J1, J2, J3, J5, J6, J7, J8, J9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
