File: PCB/MopSequencer/MopSequencer.kicad_sch (KiCad schematic)
At the start: 132 parts, among them J1 Conn_01x24_Pin, J2 Conn_01x06, J3 Conn_01x06, J4 Conn_01x06, J5 Conn_01x02_Pin, J6 Conn_01x02_Pin, J7 Conn_01x06, J8 Conn_01x24_Pin, J9 Conn_01x08_Pin, U1 74HC238, U2 74HC00, U3 74HCT574

Commit message: Update readme
Changed lines of the file:
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@@
-    (stroke (width 0) (type default))
-  )
-  (wire (pts (xy 88.9 54.61) (xy 96.52 54.61))
     (stroke (width 0) (type default))
   )
@@
     (stroke (width 0) (type default))
   )
-  (wire (pts (xy 88.9 52.07) (xy 96.52 52.07))
-    (stroke (width 0) (type default))
-  )

Commit message: Updates ;-)
Parts:
- added U4: 74LS365, Package_SO:SOIC-16W_5.3x10.2mm_P1.27mm, symbol 74xx:74LS365
- added U5: 74LS365, Package_SO:SOIC-16W_7.5x10.3mm_P1.27mm, symbol 74xx:74LS365
- added U6: 74LS365, Package_SO:SOIC-16W_7.5x12.8mm_P1.27mm, symbol 74xx:74LS365
Changed lines of the file:
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@@
     )
   )
+  (symbol (lib_id "74xx:74LS365") (at 262.89 228.6 0) (unit 1)
+    (in_bom yes) (on_board yes) (dnp no) (fields_autoplaced)
+    (property "Reference" "U6" (at 265.0841 210.82 0)
+      (effects (font (size 1.27 1.27)) (justify left))
+    )
+    (property "Value" "74LS365" (at 265.0841 213.36 0)
+      (effects (font (size 1.27 1.27)) (justify left))
+    )
+    (property "Footprint" "Package_SO:SOIC-16W_7.5x12.8mm_P1.27mm" (at 262.89 228.6 0)
+      (effects (font (size 1.27 1.27)) hide)
+    )
+    (property "Datasheet" "http://www.ti.com/lit/gpn/sn74LS365" (at 262.89 228.6 0)
+      (effects (font (size 1.27 1.27)) hide)
+    )
+    (pin "12")
+    (pin "14")
+    (pin "15")
+    (pin "13")
+    (pin "1")
+    (pin "11")
+    (pin "7")
+    (pin "8")
+    (pin "5")
+    (pin "6")
+    (pin "3")
+    (pin "4")
+    (pin "10")
+    (pin "9")
+    (pin "16")
+    (pin "2")
+    (instances
+      (project "MopSequencer"
+        (path "/aed6eade-53fd-4193-8c3b-efdb5650d6ce"
+          (reference "U6") (unit 1)
+        )
+      )
+    )
+  )
   (symbol (lib_id "Device:LED") (at 41.91 121.92 0) (unit 1)
     (in_bom yes) (on_board yes) (dnp no)
@@
     )
   )
+  (symbol (lib_id "74xx:74LS365") (at 247.65 138.43 0) (unit 1)
+    (in_bom yes) (on_board yes) (dnp no) (fields_autoplaced)
+    (property "Reference" "U4" (at 249.8441 120.65 0)
+      (effects (font (size 1.27 1.27)) (justify left))
+    )
+    (property "Value" "74LS365" (at 249.8441 123.19 0)
+      (effects (font (size 1.27 1.27)) (justify left))
+    )
+    (property "Footprint" "Package_SO:SOIC-16W_5.3x10.2mm_P1.27mm" (at 247.65 138.43 0)
+      (effects (font (size 1.27 1.27)) hide)
+    )
+    (property "Datasheet" "http://www.ti.com/lit/gpn/sn74LS365" (at 247.65 138.43 0)
+      (effects (font (size 1.27 1.27)) hide)
+    )
+    (pin "12")
+    (pin "14")
+    (pin "15")
+    (pin "13")
+    (pin "1")
+    (pin "11")
+    (pin "7")
+    (pin "8")
+    (pin "5")
+    (pin "6")
+    (pin "3")
+    (pin "4")
+    (pin "10")
+    (pin "9")
+    (pin "16")
+    (pin "2")
+    (instances
+      (project "MopSequencer"
+        (path "/aed6eade-53fd-4193-8c3b-efdb5650d6ce"
+          (reference "U4") (unit 1)
+        )
+      )
+    )
+  )
   (symbol (lib_id "Device:LED") (at 41.91 144.78 0) (unit 1)
     (in_bom yes) (on_board yes) (dnp no)
@@
         )
       )
+    )
+  )
+  (symbol (lib_id "74xx:74LS365") (at 260.35 177.8 0) (unit 1)
+    (in_bom yes) (on_board yes) (dnp no) (fields_autoplaced)
+    (property "Reference" "U5" (at 262.5441 160.02 0)
+      (effects (font (size 1.27 1.27)) (justify left))
+    )
+    (property "Value" "74LS365" (at 262.5441 162.56 0)
+      (effects (font (size 1.27 1.27)) (justify left))
+    )
+    (property "Footprint" "Package_SO:SOIC-16W_7.5x10.3mm_P1.27mm" (at 260.35 177.8 0)
+      (effects (font (size 1.27 1.27)) hide)
+    )
+    (property "Datasheet" "http://www.ti.com/lit/gpn/sn74LS365" (at 260.35 177.8 0)
+      (effects (font (size 1.27 1.27)) hide)
+    )
+    (pin "12")
+    (pin "14")
+    (pin "15")
+    (pin "13")
+    (pin "1")
+    (pin "11")
+    (pin "7")
+    (pin "8")
+    (pin "5")
+    (pin "6")
+    (pin "3")
+    (pin "4")
+    (pin "10")
+    (pin "9")
+    (pin "16")
+    (pin "2")
+    (instances
+      (project "MopSequencer"
+        (path "/aed6eade-53fd-4193-8c3b-efdb5650d6ce"
+          (reference "U5") (unit 1)
+        )
+      )
