File: PCB/MopSequencer/MopSequencer.kicad_pcb (KiCad board)
At the start: 2 copper layers, 101.6 x 76.2 mm, 490 parts, among them J1 Conn_01x24_Pin, J6 Conn_01x02_Pin, J8 Conn_01x24_Pin, J9 Conn_01x08_Pin, U1 74HC238, U2 74HC00, U3 74HCT574

Commit message: Update readme
Parts:
- C99: footprint Capacitor_SMD:C_0805_2012Metric_Pad1.18x1.45mm_HandSolder -> Capacitor_SMD:C_1206_3216Metric_Pad1.33x1.80mm_HandSolder
Routing:
- net VCC: track 238.2 -> 243.5 mm
Other:
- outline, holes or cut-outs redrawn
- board text added: "CK"
- board text added: "E3"
- board text added: "OE"
- board text added: "Q2 Q1 Q0 Tick Dis"
- board text added: "~{E1}"
- board text removed: "Q2 Q1 Q0 Tick !Reset"
- board text removed: "ck"
- board text removed: "oe"

Commit message: Misc updstes
Routing:
- net Net-(D6-A): track 0.00 -> 4.92 mm, vias 0 -> 1
- net Net-(D6-K): track 15.0 -> 17.6 mm
Other:
- board text added: "• MOP Sequencer Proto • github.com/mengstr/SUBLEQ24 • rev2 •"
- board text removed: "• MOP Sequencer Proto • github.com/mengstr/SUBLEQ24 • rev1 •"
Changed lines of the file:
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@@
     )
   )
-  (gr_text "• MOP Sequencer Proto • github.com/mengstr/SUBLEQ24 • rev1 •" (at 74.93 98.933) (layer "F.SilkS")
+  (gr_text "• MOP Sequencer Proto • github.com/mengstr/SUBLEQ24 • rev2 •" (at 74.93 98.933) (layer "F.SilkS")
     (effects (font (face "Futura") (size 1.4 1.4) (thickness 0.15)))
-    (render_cache "• MOP Sequencer Proto • github.com/mengstr/SUBLEQ24 • rev1 •" 0
+    (render_cache "• MOP Sequencer Proto • github.com/mengstr/SUBLEQ24 • rev2 •" 0
       (polygon
         (pts
@@
       (polygon
         (pts
-          (xy 103.24058 98.244718)          (xy 102.98515 98.244718)          (xy 103.107565 98.025877)          (xy 103.460789 98.025877)
-          (xy 103.460789 99.524942)          (xy 103.24058 99.524942)
+          (xy 103.216986 99.295158)          (xy 103.767167 99.295158)          (xy 103.767167 99.514)          (xy 102.774857 99.514)
+          (xy 103.287767 98.886882)          (xy 103.297117 98.875309)          (xy 103.306275 98.863929)          (xy 103.31524 98.852741)
+          (xy 103.324013 98.841745)          (xy 103.332593 98.830942)          (xy 103.345104 98.815098)          (xy 103.357181 98.799687)
+          (xy 103.368826 98.784708)          (xy 103.380038 98.770162)          (xy 103.390817 98.756049)          (xy 103.401163 98.742369)
+          (xy 103.411077 98.729122)          (xy 103.414285 98.724802)          (xy 103.423689 98.71211)          (xy 103.432666 98.69981)
+          (xy 103.441216 98.6879)          (xy 103.449339 98.67638)          (xy 103.459507 98.661629)          (xy 103.468915 98.647572)
+          (xy 103.477565 98.634209)          (xy 103.485457 98.621541)          (xy 103.492589 98.609568)          (xy 103.502306 98.592737)
+          (xy 103.511066 98.576225)          (xy 103.518871 98.560031)          (xy 103.52572 98.544156)          (xy 103.531614 98.5286)
+          (xy 103.536551 98.513362)          (xy 103.540533 98.498442)          (xy 103.54356 98.483841)          (xy 103.54563 98.469559)
+          (xy 103.546745 98.455595)          (xy 103.546958 98.446463)          (xy 103.546318 98.427206)          (xy 103.544397 98.408544)
+          (xy 103.541197 98.390477)          (xy 103.536716 98.373005)          (xy 103.530954 98.356128)          (xy 103.523913 98.339846)
+          (xy 103.515591 98.324159)          (xy 103.505989 98.309067)          (xy 103.495107 98.29457)          (xy 103.482944 98.280669)
+          (xy 103.474125 98.271732)          (xy 103.460229 98.259082)          (xy 103.445726 98.247677)          (xy 103.430616 98.237516)
+          (xy 103.414899 98.228599)          (xy 103.398575 98.220926)          (xy 103.381644 98.214498)          (xy 103.364106 98.209314)
+          (xy 103.345961 98.205374)          (xy 103.327209 98.202678)          (xy 103.30785 98.201226)          (xy 103.294606 98.20095)
+          (xy 103.280795 98.20121)          (xy 103.254292 98.203288)          (xy 103.229282 98.207445)          (xy 103.205765 98.21368)
+          (xy 103.183742 98.221993)          (xy 103.163213 98.232385)          (xy 103.144176 98.244855)          (xy 103.126633 98.259404)
+          (xy 103.110583 98.27603)          (xy 103.096027 98.294736)          (xy 103.082964 98.315519)          (xy 103.071394 98.338381)
+          (xy 103.061317 98.363321)          (xy 103.056839 98.376571)          (xy 103.052734 98.39034)          (xy 103.049002 98.404629)
+          (xy 103.045644 98.419437)          (xy 103.042659 98.434765)          (xy 103.040047 98.450612)          (xy 103.037809 98.466979)
+          (xy 102.81589 98.466979)          (xy 102.819603 98.438663)          (xy 102.82403 98.411246)          (xy 102.829172 98.384727)
+          (xy 102.835028 98.359108)          (xy 102.841599 98.334387)          (xy 102.848885 98.310566)          (xy 102.856885 98.287643)
+          (xy 102.8656 98.265619)          (xy 102.875029 98.244495)          (xy 102.885173 98.224269)          (xy 102.896032 98.204942)
+          (xy 102.907605 98.186514)          (xy 102.919893 98.168985)          (xy 102.932895 98.152354)          (xy 102.946612 98.136623)
+          (xy 102.961044 98.121791)          (xy 102.97619 98.107857)          (xy 102.992051 98.094823)          (xy 103.008626 98.082687)
+          (xy 103.025916 98.071451)          (xy 103.043921 98.061113)          (xy 103.06264 98.051674)          (xy 103.082074 98.043135)
+          (xy 103.102222 98.035494)          (xy 103.123085 98.028752)          (xy 103.144663 98.022909)          (xy 103.166955 98.017965)
+          (xy 103.189962 98.013919)          (xy 103.213683 98.010773)          (xy 103.238119 98.008526)          (xy 103.26327 98.007178)
+          (xy 103.289135 98.006728)          (xy 103.314185 98.007228)          (xy 103.338727 98.008726)          (xy 103.362762 98.011224)
+          (xy 103.386289 98.014721)          (xy 103.409308 98.019217)          (xy 103.43182 98.024712)          (xy 103.453825 98.031206)
+          (xy 103.475321 98.038699)          (xy 103.496311 98.047192)          (xy 103.516792 98.056683)          (xy 103.536766 98.067174)
+          (xy 103.556233 98.078664)          (xy 103.575192 98.091152)          (xy 103.593643 98.10464)          (xy 103.611587 98.119127)
+          (xy 103.629023 98.134614)          (xy 103.645752 98.150837)          (xy 103.661401 98.167536)          (xy 103.675971 98.18471)
+          (xy 103.689461 98.20236)          (xy 103.701873 98.220486)          (xy 103.713205 98.239087)          (xy 103.723458 98.258163)
+          (xy 103.732631 98.277715)          (xy 103.740726 98.297743)          (xy 103.747741 98.318246)          (xy 103.753676 98.339225)
+          (xy 103.758533 98.360679)          (xy 103.76231 98.382608)          (xy 103.765009 98.405013)          (xy 103.766627 98.427894)
+          (xy 103.767167 98.45125)          (xy 103.766915 98.466234)          (xy 103.766157 98.48118)          (xy 103.764895 98.49609)
+          (xy 103.763128 98.510961)          (xy 103.760856 98.525796)          (xy 103.758079 98.540593)          (xy 103.754797 98.555352)
+          (xy 103.75101 98.570074)          (xy 103.746719 98.584759)          (xy 103.741922 98.599406)          (xy 103.736621 98.614016)
+          (xy 103.730815 98.628589)          (xy 103.724503 98.643124)          (xy 103.717687 98.657621)          (xy 103.710366 98.672082)
+          (xy 103.70254 98.686505)          (xy 103.693939 98.701978)          (xy 103.686856 98.714031)          (xy 103.679232 98.726469)
+          (xy 103.671068 98.739292)          (xy 103.662362 98.752499)          (xy 103.653116 98.766091)          (xy 103.643329 98.780068)
+          (xy 103.633 98.79443)          (xy 103.622131 98.809176)          (xy 103.610721 98.824307)          (xy 103.606797 98.829436)
+          (xy 103.594709 98.845152)          (xy 103.582037 98.861396)          (xy 103.573266 98.87252)          (xy 103.564235 98.883879)
+          (xy 103.554945 98.895473)          (xy 103.545396 98.907302)          (xy 103.535588 98.919366)          (xy 103.525521 98.931665)
+          (xy 103.515195 98.944199)          (xy 103.504609 98.956969)          (xy 103.493765 98.969973)          (xy 103.482661 98.983212)
+          (xy 103.471298 98.996687)          (xy 103.459676 99.010397)          (xy 103.447795 99.024341)
         )
       )
@@
   (segment (start 32.897981 44.45) (end 34.167981 45.72) (width 0.127) (layer "F.Cu") (net 32))
   (segment (start 27.94 45.72) (end 29.21 44.45) (width 0.127) (layer "F.Cu") (net 32))
+  (segment (start 30.471 45.72) (end 27.94 45.72) (width 0.127) (layer "F.Cu") (net 32))
   (segment (start 29.21 44.45) (end 32.897981 44.45) (width 0.127) (layer "F.Cu") (net 32))
+  (segment (start 32.521 45.729) (end 33.655 46.863) (width 0.127) (layer "F.Cu") (net 33))
+  (segment (start 32.521 45.72) (end 32.521 45.729) (width 0.127) (layer "F.Cu") (net 33))
+  (via (at 33.655 46.863) (size 0.6) (drill 0.3) (layers "F.Cu" "B.Cu") (net 33))
+  (segment (start 33.528 45.847) (end 34.433 45.847) (width 0.127) (layer "B.Cu") (net 33))
+  (segment (start 33.528 45.847) (end 32.623 45.847) (width 0.127) (layer "B.Cu") (net 33))
+  (segment (start 33.655 45.847) (end 33.528 45.847) (width 0.127) (layer "B.Cu") (net 33))
+  (segment (start 32.623 45.847) (end 32.496 45.72) (width 0.127) (layer "B.Cu") (net 33))
+  (segment (start 33.655 46.863) (end 33.655 45.847) (width 0.127) (layer "B.Cu") (net 33))
+  (segment (start 34.433 45.847) (end 34.56 45.72) (width 0.127) (layer "B.Cu") (net 33))
   (segment (start 29.21 46.99) (end 32.897981 46.99) (width 0.127) (layer "F.Cu") (net 34))
   (segment (start 32.897981 46.99) (end 34.167981 48.26) (width 0.127) (layer "F.Cu") (net 34))
