File: PCB/Controlpanel/ControlPanel.kicad_pcb (KiCad board)
At the start: 2 copper layers, 101.6 x 76.2 mm, 79 parts, among them J1 Conn_01x03, J2 USB4105-GF-A, J3 Conn_02x05_Counter_Clockwise, J4 Conn_01x10_Pin, SW1 SW_Push, SW2 SW_Push, SW3 SW_Push, SW4 SW_Push, SW5 SW_Push, SW6 SW_Push, U1 74HC595, U10 74HC74, U11 74LS08, U12 74LS27, U13 74HC04, U14 74HC74, U15 74LS32, U16 74HC74, U17 74LS163, U18 74LS163, U2 74HC595, U3 74HC595, U4 74HC595, U5 74HC595, U6 74HC595, U7 FT231XS, U8 74HC14, U9 74HC74, Y1 Crystal_Small, Y2 Crystal_Small

Commit message: Update readme
Parts:
- removed C23, C24: C, Capacitor_SMD:C_0805_2012Metric_Pad1.18x1.45mm_HandSolder
- removed J3: Conn_02x05_Counter_Clockwise, Connector_PinHeader_2.54mm:PinHeader_2x05_P2.54mm_Vertical
- removed R18: R, Resistor_SMD:R_0805_2012Metric_Pad1.20x1.40mm_HandSolder
- removed U12: 74LS27, Package_SO:SO-14_3.9x8.65mm_P1.27mm
- removed Y1, Y2: Crystal_Small, Crystal:Crystal_HC49-U_Vertical
- added C25: C, Capacitor_SMD:C_1206_3216Metric_Pad1.33x1.80mm_HandSolder, F.Cu at (116.5, 16.7)
- added C26: C, Capacitor_SMD:C_1206_3216Metric_Pad1.33x1.80mm_HandSolder, F.Cu at (116.5, 20.1)
- added D1: D, Diode_THT:D_DO-34_SOD68_P2.54mm_Vertical_KathodeUp, F.Cu at (86.6, 49.9)
- added R19: R, Resistor_SMD:R_0805_2012Metric_Pad1.20x1.40mm_HandSolder, F.Cu at (111.2, 16.5)
- added R20: R, Resistor_SMD:R_0805_2012Metric_Pad1.20x1.40mm_HandSolder, F.Cu at (111.2, 19.5)
- added R21: R, Resistor_SMD:R_0805_2012Metric_Pad1.20x1.40mm_HandSolder, F.Cu at (111.2, 22.4)
- added RV1: R_Potentiometer_Trim_US, Potentiometer_THT:Potentiometer_Bourns_3006P_Horizontal, F.Cu at (105.8, 47.0)
- added SW7: SW_SPDT, Connector_PinHeader_2.54mm:PinHeader_1x03_P2.54mm_Vertical, F.Cu at (103.4, 55.0)
- added U19: 74HC14, Package_SO:SO-14_3.9x8.65mm_P1.27mm, F.Cu at (90.2, 43.8)
- added U20: 74HC74, Package_SO:SO-14_3.9x8.65mm_P1.27mm, F.Cu at (194.0, 105.0)
- C2: value C -> 47
- U18: value 74LS163 -> LTC6907IS6_TRPBF; footprint Package_SO:SO-16_3.9x9.9mm_P1.27mm -> matseng:SOT95P280X100-6N
- moved U13 150.9 mm to (188.9, 128.3), turned to 0 degrees
- moved U15 106.8 mm to (202.5, 94.8)
- moved U17 99.1 mm to (162.8, 101.6), turned to 0 degrees
- moved U8 59.7 mm to (172.2, 79.0), turned to 0 degrees
- moved U16 43.8 mm to (71.1, 40.5)
- moved U18 43.1 mm to (91.4, 52.1)
- moved C17 41.7 mm to (84.3, 44.0)
- moved U14 41.5 mm to (54.6, 40.5)
- moved J1 40.4 mm to (105.4, 41.5), turned to -90 degrees
- moved C5 39.5 mm to (51.4, 34.2), turned to 0 degrees
- moved R17 39.3 mm to (94.7, 51.7)
- moved C18 37.0 mm to (59.7, 34.2), turned to 0 degrees
- moved U10 31.3 mm to (46.4, 40.5)
- moved C6 27.5 mm to (67.9, 34.2), turned to 0 degrees
- moved C7 23.4 mm to (76.0, 34.2), turned to 0 degrees
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Connections:
- net /BUT_RESFLASH renamed PC_FLASH
- net /FEEDCLK renamed Net-(U1-SRCLK)
- net /FEEDLATCH renamed Net-(U1-RCLK)
- net /FEEDOE renamed Net-(U1-~{OE})
- J1 pad 1: Net-(J1-Pin_1) -> GNDD
- J1 pad 3: Net-(J1-Pin_3) -> VCC
- R15 pad 1: Net-(U7-USBDM) -> Net-(U7-USBDP)
- R16 pad 1: Net-(U7-USBDP) -> Net-(U7-USBDM)
- R17 pad 2: Net-(J1-Pin_2) -> Net-(U18-SET)
- U10 pad 1: ~{RES1} -> ~{RESETP}
- U10 pad 12: Net-(U10B-D) -> Net-(U10A-Q)
- U10 pad 13: ~{RES1} -> ~{RESETP}
- U10 pad 2: Net-(U10A-D) -> HALT
- U10 pad 8: unconnected-(U10B-~{Q}-Pad8) -> Net-(U10B-~{Q})
- U10 pad 9: Net-(U10B-Q) -> unconnected-(U10B-Q-Pad9)
- U11 pad 1: Net-(U10A-D) -> Net-(U10A-Q)
- U11 pad 10: unconnected-(U11-Pad10) -> Net-(U14B-~{Q})
- U11 pad 11: Net-(U11-Pad11) -> unconnected-(U11-Pad11)
- U11 pad 12: Net-(U16B-Q) -> Net-(U16A-Q)
- U11 pad 13: CK -> Net-(U16B-Q)
- U11 pad 2: Net-(U10A-Q) -> Net-(U10B-~{Q})
- U11 pad 3: Net-(U11-Pad3) -> unconnected-(U11-Pad3)
- U11 pad 4: Net-(U10B-D) -> Net-(U9A-Q)
- U11 pad 5: Net-(U10B-Q) -> Net-(U9B-~{Q})
- U11 pad 6: Net-(U11-Pad6) -> unconnected-(U11-Pad6)
- U11 pad 8: Net-(U11-Pad8) -> unconnected-(U11-Pad8)
- U11 pad 9: /BUT_TRACE -> Net-(U14A-Q)
- U13 pad 1: Net-(R17-Pad1) -> unconnected-(U13-Pad1)
- U13 pad 10: Net-(U17-~{MR}) -> unconnected-(U13-Pad10)
- U13 pad 11: MOPEND -> unconnected-(U13-Pad11)
- U13 pad 12: Net-(R17-Pad1) -> unconnected-(U13-Pad12)
- U13 pad 13: Net-(J1-Pin_2) -> unconnected-(U13-Pad13)
- U13 pad 2: Net-(J3-Pin_1) -> unconnected-(U13-Pad2)
- U13 pad 3: CK -> unconnected-(U13-Pad3)
- U13 pad 4: /~{CK} -> unconnected-(U13-Pad4)
- U13 pad 5: Net-(U11-Pad6) -> unconnected-(U13-Pad5)
- U13 pad 6: Net-(U14A-~{S}) -> unconnected-(U13-Pad6)
- U13 pad 8: ~{Tick} -> unconnected-(U13-Pad8)
- U13 pad 9: Net-(U17-CP) -> unconnected-(U13-Pad9)
- U14 pad 1: Net-(U14A-~{R}) -> ~{RESETP}
- U14 pad 10: ~{RES1} -> VCC
- U14 pad 12: MOPEND -> Net-(U14A-Q)
- U14 pad 13: VCC -> ~{RESETP}
- U14 pad 2: GNDD -> /BUT_RUNHALT
- U14 pad 3: GNDD -> CK
- U14 pad 4: Net-(U14A-~{S}) -> VCC
- U14 pad 8: Net-(U14A-~{R}) -> Net-(U14B-~{Q})
- U15 pad 2: Net-(U11-Pad3) -> unconnected-(U15-Pad2)
- U15 pad 3: Net-(U16A-C) -> unconnected-(U15-Pad3)
- U15 pad 4: Net-(U16A-Q) -> unconnected-(U15-Pad4)
- U15 pad 5: Net-(U14A-Q) -> unconnected-(U15-Pad5)
- U15 pad 6: Net-(U16B-D) -> unconnected-(U15-Pad6)
- U16 pad 1: ~{RES1} -> ~{RESETP}
- U16 pad 11: /~{CK} -> CK
- U16 pad 12: Net-(U16B-D) -> Net-(U16A-Q)
- U16 pad 13: ~{RES1} -> ~{RESETP}
- U16 pad 3: Net-(U16A-C) -> CK
- U16 pad 6: Net-(U16A-D) -> unconnected-(U16A-~{Q}-Pad6)
- U17 pad 1: Net-(U17-~{MR}) -> unconnected-(U17-~{MR}-Pad1)
- U17 pad 2: Net-(U17-CP) -> unconnected-(U17-CP-Pad2)
- U18 pad 1: VCC -> Net-(U18-OUT)
- U18 pad 2: Net-(J3-Pin_1) -> GNDD
- U18 pad 3: VCC -> Net-(J1-Pin_2)
- U18 pad 4: VCC -> Net-(U18-SET)
- U18 pad 5: VCC -> unconnected-(U18-GRD-Pad5)
- U9 pad 1: ~{RES1} -> VCC
- U9 pad 12: Net-(U9B-D) -> Net-(U9A-Q)
- U9 pad 13: ~{RES1} -> VCC
- U9 pad 2: /BUT_RUNHALT -> Net-(U9A-D)
- U9 pad 5: Net-(U10A-D) -> Net-(U9A-Q)
- U9 pad 8: unconnected-(U9B-~{Q}-Pad8) -> Net-(U9B-~{Q})
- U9 pad 9: Net-(U10B-D) -> unconnected-(U9B-Q-Pad9)
Routing:
- net GNDD: track 327.3 -> 440.4 mm, vias 20 -> 22
- net ~{RES1}: track 77.2 -> 0.00 mm
- net Net-(U11-Pad11): track 51.3 -> 0.00 mm
- net CK: track 80.9 -> 33.4 mm, vias 2 -> 0
- net Net-(U10B-~{Q}): track 0.00 -> 37.7 mm, vias 0 -> 2
- net Net-(U11-Pad8): track 36.8 -> 0.00 mm
- net Net-(U14A-Q): track 14.0 -> 49.0 mm, vias 0 -> 3
- net ~{RESETP}: track 0.00 -> 33.0 mm
- net Net-(J3-Pin_1): track 30.6 -> 0.00 mm, vias 2 -> 0
- net Net-(U14B-~{Q}): track 0.00 -> 29.7 mm, vias 0 -> 2
- net Net-(U10A-Q): track 15.2 -> 44.0 mm, vias 2 -> 5
- net Net-(U16B-Q): track 40.6 -> 12.8 mm, vias 0 -> 2
- net Net-(U16A-D): track 8.26 -> 35.0 mm
- net Net-(U10A-D): track 26.7 -> 0.00 mm, vias 2 -> 0
- net Net-(U11-Pad3): track 26.7 -> 0.00 mm, vias 2 -> 0
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Other:
- board text removed: "÷1"
- board text removed: "÷16"
- board text removed: "÷2"
- board text removed: "÷4"
- board text removed: "÷8"

Commit message: Update readme
Parts:
- added C23: C, Capacitor_SMD:C_0805_2012Metric_Pad1.18x1.45mm_HandSolder, F.Cu at (98.8, 74.8)
- added C24: C, Capacitor_SMD:C_0805_2012Metric_Pad1.18x1.45mm_HandSolder, F.Cu at (105.4, 54.0)
- added C27: C, Capacitor_SMD:C_0805_2012Metric_Pad1.18x1.45mm_HandSolder, F.Cu at (135.8, 58.5)
- added C28: C, Capacitor_SMD:C_0805_2012Metric_Pad1.18x1.45mm_HandSolder, F.Cu at (135.8, 61.5)
- added C29: C, Capacitor_SMD:C_0805_2012Metric_Pad1.18x1.45mm_HandSolder, F.Cu at (140.6, 52.4)
- added C30: C, Capacitor_SMD:C_0805_2012Metric_Pad1.18x1.45mm_HandSolder, F.Cu at (140.6, 55.4)
- added C31: C, Capacitor_SMD:C_0805_2012Metric_Pad1.18x1.45mm_HandSolder, F.Cu at (140.6, 58.5)
- added C32: C, Capacitor_SMD:C_0805_2012Metric_Pad1.18x1.45mm_HandSolder, F.Cu at (140.6, 61.5)
- added C33: C, Capacitor_SMD:C_0805_2012Metric_Pad1.18x1.45mm_HandSolder, F.Cu at (145.4, 52.4)
- added C34: C, Capacitor_SMD:C_0805_2012Metric_Pad1.18x1.45mm_HandSolder, F.Cu at (145.4, 55.4)
- added C35: C, Capacitor_SMD:C_0805_2012Metric_Pad1.18x1.45mm_HandSolder, F.Cu at (145.4, 58.5)
- added C36: C, Capacitor_SMD:C_0805_2012Metric_Pad1.18x1.45mm_HandSolder, F.Cu at (145.4, 61.5)
- moved U8 79.7 mm to (92.7, 74.9), turned to 90 degrees
- moved U17 63.3 mm to (105.4, 74.9), turned to 90 degrees
- moved R21 62.2 mm to (73.9, 72.2)
- moved R20 62.2 mm to (73.9, 69.2)
- moved R19 52.5 mm to (97.8, 67.3), turned to -90 degrees
- moved C26 48.5 mm to (88.4, 59.6)
- moved C25 45.3 mm to (99.1, 58.5), turned to 90 degrees
- moved U19 22.0 mm to (105.4, 59.7)
- moved D1 17.5 mm to (99.1, 62.2)
- moved C4 14.4 mm to (99.8, 42.8), turned to 180 degrees
- moved SW7 12.4 mm to (101.7, 67.3), turned to 90 degrees
- moved J1 11.6 mm to (94.9, 46.5), turned to 180 degrees
- moved U18 10.6 mm to (99.7, 45.5), turned to 0 degrees
- moved R17 6.00 mm to (99.8, 48.5), turned to 0 degrees
Connections:
- net Net-(C22-Pad1) renamed /DEB_RESR
- C12 pad 1: Net-(C12-Pad1) -> /DEB_RUNHALT
- C13 pad 1: Net-(C13-Pad1) -> /DEB_STEP
- C14 pad 1: Net-(C14-Pad1) -> /DEB_TRACE
- C15 pad 1: Net-(C15-Pad1) -> /DEB_USTEP
- C16 pad 1: Net-(C16-Pad1) -> /DEB_RESF
- R10 pad 2: Net-(C16-Pad1) -> /DEB_RESF
- R2 pad 2: Net-(C12-Pad1) -> /DEB_RUNHALT
- R4 pad 2: Net-(C13-Pad1) -> /DEB_STEP
- R6 pad 2: Net-(C14-Pad1) -> /DEB_TRACE
- R8 pad 2: Net-(C15-Pad1) -> /DEB_USTEP
- U8 pad 1: Net-(C14-Pad1) -> /DEB_USTEP
- U8 pad 10: PC_FLASH -> /BUT_STEP
- U8 pad 11: Net-(C16-Pad1) -> /DEB_STEP
- U8 pad 12: /BUT_USTEP -> /BUT_TRACE
- U8 pad 13: Net-(C15-Pad1) -> /DEB_TRACE
- U8 pad 2: /BUT_TRACE -> /BUT_USTEP
- U8 pad 3: Net-(C13-Pad1) -> /DEB_RUNHALT
- U8 pad 4: /BUT_STEP -> /BUT_RUNHALT
- U8 pad 5: Net-(C12-Pad1) -> /DEB_RESF
- U8 pad 6: /BUT_RUNHALT -> PC_FLASH
Routing:
- net Net-(C12-Pad1): track 104.0 -> 0.00 mm, vias 2 -> 0
- net Net-(C13-Pad1): track 89.1 -> 0.00 mm, vias 2 -> 0
- net VCC: track 368.2 -> 449.3 mm, vias 21 -> 26
- net /DEB_RUNHALT: track 0.00 -> 77.0 mm, vias 0 -> 2
- net Net-(C14-Pad1): track 71.2 -> 0.00 mm, vias 2 -> 0
- net /DEB_STEP: track 0.00 -> 68.9 mm, vias 0 -> 2
- net GNDD: track 440.4 -> 507.8 mm, vias 22 -> 26
- net Net-(C15-Pad1): track 55.2 -> 0.00 mm, vias 2 -> 0
- net Net-(J4-Pin_6): track 0.00 -> 27.3 mm
- net /DEB_TRACE: track 0.00 -> 27.1 mm, vias 0 -> 2
- net Net-(J4-Pin_7): track 0.00 -> 23.5 mm
- net /DEB_RESR: track 6.88 -> 28.6 mm
- net Net-(C16-Pad1): track 20.1 -> 0.00 mm
- net Net-(U18-OUT): track 0.00 -> 19.6 mm, vias 0 -> 2
- net Net-(J4-Pin_8): track 0.00 -> 19.1 mm
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Other:
- board text added: "HIGH"
- board text added: "LOW"
- board text added: "MED"

Commit message: Update readme
Parts:
- added R18: ~, Resistor_SMD:R_0805_2012Metric_Pad1.20x1.40mm_HandSolder, F.Cu at (106.7, 40.3)
- added U12: 4075, Package_SO:SO-14_3.9x8.65mm_P1.27mm, F.Cu at (88.9, 73.7)
- moved U13 70.9 mm to (139.4, 77.6)
- moved U20 51.4 mm to (150.2, 78.1)
- moved U15 45.5 mm to (160.5, 77.2)
- moved R21 26.6 mm to (100.3, 69.3), turned to 180 degrees
- moved R20 26.5 mm to (100.3, 67.3), turned to 180 degrees
- moved U8 21.6 mm to (71.1, 73.7)
- moved C23 20.4 mm to (119.1, 73.5)
- moved C26 18.7 mm to (101.3, 73.0), turned to -90 degrees
- moved SW7 7.55 mm to (94.5, 65.2), turned to 180 degrees
- moved D1 7.14 mm to (94.6, 56.6), turned to 90 degrees
- moved U17 6.49 mm to (111.8, 73.7)
- moved C25 3.60 mm to (99.3, 54.9)
- moved R19 3.25 mm to (100.3, 65.3), turned to 180 degrees
- moved C24 0.51 mm to (105.4, 53.5)
- turned C3 to -90 degrees
Connections:
- C3 pad 1: VCC -> GNDD
- C3 pad 2: GNDD -> +5V
- U19 pad 4: Net-(U12-Pad8) -> /POR
- U7 pad 15: VCC -> +5V
- U8 pad 1: /DEB_USTEP -> /DEB_RUNHALT
- U8 pad 10: /BUT_STEP -> /BUT_USTEP
- U8 pad 11: /DEB_STEP -> /DEB_USTEP
- U8 pad 12: /BUT_TRACE -> /BUT_STEP
- U8 pad 13: /DEB_TRACE -> /DEB_STEP
- U8 pad 2: /BUT_USTEP -> /BUT_RUNHALT
- U8 pad 3: /DEB_RUNHALT -> /DEB_TRACE
- U8 pad 4: /BUT_RUNHALT -> /BUT_TRACE
Routing:
- net /BUT_RUNHALT: track 9.04 -> 98.9 mm, vias 0 -> 2
- net Net-(U16A-D): track 35.0 -> 121.9 mm, vias 2 -> 4
- net CK: track 33.4 -> 105.0 mm, vias 0 -> 2
- net /DEB_RUNHALT: track 77.0 -> 27.4 mm, vias 2 -> 0
- net /DEB_STEP: track 68.9 -> 21.6 mm, vias 2 -> 0
- net /BUT_TRACE: track 14.1 -> 45.2 mm, vias 2 -> 0
- net /BUT_STEP: track 1.59 -> 32.1 mm, vias 0 -> 2
- net Net-(R19-Pad1): track 0.00 -> 25.6 mm
- net /POR: track 0.00 -> 24.9 mm
- net /DEB_RESR: track 28.6 -> 53.2 mm
- net /DEB_RESF: track 13.9 -> 35.6 mm, vias 2 -> 0
- net /DEB_USTEP: track 9.08 -> 29.8 mm
- net VCC: track 449.3 -> 468.6 mm, vias 26 -> 30
- net +5V: track 7.08 -> 26.3 mm
- net /DEB_TRACE: track 27.1 -> 10.6 mm, vias 2 -> 0
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Other:
- board text added: "08"
- board text added: "14"
- board text added: "163"
- board text added: "4075"
- board text added: "595"
- board text added: "74"
- board text added: "CPU"
- board text added: "CPU SPEED ADJUST"
- board text added: "FT231"

Commit message: Update README
Parts:
- added R22: ~, Resistor_SMD:R_0805_2012Metric_Pad1.20x1.40mm_HandSolder, F.Cu at (109.2, 40.2)
- moved D1 0.63 mm to (94.7, 56.0)
Connections:
- J4 pad 2: ~{RES1} -> unconnected-(J4-Pin_2-Pad2)
- J4 pad 3: RES2 -> unconnected-(J4-Pin_3-Pad3)
- J4 pad 4: MOPEND -> unconnected-(J4-Pin_4-Pad4)
- J4 pad 5: ~{Tick} -> unconnected-(J4-Pin_5-Pad5)
- U17 pad 9: ~{RES1} -> unconnected-(U17-~{PE}-Pad9)
- U7 pad 17: unconnected-(U7-CBUS1-Pad17) -> PGM
Routing:
- net PGM: track 0.00 -> 16.4 mm, vias 0 -> 2
- net GNDD: track 510.5 -> 520.7 mm
- net ~{RES1}: track 5.24 -> 0.00 mm, vias 1 -> 0
- net unconnected-(U17-~{PE}-Pad9): track 0.00 -> 5.24 mm, vias 0 -> 1
- net /BUT_TRACE: track 45.2 -> 46.1 mm

Commit message: Updates ;-)
Parts:
- added U21: 74HC74, Package_SO:SO-14_3.9x8.65mm_P1.27mm, F.Cu at (62.2, 61.0)
- added U22: 74HC02, Package_SO:SO-14_3.9x8.65mm_P1.27mm, F.Cu at (149.9, 90.2)
- added U23: 74HC02, Package_SO:SO-14_3.9x8.65mm_P1.27mm, F.Cu at (73.3, 61.0)
- added U24: 74HC14, Package_SO:SO-14_3.9x8.65mm_P1.27mm, F.Cu at (81.7, 61.0)
- moved U20 98.3 mm to (53.3, 61.0)
- moved U15 0.51 mm to (160.0, 77.5)
- moved U13 0.34 mm to (139.7, 77.5)
Connections:
- J4 pad 1: CK -> unconnected-(J4-Pin_1-Pad1)
- J4 pad 10: unconnected-(J4-Pin_10-Pad10) -> Net-(J4-Pin_10)
- J4 pad 6: Net-(J4-Pin_6) -> unconnected-(J4-Pin_6-Pad6)
- J4 pad 7: Net-(J4-Pin_7) -> unconnected-(J4-Pin_7-Pad7)
- U11 pad 11: unconnected-(U11-Pad11) -> Net-(U11-Pad11)
- U11 pad 3: unconnected-(U11-Pad3) -> Net-(U11-Pad3)
- U11 pad 6: unconnected-(U11-Pad6) -> Net-(U11-Pad6)
- U11 pad 8: unconnected-(U11-Pad8) -> Net-(U11-Pad8)
- U12 pad 10: unconnected-(U12-Pad10) -> TICK
- U12 pad 11: unconnected-(U12-Pad11) -> Net-(U11-Pad6)
- U12 pad 12: unconnected-(U12-Pad12) -> Net-(U21A-Q)
- U12 pad 13: unconnected-(U12-Pad13) -> Net-(U12-Pad13)
- U13 pad 1: unconnected-(U13-Pad1) -> Net-(U11-Pad11)
- U13 pad 2: unconnected-(U13-Pad2) -> Net-(U20B-~{S})
- U15 pad 1: unconnected-(U15-Pad1) -> Net-(U11-Pad3)
- U15 pad 2: unconnected-(U15-Pad2) -> Net-(U11-Pad8)
- U15 pad 3: unconnected-(U15-Pad3) -> Net-(U20A-C)
- U15 pad 4: unconnected-(U15-Pad4) -> Net-(U20A-Q)
- U15 pad 5: unconnected-(U15-Pad5) -> Net-(U20B-Q)
- U15 pad 6: unconnected-(U15-Pad6) -> Net-(U21B-D)
- U17 pad 1: unconnected-(U17-~{MR}-Pad1) -> VCC
- U17 pad 11: Net-(J4-Pin_9) -> unconnected-(U17-Q3-Pad11)
- U17 pad 12: Net-(J4-Pin_8) -> Net-(J4-Pin_10)
- U17 pad 13: Net-(J4-Pin_7) -> Net-(J4-Pin_9)
- U17 pad 14: Net-(J4-Pin_6) -> Net-(J4-Pin_8)
- U17 pad 2: unconnected-(U17-CP-Pad2) -> TICK
- U17 pad 9: unconnected-(U17-~{PE}-Pad9) -> Net-(U17-~{PE})
- U20 pad 1: unconnected-(U20A-~{R}-Pad1) -> ~{RESETP}
- U20 pad 10: unconnected-(U20B-~{S}-Pad10) -> Net-(U20B-~{S})
- U20 pad 11: unconnected-(U20B-C-Pad11) -> TS6
- U20 pad 12: unconnected-(U20B-D-Pad12) -> GNDD
- U20 pad 13: unconnected-(U20B-~{R}-Pad13) -> ~{RESETP}
- U20 pad 2: unconnected-(U20A-D-Pad2) -> Net-(U20A-D)
- U20 pad 3: unconnected-(U20A-C-Pad3) -> Net-(U20A-C)
- U20 pad 4: unconnected-(U20A-~{S}-Pad4) -> VCC
- U20 pad 5: unconnected-(U20A-Q-Pad5) -> Net-(U20A-Q)
- U20 pad 6: unconnected-(U20A-~{Q}-Pad6) -> Net-(U20A-D)
- U20 pad 9: unconnected-(U20B-Q-Pad9) -> Net-(U20B-Q)
Routing:
- net Net-(J4-Pin_6): track 19.6 -> 0.00 mm
- net Net-(J4-Pin_10): track 0.00 -> 17.1 mm
- net Net-(J4-Pin_7): track 15.8 -> 0.00 mm
- net unconnected-(U11-Pad3): track 6.93 -> 0.00 mm
- net Net-(U11-Pad3): track 0.00 -> 6.93 mm
- net unconnected-(U11-Pad6): track 6.68 -> 0.00 mm
- net Net-(U11-Pad6): track 0.00 -> 6.68 mm
- net unconnected-(U17-~{PE}-Pad9): track 5.24 -> 0.00 mm, vias 1 -> 0
- net Net-(U17-~{PE}): track 0.00 -> 5.24 mm, vias 0 -> 1
- net VCC: track 468.6 -> 472.5 mm
- net Net-(J4-Pin_9): track 13.3 -> 16.6 mm
- net Net-(J4-Pin_8): track 12.6 -> 15.6 mm
- net unconnected-(U11-Pad8): track 2.69 -> 0.00 mm
- net Net-(U11-Pad8): track 0.00 -> 2.69 mm
- net unconnected-(U11-Pad11): track 1.72 -> 0.00 mm
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Other:
- board text added: "02"
- board text added: "04"
- board text added: "32"
