File: PCB/Controlpanel/ControlPanel.kicad_pcb (KiCad board)
At the start: 2 copper layers, 101.6 x 76.2 mm, 101 parts, among them J1 Conn_01x03, J2 USB4105-GF-A, J4 Conn_01x10_Pin, SW1 SW_Push, SW2 SW_Push, SW3 SW_Push, SW4 SW_Push, SW5 SW_Push, SW6 SW_Push, SW7 SW_SPDT, U1 74HC595, U10 74HC74, U11 74LS08, U12 4075, U13 74HC04, U14 74HC74, U15 74LS32, U16 74HC74, U17 74LS163, U18 LTC6907IS6_TRPBF, U19 74HC14, U2 74HC595, U20 74HC74, U21 74HC74, U22 74HC02, U23 74HC02, U24 74HC14, U3 74HC595, U4 74HC595, U5 74HC595, U6 74HC595, U7 FT231XS, U8 74HC14, U9 74HC74

Commit message: Misc updstes
Parts:
- removed U23: 74HC02, Package_SO:SO-14_3.9x8.65mm_P1.27mm
- moved U22 82.2 mm to (72.8, 61.6)
Connections:
- U22 pad 4: unconnected-(U22-Pad4) -> Net-(U12-Pad13)
- U22 pad 5: unconnected-(U22-Pad5) -> Net-(U21B-~{Q})
- U22 pad 6: unconnected-(U22-Pad6) -> ~{CK}
Changed lines of the file:
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@@
   (net 180 "unconnected-(U21A-~{Q}-Pad6)")
   (net 181 "unconnected-(U21B-Q-Pad9)")
-  (net 182 "unconnected-(U22-Pad4)")
-  (net 183 "unconnected-(U22-Pad5)")
-  (net 184 "unconnected-(U22-Pad6)")
-  (net 185 "unconnected-(U22-Pad8)")
-  (net 186 "unconnected-(U22-Pad9)")
-  (net 187 "unconnected-(U22-Pad10)")
-  (net 188 "unconnected-(U22-Pad11)")
-  (net 189 "unconnected-(U22-Pad12)")
-  (net 190 "unconnected-(U22-Pad13)")
+  (net 182 "unconnected-(U22-Pad8)")
+  (net 183 "unconnected-(U22-Pad9)")
+  (net 184 "unconnected-(U22-Pad10)")
+  (net 185 "unconnected-(U22-Pad11)")
+  (net 186 "unconnected-(U22-Pad12)")
+  (net 187 "unconnected-(U22-Pad13)")
   (footprint "Package_SO:SO-14_3.9x8.65mm_P1.27mm" (layer "F.Cu")
     (at 105.41 59.69 90)
@@
   )
   (footprint "Package_SO:SO-14_3.9x8.65mm_P1.27mm" (layer "F.Cu")
-    (at 149.86 90.17)
+    (at 72.771 61.595)
     (descr "SO, 14 Pin (https://www.st.com/resource/en/datasheet/l6491.pdf), generated with kicad-footprint-generator ipc_gullwing_generator.py")
     (tags "SO SO")
@@
       (net 163 "Net-(U9A-D)") (pintype "input"))
     (pad "4" smd roundrect (at -2.475 0) (size 1.95 0.6) (layers "F.Cu" "F.Paste" "F.Mask") (roundrect_rratio 0.25)
-      (net 182 "unconnected-(U22-Pad4)") (pintype "output"))
+      (net 136 "Net-(U12-Pad13)") (pintype "output"))
     (pad "5" smd roundrect (at -2.475 1.27) (size 1.95 0.6) (layers "F.Cu" "F.Paste" "F.Mask") (roundrect_rratio 0.25)
-      (net 183 "unconnected-(U22-Pad5)") (pintype "input"))
+      (net 148 "Net-(U21B-~{Q})") (pintype "input"))
     (pad "6" smd roundrect (at -2.475 2.54) (size 1.95 0.6) (layers "F.Cu" "F.Paste" "F.Mask") (roundrect_rratio 0.25)
-      (net 184 "unconnected-(U22-Pad6)") (pintype "input"))
+      (net 150 "~{CK}") (pintype "input"))
     (pad "7" smd roundrect (at -2.475 3.81) (size 1.95 0.6) (layers "F.Cu" "F.Paste" "F.Mask") (roundrect_rratio 0.25)
       (net 2 "GNDD") (pinfunction "GND") (pintype "power_in"))
     (pad "8" smd roundrect (at 2.475 3.81) (size 1.95 0.6) (layers "F.Cu" "F.Paste" "F.Mask") (roundrect_rratio 0.25)
-      (net 185 "unconnected-(U22-Pad8)") (pintype "input"))
+      (net 182 "unconnected-(U22-Pad8)") (pintype "input"))
     (pad "9" smd roundrect (at 2.475 2.54) (size 1.95 0.6) (layers "F.Cu" "F.Paste" "F.Mask") (roundrect_rratio 0.25)
-      (net 186 "unconnected-(U22-Pad9)") (pintype "input"))
+      (net 183 "unconnected-(U22-Pad9)") (pintype "input"))
     (pad "10" smd roundrect (at 2.475 1.27) (size 1.95 0.6) (layers "F.Cu" "F.Paste" "F.Mask") (roundrect_rratio 0.25)
-      (net 187 "unconnected-(U22-Pad10)") (pintype "output"))
+      (net 184 "unconnected-(U22-Pad10)") (pintype "output"))
     (pad "11" smd roundrect (at 2.475 0) (size 1.95 0.6) (layers "F.Cu" "F.Paste" "F.Mask") (roundrect_rratio 0.25)
-      (net 188 "unconnected-(U22-Pad11)") (pintype "input"))
+      (net 185 "unconnected-(U22-Pad11)") (pintype "input"))
     (pad "12" smd roundrect (at 2.475 -1.27) (size 1.95 0.6) (layers "F.Cu" "F.Paste" "F.Mask") (roundrect_rratio 0.25)
-      (net 189 "unconnected-(U22-Pad12)") (pintype "input"))
+      (net 186 "unconnected-(U22-Pad12)") (pintype "input"))
     (pad "13" smd roundrect (at 2.475 -2.54) (size 1.95 0.6) (layers "F.Cu" "F.Paste" "F.Mask") (roundrect_rratio 0.25)
-      (net 190 "unconnected-(U22-Pad13)") (pintype "output"))
+      (net 187 "unconnected-(U22-Pad13)") (pintype "output"))
     (pad "14" smd roundrect (at 2.475 -3.81) (size 1.95 0.6) (layers "F.Cu" "F.Paste" "F.Mask") (roundrect_rratio 0.25)
       (net 1 "VCC") (pinfunction "VCC") (pintype "power_in"))
@@
     )
   )
-  (footprint "Package_SO:SO-14_3.9x8.65mm_P1.27mm" (layer "F.Cu")
-    (at 73.276 60.96)
-    (descr "SO, 14 Pin (https://www.st.com/resource/en/datasheet/l6491.pdf), generated with kicad-footprint-generator ipc_gullwing_generator.py")
-    (tags "SO SO")
-    (property "Sheetfile" "ControlPanel.kicad_sch")
-    (property "Sheetname" "")
-    (property "ki_description" "quad 2-input NOR gate")
-    (property "ki_keywords" "HCMOS Nor2")
-    (attr smd)
-    (fp_text reference "U23" (at 0 -5.28) (layer "F.SilkS")
-        (effects (font (size 1 1) (thickness 0.15)))
-    )
-    (fp_text value "74HC02" (at 0 5.28) (layer "F.Fab")
-        (effects (font (size 1 1) (thickness 0.15)))
-    )
-    (fp_text user "${REFERENCE}" (at 0 0) (layer "F.Fab")
-        (effects (font (size 0.98 0.98) (thickness 0.15)))
-    )
-    (fp_line (start 0 -4.435) (end -3.45 -4.435)
-      (stroke (width 0.12) (type solid)) (layer "F.SilkS"))
-    (fp_line (start 0 -4.435) (end 1.95 -4.435)
-      (stroke (width 0.12) (type solid)) (layer "F.SilkS"))
-    (fp_line (start 0 4.435) (end -1.95 4.435)
-      (stroke (width 0.12) (type solid)) (layer "F.SilkS"))
-    (fp_line (start 0 4.435) (end 1.95 4.435)
-      (stroke (width 0.12) (type solid)) (layer "F.SilkS"))
-    (fp_line (start -3.7 -4.58) (end -3.7 4.58)
-      (stroke (width 0.05) (type solid)) (layer "F.CrtYd"))
-    (fp_line (start -3.7 4.58) (end 3.7 4.58)
-      (stroke (width 0.05) (type solid)) (layer "F.CrtYd"))
-    (fp_line (start 3.7 -4.58) (end -3.7 -4.58)
-      (stroke (width 0.05) (type solid)) (layer "F.CrtYd"))
-    (fp_line (start 3.7 4.58) (end 3.7 -4.58)
-      (stroke (width 0.05) (type solid)) (layer "F.CrtYd"))
-    (fp_line (start -1.95 -3.35) (end -0.975 -4.325)
-      (stroke (width 0.1) (type solid)) (layer "F.Fab"))
-    (fp_line (start -1.95 4.325) (end -1.95 -3.35)
-      (stroke (width 0.1) (type solid)) (layer "F.Fab"))
-    (fp_line (start -0.975 -4.325) (end 1.95 -4.325)
-      (stroke (width 0.1) (type solid)) (layer "F.Fab"))
-    (fp_line (start 1.95 -4.325) (end 1.95 4.325)
-      (stroke (width 0.1) (type solid)) (layer "F.Fab"))
-    (fp_line (start 1.95 4.325) (end -1.95 4.325)
-      (stroke (width 0.1) (type solid)) (layer "F.Fab"))
-    (pad "1" smd roundrect (at -2.475 -3.81) (size 1.95 0.6) (layers "F.Cu" "F.Paste" "F.Mask") (roundrect_rratio 0.25)
-      (net 136 "Net-(U12-Pad13)") (pintype "output"))
-    (pad "2" smd roundrect (at -2.475 -2.54) (size 1.95 0.6) (layers "F.Cu" "F.Paste" "F.Mask") (roundrect_rratio 0.25)
-      (net 148 "Net-(U21B-~{Q})") (pintype "input"))
-    (pad "3" smd roundrect (at -2.475 -1.27) (size 1.95 0.6) (layers "F.Cu" "F.Paste" "F.Mask") (roundrect_rratio 0.25)
-      (net 150 "~{CK}") (pintype "input"))
-    (pad "4" smd roundrect (at -2.475 0) (size 1.95 0.6) (layers "F.Cu" "F.Paste" "F.Mask") (roundrect_rratio 0.25))
-    (pad "5" smd roundrect (at -2.475 1.27) (size 1.95 0.6) (layers "F.Cu" "F.Paste" "F.Mask") (roundrect_rratio 0.25))
-    (pad "6" smd roundrect (at -2.475 2.54) (size 1.95 0.6) (layers "F.Cu" "F.Paste" "F.Mask") (roundrect_rratio 0.25))
-    (pad "7" smd roundrect (at -2.475 3.81) (size 1.95 0.6) (layers "F.Cu" "F.Paste" "F.Mask") (roundrect_rratio 0.25))
-    (pad "8" smd roundrect (at 2.475 3.81) (size 1.95 0.6) (layers "F.Cu" "F.Paste" "F.Mask") (roundrect_rratio 0.25))
-    (pad "9" smd roundrect (at 2.475 2.54) (size 1.95 0.6) (layers "F.Cu" "F.Paste" "F.Mask") (roundrect_rratio 0.25))
-    (pad "10" smd roundrect (at 2.475 1.27) (size 1.95 0.6) (layers "F.Cu" "F.Paste" "F.Mask") (roundrect_rratio 0.25))
-    (pad "11" smd roundrect (at 2.475 0) (size 1.95 0.6) (layers "F.Cu" "F.Paste" "F.Mask") (roundrect_rratio 0.25))
-    (pad "12" smd roundrect (at 2.475 -1.27) (size 1.95 0.6) (layers "F.Cu" "F.Paste" "F.Mask") (roundrect_rratio 0.25))
-    (pad "13" smd roundrect (at 2.475 -2.54) (size 1.95 0.6) (layers "F.Cu" "F.Paste" "F.Mask") (roundrect_rratio 0.25))
-    (pad "14" smd roundrect (at 2.475 -3.81) (size 1.95 0.6) (layers "F.Cu" "F.Paste" "F.Mask") (roundrect_rratio 0.25))
-    (model "${KICAD6_3DMODEL_DIR}/Package_SO.3dshapes/SO-14_3.9x8.65mm_P1.27mm.wrl"
-      (offset (xyz 0 0 0))
-      (scale (xyz 1 1 1))
-      (rotate (xyz 0 0 0))
-    )
-  )
   (footprint "Resistor_SMD:R_0805_2012Metric_Pad1.20x1.40mm_HandSolder" (layer "F.Cu")
     (at 100.33 69.342 180)
@@
     (effects (font (size 1 1) (thickness 0.2) bold))
   )
-  (gr_text "02" (at 149.86 90.17 270) (layer "F.SilkS")
+  (gr_text "02" (at 72.771 61.595 270) (layer "F.SilkS")
     (effects (font (size 1.27 1.27) (thickness 0.2)))
   )
