File: PCB/Controlpanel/ControlPanel.kicad_sch (KiCad schematic)
At the start: 79 parts, among them J1 Conn_01x03, J2 USB4105-GF-A, J3 Conn_02x05_Counter_Clockwise, J4 Conn_01x10_Pin, SW1 SW_Push, SW2 SW_Push, SW3 SW_Push, SW4 SW_Push, SW5 SW_Push, SW6 SW_Push, U1 74HC595, U10 74HC74, U11 74LS08, U12 74LS27, U13 74HC04, U14 74HC74, U15 74LS32, U16 74HC74, U17 74LS163, U18 74LS163, U2 74HC595, U3 74HC595, U4 74HC595, U5 74HC595, U6 74HC595, U7 FT231XS, U8 74HC14, U9 74HC74, Y1 Crystal_Small, Y2 Crystal_Small

Commit message: Update readme
Parts:
- removed C3 (x2): C, Capacitor_SMD:C_0805_2012Metric_Pad1.18x1.45mm_HandSolder, symbol Device:C
- removed J3: Conn_02x05_Counter_Clockwise, Connector_PinHeader_2.54mm:PinHeader_2x05_P2.54mm_Vertical, symbol Connector_Generic:Conn_02x05_Odd_Even
- removed R18: R, Resistor_SMD:R_0805_2012Metric_Pad1.20x1.40mm_HandSolder, symbol Device:R
- removed U12: 74LS27, Package_SO:SO-14_3.9x8.65mm_P1.27mm, symbol 74xx:74LS27
- removed U18: 74LS163, Package_SO:SO-16_3.9x9.9mm_P1.27mm, symbol 74xx:74LS163
- removed Y1, Y2: Crystal_Small, Crystal:Crystal_HC49-U_Vertical, symbol Device:Crystal_Small
- added C25, C26: C, Capacitor_SMD:C_1206_3216Metric_Pad1.33x1.80mm_HandSolder, symbol Device:C
- added D1: D, Diode_THT:D_DO-34_SOD68_P2.54mm_Vertical_KathodeUp, symbol Device:D
- added R19, R20, R21: R, Resistor_SMD:R_0805_2012Metric_Pad1.20x1.40mm_HandSolder, symbol Device:R
- added RV1: R_Potentiometer_Trim_US, Potentiometer_THT:Potentiometer_Bourns_3006P_Horizontal, symbol Device:R_Potentiometer_Trim_US
- added SW7: SW_SPDT, Connector_PinHeader_2.54mm:PinHeader_1x03_P2.54mm_Vertical, symbol Switch:SW_SPDT
- added U12: 4075, symbol 4xxx:4075
- added U18: LTC6907IS6_TRPBF, matseng:SOT95P280X100-6N, symbol matseng:LTC6907IS6_TRPBF
- added U19: 74HC14, Package_SO:SO-14_3.9x8.65mm_P1.27mm, symbol 74xx:74HC14
- added U20: 74HC74, Package_SO:SO-14_3.9x8.65mm_P1.27mm, symbol 74xx:74HC74
- C1: value C -> 47
Connections:
- net BUT_RESRAM: now also U12.2
- net BUT_RUNHALT: now also U14.2 (D), U12.3; no longer U9.2 (D)
- net BUT_STEP: now also U12.4
- net BUT_TRACE: now also D1.2 (A); no longer U11.9
- net CK: now also U14.3 (C), U16.11 (C), U16.3 (C), U19.10; no longer U11.13, U13.3
- net GNDD: now also J1.1 (Pin_1), C25.2, C26.2, RV1.3, U12.7 (VSS), U18.2 (GND), U19.7 (GND), U20.7 (GND); no longer U14.2 (D), U14.3 (C)
- net MOPEND: no longer U13.11, U14.12 (D)
- net VCC: now also J1.3 (Pin_3), U14.10 (~{S}), U14.4 (~{S}), U9.1 (~{R}), U9.13 (~{R}), R21.2, U12.14 (VDD), U18.6 (V+), U19.14 (VCC), U20.14 (VCC); no longer U14.13 (~{R})
- net ~{CK}: now also U19.11, U19.8; no longer U13.4, U16.11 (C)
- net ~{RES1}: no longer U10.1 (~{R}), U10.13 (~{R}), U14.10 (~{S}), U16.1 (~{R}), U16.13 (~{R}), U9.1 (~{R}), U9.13 (~{R})
- net ~{Tick}: no longer U13.8
- net at U10.5 (Q): now also U10.12 (D), U11.1; no longer U11.2
- net at U11.3: no longer U15.2
- net at U13.10: no longer U17.1 (~{MR})
- net at U11.10: now also U14.8 (~{Q})
- net at U11.5: now also U9.8 (~{Q}); no longer U10.9 (Q)
- net at U11.6: no longer U13.5
- net at R15.1: now also U7.11 (USBDP); no longer U7.12 (USBDM)
- net at U13.9: no longer U17.2 (CP)
- net at U9.12 (D): now also U11.4, U9.5 (Q)
- net at U15.3: no longer U16.3 (C)
- net at U16.12 (D): now also U11.12, U16.5 (Q); no longer U15.6
- net at U16.9 (Q): now also U11.13; no longer U11.12
- net at R16.1: now also U7.12 (USBDM); no longer U7.11 (USBDP)
- net at U15.4: no longer U16.5 (Q)
- net at U14.5 (Q): now also U11.9, U14.12 (D); no longer U15.5
- net ~{RESETP}: now reaches U14.1 (~{R})
- net ~{RESETP}: now also U10.1 (~{R}), U10.13 (~{R}), U14.13 (~{R}), U16.1 (~{R}), U16.13 (~{R}); no longer U14.8 (~{Q})
- net at U13.6: no longer U14.4 (~{S})
- net at U16.2 (D): now also U12.6; no longer U16.6 (~{Q})
- net at U10.8 (~{Q}): now also U11.2
- net BUT_RESFLASH renamed PC_FLASH
- net PC_FLASH: now also U12.1
- net FEEDCLK: no longer names the net of U1.11 (SRCLK), U2.11 (SRCLK), U3.11 (SRCLK), U4.11 (SRCLK), U5.11 (SRCLK), U6.11 (SRCLK), U7.8 (~{DCD})
- net FEEDLATCH: no longer names the net of U1.12 (RCLK), U2.12 (RCLK), U3.12 (RCLK), U4.12 (RCLK), U5.12 (RCLK), U6.12 (RCLK), U7.5 (~{RI})
- net FEEDOE: no longer names the net of U1.13 (~{OE}), U2.13 (~{OE}), U3.13 (~{OE}), U4.13 (~{OE}), U5.13 (~{OE}), U6.13 (~{OE}), U7.18 (CBUS0)
- new net: R17.1, RV1.2
- new net: U12.9, U19.5, U9.2 (D)
- new net: J1.2 (Pin_2), U18.3 (DIV)
- new net: R19.1, R20.1, U12.5, U19.2
- new net: R19.2, SW7.3 (C)
- new net: C26.1, R21.1, U19.3
- new net: U12.8, U19.4
- new net: C25.1, D1.1 (K), SW7.2 (B), U19.1
- new net: U18.1 (OUT), U19.9
- new net: R17.2, U18.4 (SET)
- new net: R20.2, SW7.1 (A)
- new net HALT: U10.2 (D)
- new net ~{RESET}: U19.6
- now unconnected: U13.1, U13.12, U13.13, U9.9 (Q)
- no-connect marks 14 -> 19
Other:
- moved on the sheet: BUS2, C1, C2, C3, C4, C5, C6, C7, C8, C9, C96, C97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

Commit message: Update readme
Parts:
- added C23, C24, C27, C28, C29, C30, C31, C32, C33, C34, C35, C36: C, Capacitor_SMD:C_0805_2012Metric_Pad1.18x1.45mm_HandSolder, symbol Device:C
Connections:
- net BUT_RUNHALT: now also U8.4; no longer U8.6
- net BUT_STEP: now also U8.10; no longer U8.4
- net BUT_TRACE: now also U8.12; no longer U8.2
- net BUT_USTEP: now also U8.2; no longer U8.12
- net GNDD: now also C23.2, C24.2, C27.2, C28.2, C29.2, C30.2, C31.2, C32.2, C33.2, C34.2, C35.2, C36.2
- net PC_FLASH: now also U8.6; no longer U8.10
- net VCC: now also C23.1, C24.1, C27.1, C28.1, C29.1, C30.1, C31.1, C32.1, C33.1, C34.1, C35.1, C36.1
- net DEB_RESR: now reaches C3.1, R12.2, U8.9
- net DEB_STEP: now reaches C3.1, R4.2
- net DEB_STEP: now also U8.11; no longer U8.3
- net DEB_TRACE: now reaches C3.1, R6.2
- net DEB_TRACE: now also U8.13; no longer U8.1
- net DEB_RESF: now reaches C3.1, R10.2
- net DEB_RESF: now also U8.5; no longer U8.11
- net DEB_RUNHALT: now reaches C3.1, R2.2
- net DEB_RUNHALT: now also U8.3; no longer U8.5
- net DEB_USTEP: now reaches C3.1, R8.2
- net DEB_USTEP: now also U8.1; no longer U8.13
Other:
- moved on the sheet: U8A, U8B, U8C, U8E, U8F

Commit message: Update readme
Parts:
- added R18, R22: ~, Resistor_SMD:R_0805_2012Metric_Pad1.20x1.40mm_HandSolder, symbol Device:R
- U12: footprint (none) -> Package_SO:SO-14_3.9x8.65mm_P1.27mm
Connections:
- net +5V: now also C2.2, U7.15 (VCC)
- net BUT_RUNHALT: now also U8.2; no longer U8.4
- net BUT_STEP: now also U8.12; no longer U8.10
- net BUT_TRACE: now also U8.4; no longer U8.12
- net BUT_USTEP: now also U8.10; no longer U8.2
- net DEB_RUNHALT: now also U8.1; no longer U8.3
- net DEB_STEP: now also U8.13; no longer U8.11
- net DEB_TRACE: now also U8.3; no longer U8.13
- net DEB_USTEP: now also U8.11; no longer U8.1
- net GNDD: now also C2.1, R22.1; no longer C2.2
- net MOPEND: no longer J4.4 (Pin_4)
- net VCC: now also R18.2; no longer C2.1, U7.15 (VCC)
- net ~{Tick}: no longer J4.5 (Pin_5)
- net at U1.13 (~{OE}), U2.13 (~{OE}), U3.13 (~{OE})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: now also R18.1
- net POR: now reaches U12.8, U19.4
- net PGM: now reaches U7.17 (CBUS1)
- net PGM: now also R22.2
- net RES2: no longer names the net of J4.3 (Pin_3)
- net ~{RES1}: no longer names the net of J4.2 (Pin_2)
- net ~{RES1}: no longer U17.9 (~{PE})
- no-connect marks 19 -> 12
Other:
- moved on the sheet: BUS2, C2, C23, C24, C26, C27, C28, C29, C3, C30, C31, C33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

Commit message: Update README
Parts:
- added U21: 74HC74, symbol 74xx:74HC74
Connections:
- net GNDD: now also U21.7 (GND)
- net VCC: now also U21.14 (VCC)
Other:
- moved on the sheet: U10C, U11E, U12D, U13G, U14C, U15E, U16C, U19G, U20B, U20C, U8G, U9C

Commit message: Updates ;-)
Parts:
- added U22, U23: 74HC02, Package_SO:SO-14_3.9x8.65mm_P1.27mm, symbol 74xx:74HC02
- added U24: 74HC14, Package_SO:SO-14_3.9x8.65mm_P1.27mm, symbol 74xx:74HC14
- U21: footprint (none) -> Package_SO:SO-14_3.9x8.65mm_P1.27mm
Connections:
- net BUT_USTEP: now also U21.2 (D)
- net CK: no longer J4.1 (Pin_1)
- net GNDD: now also U20.12 (D), U22.7 (GND)
- net VCC: now also U17.1 (~{MR}), U20.4 (~{S}), U21.10 (~{S}), U21.4 (~{S}), U22.14 (VCC)
- net ~{CK}: now also U21.11 (C), U21.3 (C), U23.3
- net ~{RESETP}: now also U20.1 (~{R}), U20.13 (~{R}), U21.1 (~{R}), U21.13 (~{R}), U24.6
- net at U11.3: now also U15.1
- net at U12.9, U19.5, U9.2 (D): now also U22.3
- net at U11.8: now also U15.2
- net at J4.10 (Pin_10): now also U17.12 (Q2)
- net at J4.6 (Pin_6): no longer U17.14 (Q0)
- net at J4.7 (Pin_7): no longer U17.13 (Q1)
- net at J4.8 (Pin_8): now also U17.14 (Q0); no longer U17.12 (Q2)
- net at J4.9 (Pin_9): now also U17.13 (Q1); no longer U17.11 (Q3)
- net at U13.1: now also U11.11
- net at U13.2: now also U20.10 (~{S})
- net at U11.6: now also U12.11, U24.5
- net TICK: now reaches U12.10
- net TICK: now also U17.2 (CP)
- net at U12.12: now also U21.5 (Q)
- net at U12.13: now also U23.1
- net TS6: now reaches U20.11 (C)
- net TS6: now also U22.2
- net at U20.9 (Q): now also U15.5
- net at U20.2 (D): now also U20.6 (~{Q})
- net at U20.3 (C): now also U15.3
- net at U20.5 (Q): now also U15.4
- net at U15.6: now also U21.12 (D)
- net at U21.8 (~{Q}): now also U23.2
- net at U17.9 (~{PE}): now also U22.1
- no-connect marks 12 -> 15
Other:
- moved on the sheet: BUS2, C1, C2, C23, C24, C25, C26, C27, C28, C29, C3, C30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

Commit message: Misc updstes
Parts:
- removed unit 1 of U10
- removed unit 2 of U10
- removed unit 1 of U14
- removed unit 2 of U14
- removed unit 2 of U16
- removed unit 1 of U16
- removed U23: 74HC02, Package_SO:SO-14_3.9x8.65mm_P1.27mm, symbol 74xx:74HC02
- removed unit 2 of U9
- removed unit 1 of U9
- added U23, U25: 74LS175, Package_SO:SOIC-16_3.9x9.9mm_P1.27mm, symbol 74xx:74LS175
Connections:
- net BUT_RUNHALT: now also U23.12 (D2)
- net CK: now also U23.9 (Cp), U25.9 (Cp)
- net GNDD: now also U23.8 (GND), U25.8 (GND)
- net HALT: now also U23.5 (D1)
- net TS6: now also U22.3; no longer U22.2
- net VCC: now also U23.16 (VCC), U25.16 (VCC)
- net ~{CK}: now also U22.6
- net ~{RESETP}: now also U23.1 (~{Mr}), U25.1 (~{Mr})
- net at U11.1: now also U23.7 (Q1), U25.5 (D1)
- net at U11.2: now also U25.6 (~{Q1})
- net at U12.9, U19.5: now also U22.2, U23.4 (D0); no longer U22.3
- net at U11.10: now also U25.11 (~{Q2})
- net at U11.9: now also U23.10 (Q2), U25.12 (D2)
- net at U11.4: now also U23.2 (Q0), U25.4 (D0)
- net at U11.5: now also U25.3 (~{Q0})
- net at U12.13: now also U21.5 (Q)
- net at U21.8 (~{Q}): now also U22.5
- net at U12.12: now also U22.4; no longer U21.5 (Q)
- net at U11.12: now also U23.15 (Q3), U25.13 (D3)
- net at U11.13: now also U25.14 (~{Q3})
- net at U12.6: now also U23.13 (D3)
- no-connect marks 15 -> 18
Other:
- moved on the sheet: C25, C26, C3, D1, J1, R10, R11, R12, R13, R17, R19, R2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
