File: PCB/MAR/MAR.kicad_pcb (KiCad board)
At the start: 4 copper layers, 101.6 x 76.2 mm, 41 parts, among them J1a1 Conn_02x04_Odd_Even, J1b1 Conn_02x04_Odd_Even, J1c1 Conn_02x04_Odd_Even, J4 Conn_01x08_Pin, U1 74HC74, U13 74HC245, U14 74HC245, U15 74HC245, U2 74HC04, U7 74HCT574, U8 74HCT574, U9 74HCT574

Commit message: Update readme
Routing:
- net GNDD: track 243.3 -> 243.8 mm, vias 13 -> 15

Commit message: Updates ;-)
Routing:
- net GNDD: track 243.8 -> 240.8 mm
Other:
- board text added: "• Memory address register • github.com/mengstr/SUBLEQ24 • rev2 •"
- board text removed: "• Memory address register • github.com/mengstr/SUBLEQ24 • rev1 •"
Changed lines of the file:
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@@
     (effects (font (size 0.9 0.9) (thickness 0.15)))
   )
-  (gr_text "• Memory address register • github.com/mengstr/SUBLEQ24 • rev1 •" (at 76.2 100.203) (layer "F.SilkS")
+  (gr_text "• Memory address register • github.com/mengstr/SUBLEQ24 • rev2 •" (at 76.2 100.203) (layer "F.SilkS")
     (effects (font (face "Futura") (size 1.4 1.4) (thickness 0.15)))
-    (render_cache "• Memory address register • github.com/mengstr/SUBLEQ24 • rev1 •" 0
+    (render_cache "• Memory address register • github.com/mengstr/SUBLEQ24 • rev2 •" 0
       (polygon
         (pts
@@
       (polygon
         (pts
-          (xy 105.681382 99.514718)          (xy 105.425952 99.514718)          (xy 105.548367 99.295877)          (xy 105.901591 99.295877)
-          (xy 105.901591 100.794942)          (xy 105.681382 100.794942)
+          (xy 105.657788 100.565158)          (xy 106.207969 100.565158)          (xy 106.207969 100.784)          (xy 105.215659 100.784)
+          (xy 105.728569 100.156882)          (xy 105.737919 100.145309)          (xy 105.747077 100.133929)          (xy 105.756042 100.122741)
+          (xy 105.764815 100.111745)          (xy 105.773395 100.100942)          (xy 105.785906 100.085098)          (xy 105.797983 100.069687)
+          (xy 105.809628 100.054708)          (xy 105.82084 100.040162)          (xy 105.831619 100.026049)          (xy 105.841965 100.012369)
+          (xy 105.851879 99.999122)          (xy 105.855087 99.994802)          (xy 105.864491 99.98211)          (xy 105.873468 99.96981)
+          (xy 105.882018 99.9579)          (xy 105.890141 99.94638)          (xy 105.900309 99.931629)          (xy 105.909717 99.917572)
+          (xy 105.918367 99.904209)          (xy 105.926259 99.891541)          (xy 105.933391 99.879568)          (xy 105.943108 99.862737)
+          (xy 105.951868 99.846225)          (xy 105.959673 99.830031)          (xy 105.966522 99.814156)          (xy 105.972416 99.7986)
+          (xy 105.977353 99.783362)          (xy 105.981335 99.768442)          (xy 105.984362 99.753841)          (xy 105.986432 99.739559)
+          (xy 105.987547 99.725595)          (xy 105.98776 99.716463)          (xy 105.98712 99.697206)          (xy 105.985199 99.678544)
+          (xy 105.981999 99.660477)          (xy 105.977518 99.643005)          (xy 105.971756 99.626128)          (xy 105.964715 99.609846)
+          (xy 105.956393 99.594159)          (xy 105.946791 99.579067)          (xy 105.935909 99.56457)          (xy 105.923746 99.550669)
+          (xy 105.914927 99.541732)          (xy 105.901031 99.529082)          (xy 105.886528 99.517677)          (xy 105.871418 99.507516)
+          (xy 105.855701 99.498599)          (xy 105.839378 99.490926)          (xy 105.822446 99.484498)          (xy 105.804908 99.479314)
+          (xy 105.786763 99.475374)          (xy 105.768011 99.472678)          (xy 105.748652 99.471226)          (xy 105.735408 99.47095)
+          (xy 105.721597 99.47121)          (xy 105.695094 99.473288)          (xy 105.670084 99.477445)          (xy 105.646567 99.48368)
+          (xy 105.624544 99.491993)          (xy 105.604015 99.502385)          (xy 105.584978 99.514855)          (xy 105.567435 99.529404)
+          (xy 105.551385 99.54603)          (xy 105.536829 99.564736)          (xy 105.523766 99.585519)          (xy 105.512196 99.608381)
+          (xy 105.502119 99.633321)          (xy 105.497641 99.646571)          (xy 105.493536 99.66034)          (xy 105.489804 99.674629)
+          (xy 105.486446 99.689437)          (xy 105.483461 99.704765)          (xy 105.480849 99.720612)          (xy 105.478611 99.736979)
+          (xy 105.256692 99.736979)          (xy 105.260405 99.708663)          (xy 105.264832 99.681246)          (xy 105.269974 99.654727)
+          (xy 105.27583 99.629108)          (xy 105.282401 99.604387)          (xy 105.289687 99.580566)          (xy 105.297687 99.557643)
+          (xy 105.306402 99.535619)          (xy 105.315831 99.514495)          (xy 105.325975 99.494269)          (xy 105.336834 99.474942)
+          (xy 105.348407 99.456514)          (xy 105.360695 99.438985)          (xy 105.373697 99.422354)          (xy 105.387414 99.406623)
+          (xy 105.401846 99.391791)          (xy 105.416992 99.377857)          (xy 105.432853 99.364823)          (xy 105.449428 99.352687)
+          (xy 105.466718 99.341451)          (xy 105.484723 99.331113)          (xy 105.503442 99.321674)          (xy 105.522876 99.313135)
+          (xy 105.543024 99.305494)          (xy 105.563887 99.298752)          (xy 105.585465 99.292909)          (xy 105.607757 99.287965)
+          (xy 105.630764 99.283919)          (xy 105.654485 99.280773)          (xy 105.678921 99.278526)          (xy 105.704072 99.277178)
+          (xy 105.729937 99.276728)          (xy 105.754987 99.277228)          (xy 105.779529 99.278726)          (xy 105.803564 99.281224)
+          (xy 105.827091 99.284721)          (xy 105.85011 99.289217)          (xy 105.872622 99.294712)          (xy 105.894627 99.301206)
+          (xy 105.916123 99.308699)          (xy 105.937113 99.317192)          (xy 105.957594 99.326683)          (xy 105.977568 99.337174)
+          (xy 105.997035 99.348664)          (xy 106.015994 99.361152)          (xy 106.034445 99.37464)          (xy 106.052389 99.389127)
+          (xy 106.069825 99.404614)          (xy 106.086554 99.420837)          (xy 106.102203 99.437536)          (xy 106.116773 99.45471)
+          (xy 106.130263 99.47236)          (xy 106.142675 99.490486)          (xy 106.154007 99.509087)          (xy 106.16426 99.528163)
+          (xy 106.173433 99.547715)          (xy 106.181528 99.567743)          (xy 106.188543 99.588246)          (xy 106.194479 99.609225)
+          (xy 106.199335 99.630679)          (xy 106.203113 99.652608)          (xy 106.205811 99.675013)          (xy 106.207429 99.697894)
+          (xy 106.207969 99.72125)          (xy 106.207717 99.736234)          (xy 106.206959 99.75118)          (xy 106.205697 99.76609)
+          (xy 106.20393 99.780961)          (xy 106.201658 99.795796)          (xy 106.198881 99.810593)          (xy 106.195599 99.825352)
+          (xy 106.191812 99.840074)          (xy 106.187521 99.854759)          (xy 106.182724 99.869406)          (xy 106.177423 99.884016)
+          (xy 106.171617 99.898589)          (xy 106.165305 99.913124)          (xy 106.158489 99.927621)          (xy 106.151168 99.942082)
+          (xy 106.143342 99.956505)          (xy 106.134741 99.971978)          (xy 106.127658 99.984031)          (xy 106.120034 99.996469)
+          (xy 106.11187 100.009292)          (xy 106.103165 100.022499)          (xy 106.093918 100.036091)          (xy 106.084131 100.050068)
+          (xy 106.073802 100.06443)          (xy 106.062933 100.079176)          (xy 106.051523 100.094307)          (xy 106.047599 100.099436)
+          (xy 106.035511 100.115152)          (xy 106.022839 100.131396)          (xy 106.014068 100.14252)          (xy 106.005037 100.153879)
+          (xy 105.995747 100.165473)          (xy 105.986198 100.177302)          (xy 105.97639 100.189366)          (xy 105.966323 100.201665)
+          (xy 105.955997 100.214199)          (xy 105.945411 100.226969)          (xy 105.934567 100.239973)          (xy 105.923463 100.253212)
+          (xy 105.9121 100.266687)          (xy 105.900478 100.280397)          (xy 105.888597 100.294341)
         )
       )
@@
   (segment (start 92.775 66.04) (end 94.234 66.04) (width 0.4) (layer "F.Cu") (net 2))
   (segment (start 90.805 66.04) (end 92.775 66.04) (width 0.127) (layer "F.Cu") (net 2))
-  (segment (start 73.025 67.945) (end 71.55 67.945) (width 0.4) (layer "F.Cu") (net 2))
   (segment (start 73.025 64.77) (end 73.025 61.595) (width 0.4) (layer "F.Cu") (net 2))
   (segment (start 47.625 64.77) (end 47.625 61.595) (width 0.4) (layer "F.Cu") (net 2))
@@
   (segment (start 47.625 97.155) (end 47.625 85.725) (width 0.4) (layer "F.Cu") (net 2))
   (segment (start 26.67 27.695) (end 30.099 27.695) (width 0.127) (layer "F.Cu") (net 2))
-  (segment (start 73.025 50.165) (end 71.55 50.165) (width 0.4) (layer "F.Cu") (net 2))
   (segment (start 94.2125 67.9665) (end 94.234 67.945) (width 0.4) (layer "F.Cu") (net 2))
   (segment (start 99.441 62.23) (end 99.441 64.77) (width 0.127) (layer "F.Cu") (net 2))
