File: PCB/Memory/Memory.kicad_pcb (KiCad board)
At the start: 2 copper layers, 101.6 x 76.2 mm, 36 parts, among them J1 Conn_01x08_Pin, U1 74LS139, U7 SST39SF020, U8 SST39SF020, U9 SST39SF020

Commit message: Update readme
Parts:
- removed JP7, JP8: SolderJumper_2_Open, Jumper:SolderJumper-2_P1.3mm_Open_Pad1.0x1.5mm
- added D1: LED, LED_SMD:LED_0805_2012Metric_Pad1.15x1.40mm_HandSolder, F.Cu at (40.6, 94.0)
- added D2: LED, LED_SMD:LED_0805_2012Metric_Pad1.15x1.40mm_HandSolder, F.Cu at (38.1, 94.0)
- added D3: LED, LED_SMD:LED_0805_2012Metric_Pad1.15x1.40mm_HandSolder, F.Cu at (48.3, 94.0)
- added D4: LED, LED_SMD:LED_0805_2012Metric_Pad1.15x1.40mm_HandSolder, F.Cu at (45.7, 94.0)
- added D5: LED, LED_SMD:LED_0805_2012Metric_Pad1.15x1.40mm_HandSolder, F.Cu at (104.1, 94.0)
- added D6: LED, LED_SMD:LED_0805_2012Metric_Pad1.15x1.40mm_HandSolder, F.Cu at (106.7, 94.0)
- added D7: LED, LED_SMD:LED_0805_2012Metric_Pad1.15x1.40mm_HandSolder, F.Cu at (109.2, 94.0)
- added R1: R, Resistor_SMD:R_0805_2012Metric_Pad1.20x1.40mm_HandSolder, F.Cu at (40.6, 89.9)
- added R2: R, Resistor_SMD:R_0805_2012Metric_Pad1.20x1.40mm_HandSolder, F.Cu at (38.1, 89.9)
- added R3: R, Resistor_SMD:R_0805_2012Metric_Pad1.20x1.40mm_HandSolder, F.Cu at (48.3, 89.9)
- added R4: R, Resistor_SMD:R_0805_2012Metric_Pad1.20x1.40mm_HandSolder, F.Cu at (45.7, 89.9)
- added R5: R, Resistor_SMD:R_0805_2012Metric_Pad1.20x1.40mm_HandSolder, F.Cu at (104.1, 89.9)
- added R6: R, Resistor_SMD:R_0805_2012Metric_Pad1.20x1.40mm_HandSolder, F.Cu at (106.7, 89.9)
- added R7: R, Resistor_SMD:R_0805_2012Metric_Pad1.20x1.40mm_HandSolder, F.Cu at (109.2, 89.9)
- J1: value Conn_01x08_Pin -> Conn_01x06_Pin; footprint Connector_PinHeader_2.54mm:PinHeader_1x08_P2.54mm_Vertical -> Connector_PinHeader_2.54mm:PinHeader_1x06_P2.54mm_Vertical
- renumbered RAM-L0 to U1, U1 to U10, RAM0-M1 to U2, RAM-0H1 to U3, RAM-1L1 to U4, RAM-1M1 to U5, RAM-1H1 to U6, U9 to U7, U7 to U8, U8 to U9
Connections:
- J1 pad 1: /~{WER1} -> /~{WER}
- J1 pad 2: /~{WER0} -> /~{OER}
- J1 pad 3: /~{OER1} -> /~{WEF}
- J1 pad 4: /~{OER0} -> /~{OEF}
- J1 pad 5: /~{WEF} -> unconnected-(J1-Pin_5-Pad5)
- J1 pad 6: /~{OEF} -> unconnected-(J1-Pin_6-Pad6)
- U1 pad 11: /~{WER0} -> /~{WER}
- U1 pad 28: /~{OER0} -> /~{OER}
- U2 pad 11: /~{WER0} -> /~{WER}
- U2 pad 28: /~{OER0} -> /~{OER}
- U3 pad 11: /~{WER0} -> /~{WER}
- U3 pad 28: /~{OER0} -> /~{OER}
- U4 pad 11: /~{WER1} -> /~{WER}
- U4 pad 28: /~{OER1} -> /~{OER}
- U5 pad 11: /~{WER1} -> /~{WER}
- U5 pad 28: /~{OER1} -> /~{OER}
- U6 pad 11: /~{WER1} -> /~{WER}
- U6 pad 28: /~{OER1} -> /~{OER}
Routing:
- net /~{WER}: track 0.00 -> 158.5 mm, vias 0 -> 7
- net /~{OER}: track 0.00 -> 136.5 mm, vias 0 -> 7
- net /~{WER1}: track 113.2 -> 0.00 mm, vias 4 -> 0
- net /~{OER1}: track 102.8 -> 0.00 mm, vias 4 -> 0
- net /~{WER0}: track 102.3 -> 0.00 mm, vias 4 -> 0
- net /~{OER0}: track 87.1 -> 0.00 mm, vias 4 -> 0
- net VCC: track 277.1 -> 359.3 mm
- net /~{OEF}: track 54.0 -> 97.2 mm, vias 1 -> 2
- net /~{CS_RAM0}: track 108.8 -> 141.1 mm
- net /~{CS_RAM1}: track 98.1 -> 119.0 mm, vias 5 -> 7
- net /~{WEF}: track 96.5 -> 115.8 mm
- net /~{CS_FLASH}: track 98.4 -> 102.3 mm
- net Net-(D7-K): track 0.00 -> 2.08 mm
- net Net-(D6-K): track 0.00 -> 2.08 mm
- net Net-(D5-K): track 0.00 -> 2.08 mm
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Other:
- board text added: "139"
- board text added: "CSF"
- board text added: "CSR0"
- board text added: "CSR1"
- board text added: "OEF"
- board text added: "OER"
- board text added: "RAM1"
- board text added: "RMLV1616A BANK 0 HIGH"
- board text added: "RMLV1616A BANK 0 LOW"
- board text added: "RMLV1616A BANK 0 MID"
- board text added: "RMLV1616A BANK 1 HIGH"
- board text added: "RMLV1616A BANK 1 LOW"
- board text added: "RMLV1616A BANK 1 MID"
- board text added: "SST39SF040 HIGH"
- board text added: "SST39SF040 LOW"
- board text added: "SST39SF040 MID"
- board text added: "WEF"
- board text added: "WER"
- board text added: "~{OER}"
- board text added: "~{WER}"
- board text removed: "OE+"
- board text removed: "RAM3"
- board text removed: "WE+"
- board text removed: "~{OER0}"
- board text removed: "~{OER1}"
- board text removed: "~{WER0}"
- board text removed: "~{WER1}"

Commit message: Misc updstes
Connections:
- U7 pad 1: /A2 -> /A18
- U7 pad 10: /A14 -> /A2
- U7 pad 11: /A16 -> /A1
- U7 pad 12: /A17 -> /A0
- U7 pad 2: /A1 -> /A16
- U7 pad 23: /A15 -> /A10
- U7 pad 25: /A12 -> /A11
- U7 pad 26: /A10 -> /A9
- U7 pad 28: /A6 -> /A13
- U7 pad 29: /A4 -> /A14
- U7 pad 3: /A0 -> /A15
- U7 pad 30: /A3 -> /A17
- U7 pad 4: /A18 -> /A12
- U7 pad 5: /A5 -> /A7
- U7 pad 6: /A7 -> /A6
- U7 pad 7: /A9 -> /A5
- U7 pad 8: /A11 -> /A4
- U7 pad 9: /A13 -> /A3
- U8 pad 1: /A2 -> /A18
- U8 pad 10: /A14 -> /A2
- U8 pad 11: /A16 -> /A1
- U8 pad 12: /A17 -> /A0
- U8 pad 2: /A1 -> /A16
- U8 pad 23: /A15 -> /A10
- U8 pad 25: /A12 -> /A11
- U8 pad 26: /A10 -> /A9
- U8 pad 28: /A6 -> /A13
- U8 pad 29: /A4 -> /A14
- U8 pad 3: /A0 -> /A15
- U8 pad 30: /A3 -> /A17
- U8 pad 4: /A18 -> /A12
- U8 pad 5: /A5 -> /A7
- U8 pad 6: /A7 -> /A6
- U8 pad 7: /A9 -> /A5
- U8 pad 8: /A11 -> /A4
- U8 pad 9: /A13 -> /A3
- U9 pad 1: /A2 -> /A18
- U9 pad 10: /A14 -> /A2
- U9 pad 11: /A16 -> /A1
- U9 pad 12: /A17 -> /A0
- U9 pad 2: /A1 -> /A16
- U9 pad 23: /A15 -> /A10
- U9 pad 25: /A12 -> /A11
- U9 pad 26: /A10 -> /A9
- U9 pad 28: /A6 -> /A13
- U9 pad 29: /A4 -> /A14
- U9 pad 3: /A0 -> /A15
- U9 pad 30: /A3 -> /A17
- U9 pad 4: /A18 -> /A12
- U9 pad 5: /A5 -> /A7
- U9 pad 6: /A7 -> /A6
- U9 pad 7: /A9 -> /A5
- U9 pad 8: /A11 -> /A4
- U9 pad 9: /A13 -> /A3
Routing:
- net /A12: track 212.5 -> 247.9 mm, vias 0 -> 3
- net /A15: track 207.6 -> 242.0 mm, vias 0 -> 3
- net /A18: track 303.4 -> 270.2 mm, vias 15 -> 14
- net /A0: track 232.6 -> 212.5 mm, vias 3 -> 2
- net /A16: track 222.7 -> 242.4 mm, vias 0 -> 3
- net /A1: track 238.7 -> 223.1 mm, vias 3 -> 2
- net /A6: track 214.8 -> 229.6 mm, vias 0 -> 2
- net /A17: track 206.8 -> 219.5 mm, vias 0 -> 4
- net /A9: track 222.9 -> 211.8 mm, vias 0 -> 2
- net /A11: track 222.3 -> 211.2 mm, vias 0 -> 2
- net /A2: track 236.7 -> 225.7 mm, vias 3 -> 2
- net /A4: track 215.5 -> 226.2 mm, vias 0 -> 2
- net /~{WEF}: track 115.8 -> 105.5 mm
- net /A13: track 221.4 -> 214.5 mm, vias 0 -> 2
- net /~{OEF}: track 97.2 -> 103.4 mm
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Other:
- board text added: "A0"
- board text added: "A1"
- board text added: "A10"
- board text added: "A11"
- board text added: "A12"
- board text added: "A13"
- board text added: "A14"
- board text added: "A15"
- board text added: "A16"
- board text added: "A17"
- board text added: "A18"
- board text added: "A2"
- board text added: "A3"
- board text added: "A4"
- board text added: "A5"
- board text added: "A6"
- board text added: "A7"
- board text added: "A8"
- board text added: "A9"
- board text added: "CE#"
- board text added: "D0"
- board text added: "D1"
- board text added: "D2"
- board text added: "D3"
- board text added: "D4"
- board text added: "D5"
- board text added: "D6"
- board text added: "D7"
- board text added: "OE#"
- board text added: "VDD"
- board text added: "WE#"
- board text added: "• Memory • github.com/mengstr/SUBLEQ24 • rev2 •"
- board text removed: "• Memory • github.com/mengstr/SUBLEQ24 • rev1 •"
