File: PCB/Memory/Memory.kicad_sch (KiCad schematic)
At the start: 32 parts, among them J1 Conn_01x08_Pin, U1 74LS139, U1 RMLV1616A, U2 RMLV1616A, U3 RMLV1616A, U4 SST39SF020, U5 SST39SF020, U7 SST39SF020

Commit message: Update readme
Parts:
- removed JP1 (x2): SolderJumper_2_Open, Jumper:SolderJumper-2_P1.3mm_Open_Pad1.0x1.5mm, symbol Jumper:SolderJumper_2_Open
- added D1, D2, D3, D4, D5, D6, D7: LED, LED_SMD:LED_0805_2012Metric_Pad1.15x1.40mm_HandSolder, symbol Device:LED
- added R1, R2, R3, R4, R5, R6, R7: R, Resistor_SMD:R_0805_2012Metric_Pad1.20x1.40mm_HandSolder, symbol Device:R
- J1: value Conn_01x08_Pin -> Conn_01x06_Pin; footprint Connector_PinHeader_2.54mm:PinHeader_1x08_P2.54mm_Vertical -> Connector_PinHeader_2.54mm:PinHeader_1x06_P2.54mm_Vertical; symbol Connector:Conn_01x08_Pin -> Connector:Conn_01x06_Pin
- renumbered U1 to U10
Connections:
- net ~{WER1} is gone; now on net ~{WER}: J1.1 (Pin_1), U1.11 (WE#), U2.11 (WE#), U3.11 (WE#)
- net VCC: now also D1.2 (A), D2.2 (A), D3.2 (A), D4.2 (A), D5.2 (A), D6.2 (A), D7.2 (A)
- net ~{CS_FLASH}: now also R7.1
- net ~{CS_RAM0}: now also R5.1
- net ~{CS_RAM1}: now also R6.1
- net ~{OEF}: now also J1.4 (Pin_4), R4.1; no longer J1.6 (Pin_6)
- net ~{WEF}: now also J1.3 (Pin_3), R3.1; no longer J1.5 (Pin_5)
- net ~{OER0} renamed ~{OER}
- net ~{OER}: now also J1.2 (Pin_2), U1.28 (OE#), U2.28 (OE#), U3.28 (OE#), R2.1; no longer J1.4 (Pin_4)
- removed net ~{OER1}: J1.3 (Pin_3), U1.28 (OE#), U2.28 (OE#), U3.28 (OE#)
- net ~{WER0} renamed ~{WER}
- net ~{WER}: now also R1.1; no longer J1.2 (Pin_2)
- new net: D4.1 (K), R4.2
- new net: D6.1 (K), R6.2
- new net: D7.1 (K), R7.2
- new net: D5.1 (K), R5.2
- new net: D1.1 (K), R1.2
- new net: D2.1 (K), R2.2
- new net: D3.1 (K), R3.2
Other:
- moved on the sheet: U1, U2, U3, U4, U5, U7

Commit message: Misc updstes
Connections:
- net A0: now also U4.12 (A0), U5.12 (A0), U7.12 (A0); no longer U4.3 (A15), U5.3 (A15), U7.3 (A15)
- net A1: now also U4.11 (A1), U5.11 (A1), U7.11 (A1); no longer U4.2 (A16), U5.2 (A16), U7.2 (A16)
- net A10: now also U4.23 (A10), U5.23 (A10), U7.23 (A10); no longer U4.26 (A9), U5.26 (A9), U7.26 (A9)
- net A11: now also U4.25 (A11), U5.25 (A11), U7.25 (A11); no longer U4.8 (A4), U5.8 (A4), U7.8 (A4)
- net A12: now also U4.4 (A12), U5.4 (A12), U7.4 (A12); no longer U4.25 (A11), U5.25 (A11), U7.25 (A11)
- net A13: now also U4.28 (A13), U5.28 (A13), U7.28 (A13); no longer U4.9 (A3), U5.9 (A3), U7.9 (A3)
- net A14: now also U4.29 (A14), U5.29 (A14), U7.29 (A14); no longer U4.10 (A2), U5.10 (A2), U7.10 (A2)
- net A15: now also U4.3 (A15), U5.3 (A15), U7.3 (A15); no longer U4.23 (A10), U5.23 (A10), U7.23 (A10)
- net A16: now also U4.2 (A16), U5.2 (A16), U7.2 (A16); no longer U4.11 (A1), U5.11 (A1), U7.11 (A1)
- net A17: now also U4.30 (A17), U5.30 (A17), U7.30 (A17); no longer U4.12 (A0), U5.12 (A0), U7.12 (A0)
- net A18: now also U4.1 (NC), U5.1 (NC), U7.1 (NC); no longer U4.4 (A12), U5.4 (A12), U7.4 (A12)
- net A2: now also U4.10 (A2), U5.10 (A2), U7.10 (A2); no longer U4.1 (NC), U5.1 (NC), U7.1 (NC)
- net A3: now also U4.9 (A3), U5.9 (A3), U7.9 (A3); no longer U4.30 (A17), U5.30 (A17), U7.30 (A17)
- net A4: now also U4.8 (A4), U5.8 (A4), U7.8 (A4); no longer U4.29 (A14), U5.29 (A14), U7.29 (A14)
- net A5: now also U4.7 (A5), U5.7 (A5), U7.7 (A5); no longer U4.5 (A7), U5.5 (A7), U7.5 (A7)
- net A6: now also U4.6 (A6), U5.6 (A6), U7.6 (A6); no longer U4.28 (A13), U5.28 (A13), U7.28 (A13)
- net A7: now also U4.5 (A7), U5.5 (A7), U7.5 (A7); no longer U4.6 (A6), U5.6 (A6), U7.6 (A6)
- net A9: now also U4.26 (A9), U5.26 (A9), U7.26 (A9); no longer U4.7 (A5), U5.7 (A5), U7.7 (A5)
