File: PCB/Subtractor/LatchedSubtractor.kicad_pcb (KiCad board)
At the start: 4 copper layers, 101.6 x 76.2 mm, 67 parts, among them J1a1 Conn_02x04_Odd_Even, J1b1 Conn_02x04_Odd_Even, J1c1 Conn_02x04_Odd_Even, J2a1 Conn_02x04_Odd_Even, J2b1 Conn_02x04_Odd_Even, J2c1 Conn_02x04_Odd_Even, J3a1 Conn_02x04_Odd_Even, J3b1 Conn_02x04_Odd_Even, J3c1 Conn_02x04_Odd_Even, J4 Conn_01x08_Pin, U1 74LS283, U10 74HCT564, U11 74HCT564, U12 74HCT564, U13 74HC245, U14 74HC245, U15 74HC245, U16 74LS27, U17 74LS27, U18 74LS27, U19 74LS30, U2 74LS283, U20 74LS00, U3 74LS283, U4 74LS283, U5 74LS283, U6 74LS283, U7 74HCT574, U8 74HCT574, U9 74HCT574

Commit message: Update readme
Other:
- board text added: "• Latched value subtractor • github.com/mengstr/SUBLEQ24 • rev1 •"
- board text removed: "• ValueSubtractor • github.com/mengstr/SUBLEQ24 • rev1 •"
