File: PCB/UART/UART.kicad_pcb (KiCad board)
At the start: 2 copper layers, 101.6 x 76.2 mm, 58 parts, among them J1 DE9_Plug_MountingHoles, J11 Conn_01x08_Pin, J2 Conn_01x03_Pin, J3 Conn_02x09_Odd_Even, J4 USB4105-GF-A, U1 74HC165, U10 74HC04, U11 MAX3221, U13 FT231XS, U2 74HC165, U3 74LS393, U4 74LS393, U5 74HC74, U6 74HC74, U7 74HC595, U8 74HC00, U9 74HC00, Y1 Crystal_Small

Commit message: Updates ;-)
Parts:
- added C21: C, Capacitor_SMD:C_0805_2012Metric_Pad1.18x1.45mm_HandSolder, F.Cu at (87.6, 64.1)
- added C22: C, Capacitor_SMD:C_0805_2012Metric_Pad1.18x1.45mm_HandSolder, F.Cu at (57.6, 85.1)
- added C23: C, Capacitor_SMD:C_0805_2012Metric_Pad1.18x1.45mm_HandSolder, F.Cu at (67.3, 85.1)
- added C24: C, Capacitor_SMD:C_0805_2012Metric_Pad1.18x1.45mm_HandSolder, F.Cu at (77.4, 85.1)
- added C25: C, Capacitor_SMD:C_0805_2012Metric_Pad1.18x1.45mm_HandSolder, F.Cu at (87.6, 85.1)
- added C26: C, Capacitor_SMD:C_0805_2012Metric_Pad1.18x1.45mm_HandSolder, F.Cu at (97.8, 85.1)
- added J5: Conn_01x08_Pin, Connector_PinHeader_2.54mm:PinHeader_1x08_P2.54mm_Vertical, F.Cu at (50.8, 48.9)
- added J6: Conn_01x08_Pin, Connector_PinHeader_2.54mm:PinHeader_1x08_P2.54mm_Vertical, F.Cu at (50.8, 69.8)
- added U14: 74HCT541, Package_SO:SOIC-20W_7.5x12.8mm_P1.27mm, F.Cu at (44.5, 57.1)
- added U15: 74HCT541, Package_SO:SOIC-20W_7.5x12.8mm_P1.27mm, F.Cu at (44.5, 35.6)
- added U16: 74LS151, Package_SO:SOIC-16W_5.3x10.2mm_P1.27mm, F.Cu at (67.3, 35.6)
- added U17: 74LS11, Package_SO:SOIC-14_3.9x8.7mm_P1.27mm, F.Cu at (57.1, 35.6)
- U10: value 74HC04 -> 74HCT564; footprint Package_SO:SO-14_3.9x8.65mm_P1.27mm -> Package_SO:SOIC-20W_7.5x12.8mm_P1.27mm
- U5, U6: footprint Package_SO:SO-14_3.9x8.65mm_P1.27mm -> Package_SO:SOIC-14_3.9x8.7mm_P1.27mm
- moved C9 97.6 mm to (57.1, 64.1)
- moved C6 96.3 mm to (57.2, 42.5)
- moved C8 89.8 mm to (67.3, 43.2)
- moved C10 87.6 mm to (67.3, 64.1)
- moved C11 77.7 mm to (77.5, 64.1)
- moved C7 54.5 mm to (44.4, 87.2), turned to 0 degrees
- moved U10 48.7 mm to (44.5, 78.7), turned to 180 degrees
- moved U3 48.6 mm to (97.8, 78.1), turned to 180 degrees
- moved U1 46.1 mm to (67.3, 78.1), turned to 180 degrees
- moved C5 43.8 mm to (44.4, 65.8), turned to 0 degrees
- moved C12 43.0 mm to (99.1, 96.8), turned to 180 degrees
- moved U8 41.3 mm to (87.6, 78.1), turned to 180 degrees
- moved U2 41.1 mm to (57.1, 78.1), turned to 180 degrees
- moved C15 41.0 mm to (105.4, 94.7), turned to -90 degrees
- moved C2 40.8 mm to (93.3, 94.4)
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Connections:
- J11 pad 1: UART_Send -> ~{StatRd}
- J11 pad 2: UART_Read -> ~{BusyRd}
- J11 pad 3: MOPend -> ~{AvailRd}
- J11 pad 4: BUSY -> Stat
- J11 pad 5: ~{RES1} -> ~{RESET}
- J11 pad 6: RESET -> ~{OE}
- J11 pad 7: unconnected-(J11-Pin_7-Pad7) -> TxTrig
- U1 pad 10: Net-(U1-DS) -> VCC
- U1 pad 11: /D6 -> VCC
- U1 pad 12: /D5 -> VCC
- U1 pad 13: /D4 -> VCC
- U1 pad 14: /D3 -> VCC
- U1 pad 3: /D2 -> VCC
- U1 pad 4: /D1 -> VCC
- U1 pad 5: /D0 -> VCC
- U1 pad 6: VCC -> /Tx7
- U1 pad 7: /TXD -> unconnected-(U1-~{Q7}-Pad7)
- U1 pad 9: unconnected-(U1-Q7-Pad9) -> Net-(U1-Q7)
- U10 pad 1: Net-(U3A-Q3) -> GNDD
- U10 pad 10: Net-(U7-SER) -> GNDD
- U10 pad 11: /RXD -> TxTrig
- U10 pad 12: Net-(U5A-~{R}) -> /Tx0
- U10 pad 13: MOPend -> /Tx1
- U10 pad 14: VCC -> /Tx2
- U10 pad 2: Net-(U1-CP) -> /D7
- U10 pad 3: Net-(U10-Pad3) -> /D6
- U10 pad 4: Net-(U7-RCLK) -> /D5
- U10 pad 5: Net-(U6A-~{Q}) -> /D4
- U10 pad 6: Net-(U10-Pad6) -> /D3
- U10 pad 7: GNDD -> /D2
- U10 pad 8: Net-(U4A-MR) -> /D1
- U10 pad 9: Net-(U10-Pad6) -> /D0
- U2 pad 10: GNDD -> Net-(U1-Q7)
- U2 pad 11: GNDD -> /Tx6
- U2 pad 12: GNDD -> /Tx5
- U2 pad 13: GNDD -> /Tx4
- U2 pad 14: GNDD -> /Tx3
- U2 pad 3: GNDD -> /Tx2
- U2 pad 4: GNDD -> /Tx1
- U2 pad 5: GNDD -> /Tx0
- U2 pad 6: /D7 -> GNDD
- U2 pad 9: Net-(U1-DS) -> /TXD
- U3 pad 10: unconnected-(U3B-Q1-Pad10) -> Net-(U3B-Q1)
- U3 pad 11: Net-(U3B-Q0) -> unconnected-(U3B-Q0-Pad11)
- U3 pad 12: Net-(U3A-MR) -> /~{TxBusy}
- U3 pad 2: Net-(U3A-MR) -> /~{TxBusy}
- U5 pad 11: VCC -> TxTrig
- U5 pad 13: VCC -> /~{TxBusy}
- U5 pad 2: GNDD -> VCC
- U5 pad 3: ~{RES1} -> VCC
- U5 pad 5: Net-(U5A-Q) -> /TxBusy
- U5 pad 6: unconnected-(U5A-~{Q}-Pad6) -> /~{TxBusy}
- U5 pad 8: unconnected-(U5B-~{Q}-Pad8) -> Net-(U5B-~{Q})
- U6 pad 11: GNDD -> ~{RESET}
- U6 pad 13: Net-(U6B-~{R}) -> ~{OE}
- U6 pad 3: RESET -> ~{RESET}
- U6 pad 6: Net-(U6A-~{Q}) -> Net-(U4A-MR)
- U6 pad 8: unconnected-(U6B-~{Q}-Pad8) -> /~{RxRdy}
- U6 pad 9: AVAIL -> /RxRdy
- U7 pad 1: /D1 -> Net-(J5-Pin_7)
- U7 pad 10: VCC -> ~{RESET}
- U7 pad 13: Net-(U5A-~{S}) -> GNDD
- U7 pad 15: /D0 -> Net-(J5-Pin_8)
- U7 pad 2: /D2 -> Net-(J5-Pin_6)
- U7 pad 3: /D3 -> Net-(J5-Pin_5)
- U7 pad 4: /D4 -> Net-(J5-Pin_4)
- U7 pad 5: /D5 -> Net-(J5-Pin_3)
- U7 pad 6: /D6 -> Net-(J5-Pin_2)
- U7 pad 7: /D7 -> Net-(J5-Pin_1)
- U8 pad 1: Net-(U1-~{PL}) -> Net-(U3A-Q3)
- U8 pad 10: Net-(U3B-Q3) -> ~{RESET}
- U8 pad 11: Net-(U1-~{PL}) -> Net-(U5A-~{S})
- U8 pad 12: UART_Send -> Net-(U8-Pad12)
- U8 pad 13: UART_Send -> Net-(U8-Pad12)
- U8 pad 2: Net-(U3A-MR) -> Net-(U3A-Q3)
- U8 pad 3: BUSY -> Net-(U1-CP)
- U8 pad 4: BUSY -> Net-(U3B-Q1)
- U8 pad 5: Net-(U8-Pad5) -> Net-(U3B-Q3)
- U8 pad 6: Net-(U3A-MR) -> Net-(U5A-~{R})
- U8 pad 8: Net-(U8-Pad5) -> Net-(U8-Pad12)
- U8 pad 9: Net-(U3B-Q0) -> Net-(U5B-~{Q})
- U9 pad 1: Net-(U4B-Q0) -> /RXD
- U9 pad 10: UART_Read -> Net-(U7-RCLK)
- U9 pad 11: Net-(U6B-~{R}) -> Net-(U7-RCLK)
- U9 pad 12: Net-(U5A-Q) -> Net-(U9-Pad12)
- U9 pad 13: unconnected-(U9-Pad13) -> Net-(U9-Pad12)
- U9 pad 2: Net-(U4B-Q3) -> /RXD
- U9 pad 3: Net-(U10-Pad3) -> Net-(U7-SER)
- U9 pad 4: Net-(U4A-Q3) -> Net-(U4B-Q0)
- U9 pad 5: Net-(U7-RCLK) -> Net-(U4B-Q3)
- U9 pad 6: Net-(U6A-~{R}) -> Net-(U9-Pad12)
- U9 pad 8: Net-(U5A-~{S}) -> Net-(U6A-~{R})
- U9 pad 9: AVAIL -> Net-(U4A-Q3)
Routing:
- net GNDD: track 261.2 -> 702.6 mm, vias 14 -> 45
- net VCC: track 111.1 -> 508.9 mm, vias 6 -> 38
- net TxTrig: track 0.00 -> 109.9 mm, vias 0 -> 2
- net ~{RESET}: track 0.00 -> 103.9 mm, vias 0 -> 2
- net ~{OE}: track 0.00 -> 96.2 mm, vias 0 -> 2
- net ~{AvailRd}: track 0.00 -> 89.0 mm
- net /~{TxBusy}: track 0.00 -> 86.6 mm, vias 0 -> 4
- net ~{BusyRd}: track 0.00 -> 86.2 mm
- net ~{StatRd}: track 0.00 -> 83.4 mm
- net Stat: track 0.00 -> 82.6 mm
- net /BAUDCLK: track 24.3 -> 98.3 mm, vias 2 -> 3
- net /Tx6: track 0.00 -> 62.7 mm, vias 0 -> 2
- net Net-(J5-Pin_7): track 0.00 -> 59.1 mm
- net Net-(J5-Pin_8): track 0.00 -> 59.1 mm, vias 0 -> 2
- net Net-(U4A-Q3): track 0.00 -> 58.3 mm, vias 0 -> 4
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Other:
- board text added: "11"
- board text added: "151"
- board text added: "541"
- board text added: "564"
- board text added: "74"
- board text added: "Stat"
- board text added: "TxTrig"
- board text added: "~{AvailRd}"
- board text added: "~{BusyRd}"
- board text added: "~{OE}"
- board text added: "~{Reset}"
- board text added: "~{StatRd}"
- board text added: "• Serial • github.com/mengstr/SUBLEQ24 • rev1 •"
- board text removed: "• Template • github.com/mengstr/SUBLEQ24 • rev1 •"

Commit message: Misc updstes
Routing:
- net /TXD: track 123.2 -> 116.0 mm
Other:
- board text removed: "• Serial • github.com/mengstr/SUBLEQ24 • rev1 •"
