File: PCB/UART/UART.kicad_sch (KiCad schematic)
At the start: 58 parts, among them J1 DE9_Plug_MountingHoles, J2 Conn_01x03_Pin, J3 Conn_02x09_Odd_Even, J4 Conn_01x08_Pin, J4 USB4105-GF-A, U1 74HC165, U10 74HC04, U11 MAX3221, U13 FT231XS, U2 74HC165, U3 74LS393, U4 74LS393, U5 74HC74, U6 74HC74, U7 74HC595, U8 74HC00, U9 74HC00, Y1 Crystal_Small

Commit message: Updates ;-)
Parts:
- removed U10: 74HC04, Package_SO:SO-14_3.9x8.65mm_P1.27mm, symbol 74xx:74HC04
- added C21, C22, C23, C24, C25, C26: C, Capacitor_SMD:C_0805_2012Metric_Pad1.18x1.45mm_HandSolder, symbol Device:C
- added J5, J6: Conn_01x08_Pin, Connector_PinHeader_2.54mm:PinHeader_1x08_P2.54mm_Vertical, symbol Connector:Conn_01x08_Pin
- added U10: 74HCT564, Package_SO:SOIC-20W_7.5x12.8mm_P1.27mm, symbol 74xx:74HCT574
- added U14, U15: 74HCT541, Package_SO:SOIC-20W_7.5x12.8mm_P1.27mm, symbol 74xx:74HCT541
- added U16: 74LS151, Package_SO:SOIC-16W_5.3x10.2mm_P1.27mm, symbol 74xx:74LS151
- added U17: 74LS11, Package_SO:SOIC-14_3.9x8.7mm_P1.27mm, symbol 74xx:74LS11
- U5, U6: footprint Package_SO:SO-14_3.9x8.65mm_P1.27mm -> Package_SO:SOIC-14_3.9x8.7mm_P1.27mm
Connections:
- net D0: now also U10.9 (D7), U14.11 (Y7), U15.18 (Y0); no longer U1.5 (D6), U7.15 (QA)
- net D1: now also U10.8 (D6), U14.12 (Y6), U15.17 (Y1); no longer U1.4 (D5), U7.1 (QB)
- net D2: now also U10.7 (D5), U14.13 (Y5), U15.16 (Y2); no longer U1.3 (D4), U7.2 (QC)
- net D3: now also U10.6 (D4), U14.14 (Y4), U15.15 (Y3); no longer U1.14 (D3), U7.3 (QD)
- net D4: now also U10.5 (D3), U14.15 (Y3), U15.14 (Y4); no longer U1.13 (D2), U7.4 (QE)
- net D5: now also U10.4 (D2), U14.16 (Y2), U15.13 (Y5); no longer U1.12 (D1), U7.5 (QF)
- net D6: now also U10.3 (D1), U14.17 (Y1), U15.12 (Y6); no longer U1.11 (D0), U7.6 (QG)
- net D7: now also U10.2 (D0), U14.18 (Y0), U15.11 (Y7); no longer U2.6 (D7), U7.7 (QH)
- net GNDD: now also U2.6 (D7), U7.13 (~{OE}), C21.2, C22.2, C23.2, C24.2, C25.2, C26.2, U10.1 (OE), U10.10 (GND), U14.10 (GND), U15.10 (GND), U15.3 (A1), U15.4 (A2), U15.5 (A3), U15.6 (A4), U15.7 (A5), U15.8 (A6), U15.9 (A7), U16.12 (I7), U16.15 (I4), U16.2 (I2), U16.3 (I1), U16.4 (I0), U16.7 (~{E}), U16.8 (GND), U17.1, U17.10, U17.11, U17.13, U17.2, U17.7 (GND), U17.9; no longer U2.10 (DS), U2.11 (D0), U2.12 (D1), U2.13 (D2), U2.14 (D3), U2.3 (D4), U2.4 (D5), U2.5 (D6), U5.2 (D), U6.11 (C)
- net RXD: now also U9.1, U9.2
- net TXD: now also U2.9 (Q7); no longer U1.7 (~{Q7})
- net VCC: now also U1.10 (DS), U1.11 (D0), U1.12 (D1), U1.13 (D2), U1.14 (D3), U1.3 (D4), U1.4 (D5), U1.5 (D6), U5.2 (D), U5.3 (C), C21.1, C22.1, C23.1, C24.1, C25.1, C26.1, U10.20 (VCC), U14.20 (VCC), U15.20 (VCC), U16.16 (VCC), U17.14 (VCC); no longer U1.6 (D7), U5.11 (C), U5.13 (~{R}), U7.10 (~{SRCLR})
- net at U4.13 (CP), U4.6 (Q3), U7.11 (SRCLK): now also U9.9; no longer U9.4
- net at U9.5: now also U4.8 (Q3); no longer U7.12 (RCLK)
- net at U6.1 (~{R}), U6.10 (~{S}): now also U9.8; no longer U9.6
- net at U6.6 (~{Q}): now also U4.12 (MR), U4.2 (MR)
- net at U5.8 (~{Q}): now also U8.9
- net at U5.1 (~{R}): now also U8.6
- net ~{TxBusy}: now reaches U3.12 (MR), U3.2 (MR)
- net ~{TxBusy}: now also U5.13 (~{R}), U5.6 (~{Q}), U16.14 (I5); no longer U8.2, U8.6
- net at U3.13 (CP), U3.6 (Q3): now also U8.1, U8.2
- net at U4.11 (Q0): now also U9.4; no longer U9.1
- net at U9.3: now also U7.14 (SER)
- net at U9.12: now also U9.13, U9.6; no longer U5.5 (Q)
- net at U3.8 (Q3): now also U8.5; no longer U8.10
- net at U8.8: now also U8.12, U8.13; no longer U8.5
- net at U3.11 (Q0): no longer U8.9
- net at U9.11: now also U7.12 (RCLK), U9.10; no longer U6.13 (~{R})
- net ~{RxRdy}: now reaches U6.8 (~{Q})
- net at U1.1 (~{PL}), U2.1 (~{PL}): no longer U8.1, U8.11
- net at U3.10 (Q1): now also U8.4
- net TxTrig: now reaches J4.7 (Pin_7)
- net TxTrig: now also U5.11 (C), U10.11 (Cp)
- net at U1.2 (CP), U2.2 (CP): now also U8.3
- net at U1.9 (Q7): now also U2.10 (DS)
- net AVAIL renamed RxRdy
- net RxRdy: now also U16.13 (I6); no longer U9.9
- removed net BUSY: J4.4 (Pin_4), U8.3, U8.4
- net MOPend renamed ~{AvailRd}
- net ~{AvailRd}: now also U16.11 (S0), U17.3
- net RESET renamed ~{OE}
- net ~{OE}: now also U6.13 (~{R}), U14.1 (G1), U14.19 (G2); no longer U6.3 (C)
- net UART_Read renamed ~{BusyRd}
- net ~{BusyRd}: now also U16.10 (S1), U17.4; no longer U9.10
- removed net UART_Send: J4.1 (Pin_1), U8.12, U8.13
- net ~{RES1} renamed ~{RESET}
- net ~{RESET}: now also U6.11 (C), U6.3 (C), U7.10 (~{SRCLR}), U8.10; no longer U5.3 (C)
- new net: J5.1 (Pin_1), U14.9 (A7), U7.7 (QH)
- new net: J5.2 (Pin_2), U14.8 (A6), U7.6 (QG)
- new net: J5.3 (Pin_3), U14.7 (A5), U7.5 (QF)
- new net: J5.4 (Pin_4), U14.6 (A4), U7.4 (QE)
- new net: J5.5 (Pin_5), U14.5 (A3), U7.3 (QD)
- new net: J5.6 (Pin_6), U14.4 (A2), U7.2 (QC)
- new net: J5.7 (Pin_7), U14.3 (A1), U7.1 (QB)
- new net: J5.8 (Pin_8), U14.2 (A0), U7.15 (QA)
- new net: U15.1 (G1), U15.19 (G2), U17.6
- new net: U15.2 (A0), U16.5 (Z)
- new net: U5.4 (~{S}), U8.11
- new net Stat: J4.4 (Pin_4), U16.1 (I3)
- new net Tx0: J6.1 (Pin_1), U10.12 (Q7), U2.5 (D6)
- new net Tx1: J6.2 (Pin_2), U10.13 (Q6), U2.4 (D5)
- new net Tx2: J6.3 (Pin_3), U10.14 (Q5), U2.3 (D4)
- new net Tx3: J6.4 (Pin_4), U10.15 (Q4), U2.14 (D3)
- new net Tx4: J6.5 (Pin_5), U10.16 (Q3), U2.13 (D2)
- new net Tx5: J6.6 (Pin_6), U10.17 (Q2), U2.12 (D1)
- new net Tx6: J6.7 (Pin_7), U10.18 (Q1), U2.11 (D0)
- new net Tx7: J6.8 (Pin_8), U1.6 (D7), U10.19 (Q0)
- new net TxBusy: U5.5 (Q)
- new net ~{StatRd}: J4.1 (Pin_1), U16.9 (S2), U17.5
- no-connect marks 26 -> 25
Other:
- note added: "ABC 111 = 7 011 = 6 101 = 5 110 = 3"
- moved on the sheet: C1, C16, C17, C2, C3, C4, C5, C6, C7, C8, C9, C96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

Commit message: Misc updstes
Connections:
- net at U5.8 (~{Q}), U8.9: now also U1.1 (~{PL}), U2.1 (~{PL})
Changed lines of the file:
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@@
   (junction (at 78.74 115.57) (diameter 0) (color 0 0 0 0)
   )
+  (junction (at 185.42 165.1) (diameter 0) (color 0 0 0 0)
+  )
   (junction (at 183.515 271.78) (diameter 0) (color 0 0 0 0)
   )
@@
     (stroke (width 0) (type default))
   )
+  (wire (pts (xy 185.42 158.75) (xy 302.26 158.75))
+    (stroke (width 0) (type default))
+  )
   (wire (pts (xy 354.33 146.05) (xy 354.33 201.93))
     (stroke (width 0) (type default))
@@
     (stroke (width 0) (type default))
   )
+  (wire (pts (xy 185.42 158.75) (xy 185.42 165.1))
+    (stroke (width 0) (type default))
+  )
   (wire (pts (xy 96.52 118.11) (xy 97.79 118.11))
     (stroke (width 0) (type default))
@@
     (stroke (width 0) (type default))
   )
+  (wire (pts (xy 302.26 158.75) (xy 302.26 163.83))
+    (stroke (width 0) (type default))
+  )
   (wire (pts (xy 69.85 113.03) (xy 68.58 113.03))
     (stroke (width 0) (type default))
@@
       (effects (font (size 1.27 1.27)) hide)
     )
-    (property "Datasheet" "https://www.ftdichip.com/Support/Documents/DataSheets/ICs/DS_FT231X.pdf" (at 119.38 128.27 0)
+    (property "Datasheet" "https://ftdichip.com/wp-content/uploads/2021/10/DS_FT231X.pdf" (at 119.38 128.27 0)
       (effects (font (size 1.27 1.27)) hide)
     )
